File: main/keyboard.kicad_sch (KiCad schematic)
At the start: 9 parts, among them SW1 SW_Push, SW2 SW_Push, SW3 SW_Push, SW4 SW_Push, SW5 SW_Push

Commit message: keyboard circuit fix
Connections:
- net at SW3.1, SW4.1: now also R?.2
Changed lines of the file:
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@@
   (junction (at 121.92 91.44) (diameter 0) (color 0 0 0 0)
+  )
+  (junction (at 107.95 78.74) (diameter 0) (color 0 0 0 0)
   )
   (junction (at 88.9 78.74) (diameter 0) (color 0 0 0 0)
@@
     (stroke (width 0) (type default))
   )
-  (wire (pts (xy 107.95 66.04) (xy 107.95 91.44))
+  (wire (pts (xy 107.95 66.04) (xy 107.95 78.74))
     (stroke (width 0) (type default))
   )
@@
   )
   (wire (pts (xy 107.95 91.44) (xy 111.76 91.44))
+    (stroke (width 0) (type default))
+  )
+  (wire (pts (xy 107.95 78.74) (xy 107.95 91.44))
     (stroke (width 0) (type default))
   )
@@
     (stroke (width 0) (type default))
   )
-  (wire (pts (xy 101.6 78.74) (xy 102.87 78.74))
+  (wire (pts (xy 101.6 78.74) (xy 107.95 78.74))
     (stroke (width 0) (type default))
   )
