File: main/main.kicad_sch (KiCad schematic)
At the start: 19 parts, among them U1 STM32F411CEU6, U100 AP1117-33, U4 AT24CS64-SSHM, Y1 32768kHz

Commit message: keyboard circuit added
Connections:
- net Keyboard/keyb: now reaches U1.12 (PA2)
Other:
- added sheet Keyboard (keyboard.kicad_sch)
- moved on the sheet: C7, C8, U100

Commit message: keyboard circuit fix
Changed lines of the file:
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@@
     (stroke (width 0) (type default))
   )
-  (wire (pts (xy 154.94 63.5) (xy 129.54 63.5))
+  (wire (pts (xy 129.54 63.5) (xy 162.56 63.5))
     (stroke (width 0) (type default))
   )
@@
     (stroke (width 0) (type default))
   )
-  (wire (pts (xy 154.94 60.96) (xy 154.94 63.5))
-    (stroke (width 0) (type default))
-  )
   (wire (pts (xy 86.36 39.37) (xy 86.36 40.64))
     (stroke (width 0) (type default))
@@
   )
   (bus (pts (xy 142.24 82.55) (xy 142.24 157.48))
-    (stroke (width 0) (type default))
-  )
-  (wire (pts (xy 162.56 60.96) (xy 154.94 60.96))
     (stroke (width 0) (type default))
   )
@@
     )
   )
-  (sheet (at 162.56 58.42) (size 13.97 5.08) (fields_autoplaced)
+  (sheet (at 162.56 60.96) (size 13.97 5.08) (fields_autoplaced)
     (stroke (width 0.1524) (type solid))
     (fill (color 0 0 0 0.0000))
-    (property "Sheetname" "Keyboard" (at 162.56 57.7084 0)
+    (property "Sheetname" "Keyboard" (at 162.56 60.2484 0)
       (effects (font (size 1.27 1.27)) (justify left bottom))
     )
-    (property "Sheetfile" "keyboard.kicad_sch" (at 162.56 64.0846 0)
+    (property "Sheetfile" "keyboard.kicad_sch" (at 162.56 66.6246 0)
       (effects (font (size 1.27 1.27)) (justify left top))
     )
-    (pin "keyb" output (at 162.56 60.96 180)
-      (effects (font (size 1.27 1.27)) (justify left))
-    )
+    (pin "keyb" output (at 162.56 63.5 180)
+      (effects (font (size 1.27 1.27)) (justify left))
+    )

Commit message: Display added, PA6 used for display  MISO, PA3 used for i2s MCLK
Connections:
- net mck: now also U1.13 (PA3); no longer U1.16 (PA6)
- net SCLK: now reaches U1.15 (PA5)
- net MOSI: now reaches U1.17 (PA7)
- net displ_DC: now reaches U1.18 (PB0)
- net displ_CS: now reaches U1.19 (PB1)
- net displ_RESET: now reaches U1.20 (PB2)
- new net MISO: U1.16 (PA6)
- no-connect marks 1 -> 6
Other:
- added sheet Display ILI9341 (display.kicad_sch)
- moved on the sheet: R14, R15, Y1

Commit message: Power supply connectors added
Connections:
- net usb_dm: now reaches U1.32 (PA11)
- net usb_dp: now reaches U1.33 (PA12)
Other:
- added sheet Power supply (power.kicad_sch)

Commit message: Encoder added
Parts:
- added SW6: RotaryEncoder, symbol Device:RotaryEncoder
Connections:
- net GND: now also SW6.C
- net enc_a: now reaches U1.38 (PA15)
- net enc_a: now also SW6.A
- net enc_b: now reaches U1.39 (PB3)
- net enc_b: now also SW6.B
Changed lines of the file:
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@@
     (stroke (width 0) (type default))
   )
-  (bus_entry (at 90.17 93.98) (size 2.54 2.54)
+  (bus_entry (at 88.9 93.98) (size 2.54 2.54)
     (stroke (width 0) (type default))
   )
@@
     (stroke (width 0) (type default))
   )
-  (wire (pts (xy 92.71 96.52) (xy 96.52 96.52))
+  (wire (pts (xy 91.44 96.52) (xy 96.52 96.52))
     (stroke (width 0) (type default))
   )
@@
     (stroke (width 0) (type default))
   )
-  (bus (pts (xy 80.01 93.98) (xy 90.17 93.98))
+  (bus (pts (xy 80.01 93.98) (xy 88.9 93.98))
     (stroke (width 0) (type default))
   )
@@
     (effects (font (size 1.27 1.27)) (justify right bottom))
   )
+  (label "enc_a" (at 129.54 96.52 0) (fields_autoplaced)
+    (effects (font (size 1.27 1.27)) (justify left bottom))
+  )
   (label "scl" (at 64.77 110.49 0) (fields_autoplaced)
     (effects (font (size 1.27 1.27)) (justify left bottom))
@@
     (effects (font (size 1.27 1.27)) (justify right bottom))
   )
+  (label "enc_b" (at 231.14 139.7 180) (fields_autoplaced)
+    (effects (font (size 1.27 1.27)) (justify right bottom))
+  )
   (label "MCK_EXT" (at 187.96 139.7 180) (fields_autoplaced)
     (effects (font (size 1.27 1.27)) (justify right bottom))
@@
     (effects (font (size 1.27 1.27)) (justify right bottom))
   )
+  (label "enc_b" (at 96.52 93.98 180) (fields_autoplaced)
+    (effects (font (size 1.27 1.27)) (justify right bottom))
+  )
   (label "MOSI" (at 129.54 76.2 0)
     (effects (font (size 1.27 1.27)) (justify left bottom))
@@
   )
   (label "reset" (at 96.52 99.06 180) (fields_autoplaced)
+    (effects (font (size 1.27 1.27)) (justify right bottom))
+  )
+  (label "enc_a" (at 231.14 134.62 180) (fields_autoplaced)
     (effects (font (size 1.27 1.27)) (justify right bottom))
   )
@@
         (path "/cb08c644-d155-44e5-86e1-31645eace055"
           (reference "R14") (unit 1)
+        )
+      )
+    )
+  )
+  (symbol (lib_id "Device:RotaryEncoder") (at 238.76 137.16 0) (unit 1)
+    (in_bom yes) (on_board yes) (dnp no) (fields_autoplaced)
+    (property "Reference" "SW6" (at 245.11 135.89 0)
+      (effects (font (size 1.27 1.27)) (justify left))
+    )
+    (property "Value" "RotaryEncoder" (at 245.11 138.43 0)
+      (effects (font (size 1.27 1.27)) (justify left))
+    )
+    (property "Footprint" "" (at 234.95 133.096 0)
+      (effects (font (size 1.27 1.27)) hide)
+    )
+    (property "Datasheet" "~" (at 238.76 130.556 0)
+      (effects (font (size 1.27 1.27)) hide)
+    )
+    (pin "A")
+    (pin "B")
+    (pin "C")
+    (instances
+      (project "main"
+        (path "/cb08c644-d155-44e5-86e1-31645eace055"
+          (reference "SW6") (unit 1)
         )
       )
@@
         )
       )
+    )
+  )
+  (symbol (lib_id "power:GND") (at 231.14 137.16 270) (unit 1)
+    (in_bom yes) (on_board yes) (dnp no) (fields_autoplaced)
+    (property "Reference" "#PWR022" (at 224.79 137.16 0)
+      (effects (font (size 1.27 1.27)) hide)
+    )
+    (property "Value" "GND" (at 227.33 137.16 90)
+      (effects (font (size 1.27 1.27)) (justify right))
+    )
+    (property "Footprint" "" (at 231.14 137.16 0)
+      (effects (font (size 1.27 1.27)) hide)
+    )
+    (property "Datasheet" "" (at 231.14 137.16 0)
+      (effects (font (size 1.27 1.27)) hide)
+    )
+    (pin "1")
+    (instances
+      (project "main"
+        (path "/cb08c644-d155-44e5-86e1-31645eace055/e511764a-2dd7-4601-8d00-331d6dbffa9f"
+          (reference "#PWR022") (unit 1)
+        )
+        (path "/cb08c644-d155-44e5-86e1-31645eace055"
+          (reference "#PWR045") (unit 1)
+        )
+      )

Commit message: PWR flags added
Other:
- moved on the sheet: BT1
Changed lines of the file:
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@@
   (bus_alias "i2s" (members "ws" "ck" "sdi" "sdo" "mck" "reset"))
   (bus_alias "spi" (members "MOSI" "MISO" "SCLK"))
+  (junction (at 109.22 50.8) (diameter 0) (color 0 0 0 0)
+  )
   (junction (at 182.88 109.22) (diameter 0) (color 0 0 0 0)
   )
@@
   )
   (junction (at 172.72 116.84) (diameter 0) (color 0 0 0 0)
+  )
+  (junction (at 135.89 40.64) (diameter 0) (color 0 0 0 0)
   )
   (junction (at 138.43 85.09) (diameter 0) (color 0 0 0 0)
@@
     (stroke (width 0) (type default))
   )
+  (wire (pts (xy 102.87 50.8) (xy 109.22 50.8))
+    (stroke (width 0) (type default))
+  )
   (wire (pts (xy 182.88 116.84) (xy 172.72 116.84))
     (stroke (width 0) (type default))
@@
     (stroke (width 0) (type default))
   )
+  (wire (pts (xy 109.22 50.8) (xy 109.22 53.34))
+    (stroke (width 0) (type default))
+  )
   (bus (pts (xy 146.05 76.2) (xy 146.05 78.74))
     (stroke (width 0) (type default))
@@
     (stroke (width 0) (type default))
   )
-  (wire (pts (xy 109.22 45.72) (xy 109.22 53.34))
+  (wire (pts (xy 109.22 44.45) (xy 109.22 50.8))
     (stroke (width 0) (type default))
   )
@@
     (stroke (width 0) (type default))
   )
+  (bus (pts (xy 146.05 73.66) (xy 146.05 76.2))
+    (stroke (width 0) (type default))
+  )
+  (wire (pts (xy 54.61 78.74) (xy 54.61 80.01))
+    (stroke (width 0) (type default))
+  )
   (wire (pts (xy 87.63 99.06) (xy 96.52 99.06))
     (stroke (width 0) (type default))
   )
-  (bus (pts (xy 146.05 73.66) (xy 146.05 76.2))
-    (stroke (width 0) (type default))
-  )
-  (wire (pts (xy 54.61 78.74) (xy 54.61 80.01))
-    (stroke (width 0) (type default))
-  )
   (wire (pts (xy 87.63 114.3) (xy 96.52 114.3))
     (stroke (width 0) (type default))
@@
     (stroke (width 0) (type default))
   )
-  (wire (pts (xy 109.22 38.1) (xy 109.22 35.56))
+  (wire (pts (xy 109.22 36.83) (xy 109.22 35.56))
     (stroke (width 0) (type default))
   )
@@
     (stroke (width 0) (type default))
   )
+  (wire (pts (xy 135.89 40.64) (xy 139.7 40.64))
+    (stroke (width 0) (type default))
+  )
   (bus (pts (xy 220.98 73.66) (xy 220.98 76.2))
     (stroke (width 0) (type default))
@@
     (stroke (width 0) (type default))
   )
-  (wire (pts (xy 128.27 40.64) (xy 139.7 40.64))
+  (wire (pts (xy 128.27 40.64) (xy 135.89 40.64))
     (stroke (width 0) (type default))
   )
@@
     )
   )
-  (symbol (lib_id "Device:Battery_Cell") (at 109.22 40.64 0) (mirror x) (unit 1)
+  (symbol (lib_id "Device:Battery_Cell") (at 109.22 39.37 0) (mirror x) (unit 1)
     (in_bom yes) (on_board yes) (dnp no)
-    (property "Reference" "BT1" (at 105.41 41.2115 0)
+    (property "Reference" "BT1" (at 105.41 39.9415 0)
       (effects (font (size 1.27 1.27)) (justify right))
     )
-    (property "Value" "3.3V" (at 105.41 43.7515 0)
+    (property "Value" "3.3V" (at 105.41 42.4815 0)
       (effects (font (size 1.27 1.27)) (justify right))
     )
-    (property "Footprint" "" (at 109.22 42.164 90)
-      (effects (font (size 1.27 1.27)) hide)
-    )
-    (property "Datasheet" "~" (at 109.22 42.164 90)
+    (property "Footprint" "" (at 109.22 40.894 90)
+      (effects (font (size 1.27 1.27)) hide)
+    )
+    (property "Datasheet" "~" (at 109.22 40.894 90)
       (effects (font (size 1.27 1.27)) hide)
     )
@@
     )
   )
+  (symbol (lib_id "power:PWR_FLAG") (at 102.87 50.8 0) (unit 1)
+    (in_bom yes) (on_board yes) (dnp no) (fields_autoplaced)
+    (property "Reference" "#FLG01" (at 102.87 48.895 0)
+      (effects (font (size 1.27 1.27)) hide)
+    )
+    (property "Value" "PWR_FLAG" (at 102.87 45.72 0)
+      (effects (font (size 1.27 1.27)))
+    )
+    (property "Footprint" "" (at 102.87 50.8 0)
+      (effects (font (size 1.27 1.27)) hide)
+    )
+    (property "Datasheet" "~" (at 102.87 50.8 0)
+      (effects (font (size 1.27 1.27)) hide)
+    )
+    (pin "1")
+    (instances
+      (project "main"
+        (path "/cb08c644-d155-44e5-86e1-31645eace055"
+          (reference "#FLG01") (unit 1)
+        )
+      )
+    )
+  )
   (symbol (lib_id "power:GND") (at 243.84 114.3 0) (unit 1)
     (in_bom yes) (on_board yes) (dnp no) (fields_autoplaced)
@@
         )
       )
+    )
+  )
+  (symbol (lib_id "power:PWR_FLAG") (at 135.89 40.64 0) (unit 1)
+    (in_bom yes) (on_board yes) (dnp no) (fields_autoplaced)
+    (property "Reference" "#FLG03" (at 135.89 38.735 0)
+      (effects (font (size 1.27 1.27)) hide)
+    )
+    (property "Value" "PWR_FLAG" (at 135.89 35.56 0)
+      (effects (font (size 1.27 1.27)))
+    )
+    (property "Footprint" "" (at 135.89 40.64 0)
+      (effects (font (size 1.27 1.27)) hide)
+    )
+    (property "Datasheet" "~" (at 135.89 40.64 0)
+      (effects (font (size 1.27 1.27)) hide)
+    )
+    (pin "1")
+    (instances
+      (project "main"
+        (path "/cb08c644-d155-44e5-86e1-31645eace055"
+          (reference "#FLG03") (unit 1)
+        )
+      )

Commit message: LED control moved back to its original place
Connections:
- net displ_LED: now also U1.21 (PB10)
- no-connect marks 6 -> 8
Changed lines of the file:
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@@
   (junction (at 182.88 111.76) (diameter 0) (color 0 0 0 0)
   )
+  (no_connect (at 96.52 101.6))
   (no_connect (at 233.68 102.87))
   (no_connect (at 233.68 95.25))
   (no_connect (at 233.68 105.41))
+  (no_connect (at 96.52 104.14))
   (no_connect (at 233.68 97.79))
   (no_connect (at 96.52 71.12))
@@
     (effects (font (size 1.27 1.27)) (justify right bottom))
   )
-  (label "displ_LED" (at 76.2 87.63 180) (fields_autoplaced)
-    (effects (font (size 1.27 1.27)) (justify right bottom))
-  )
+  (label "displ_LED" (at 96.52 111.76 180) (fields_autoplaced)
+    (effects (font (size 1.27 1.27)) (justify right bottom))
+  )

Commit message: TODO comment about WKUP pin added
Connections:
- no-connect marks 8 -> 11
Other:
- note added: "TODO: PA0 is WKUP pin and will be used in the future, leave it unused"
Changed lines of the file:
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@@
   )
   (no_connect (at 96.52 101.6))
+  (no_connect (at 96.52 109.22))
   (no_connect (at 233.68 102.87))
   (no_connect (at 233.68 95.25))
@@
   (no_connect (at 96.52 71.12))
   (no_connect (at 233.68 100.33))
+  (no_connect (at 96.52 106.68))
+  (no_connect (at 96.52 76.2))
   (bus_entry (at 67.31 114.3) (size -2.54 -2.54)
     (stroke (width 0) (type default))
@@
     (stroke (width 0) (type default))
   )
+  (text "TODO: PA0 is WKUP pin and will be used in the\nfuture, leave it unused"
+    (at 144.78 55.88 0)
+    (effects (font (size 1.27 1.27)) (justify left bottom))
+  )
   (label "MCK_EXT" (at 63.5 68.58 0) (fields_autoplaced)
