File: main/main.kicad_sch (KiCad schematic)
At the start: 20 parts, among them SW6 RotaryEncoder, U1 STM32F411CEU6, U100 AP1117-33, U4 AT24CS64-SSHM, Y1 32768kHz

Commit message: Key added
Connections:
- net Telegraph key/KEY_DAH: now reaches U1.30 (PA9)
- net Telegraph key/KEY_DIT: now reaches U1.31 (PA10)
Other:
- added sheet Telegraph key (tkey.kicad_sch)
- moved on the sheet: U4

Commit message: SWD connector added
Parts:
- added J6: Conn_01x05_Pin, symbol Connector:Conn_01x05_Pin
Connections:
- net +3.3V: now also J6.2 (Pin_2)
- net GND: now also J6.1 (Pin_1)
- net swdio: now reaches U1.34 (PA13)
- net swdio: now also J6.4 (Pin_4)
- net swclk: now reaches U1.37 (PA14)
- net swclk: now also J6.3 (Pin_3)
- net swrst: now reaches C1.1, R1.1, U1.7 (NRST)
- net swrst: now also J6.5 (Pin_5)
Other:
- note added: "TODO: rewire to SWD standard"
Changed lines of the file:
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@@
+    (stroke (width 0) (type default))
+  )
+  (wire (pts (xy 62.23 40.64) (xy 86.36 40.64))
     (stroke (width 0) (type default))
   )
@@
   (wire (pts (xy 194.31 109.22) (xy 194.31 111.76))
     (stroke (width 0) (type default))
+  )
+  (text "TODO: rewire to SWD standard" (at 41.91 44.45 0)
+    (effects (font (size 1.27 1.27)) (justify left bottom))
   )
   (text "TODO: PA0 is WKUP pin and will be used in the\nfuture, leave it unused"
@@
     (effects (font (size 1.27 1.27)) (justify right bottom))
   )
+  (label "swclk" (at 129.54 93.98 0) (fields_autoplaced)
+    (effects (font (size 1.27 1.27)) (justify left bottom))
+  )
   (label "displ_DC" (at 233.68 73.66 180) (fields_autoplaced)
     (effects (font (size 1.27 1.27)) (justify right bottom))
@@
     (effects (font (size 1.27 1.27)) (justify right bottom))
   )
+  (label "swclk" (at 62.23 35.56 0) (fields_autoplaced)
+    (effects (font (size 1.27 1.27)) (justify left bottom))
+  )
   (label "enc_b" (at 96.52 93.98 180) (fields_autoplaced)
     (effects (font (size 1.27 1.27)) (justify right bottom))
@@
     (effects (font (size 1.27 1.27)) (justify left bottom))
   )
+  (label "swrst" (at 62.23 40.64 0) (fields_autoplaced)
+    (effects (font (size 1.27 1.27)) (justify left bottom))
+  )
   (label "displ_CS" (at 233.68 83.82 180) (fields_autoplaced)
     (effects (font (size 1.27 1.27)) (justify right bottom))
+  )
+  (label "swdio" (at 129.54 91.44 0) (fields_autoplaced)
+    (effects (font (size 1.27 1.27)) (justify left bottom))
+  )
+  (label "swdio" (at 62.23 38.1 0) (fields_autoplaced)
+    (effects (font (size 1.27 1.27)) (justify left bottom))
   )
   (label "displ_LED" (at 96.52 111.76 180) (fields_autoplaced)
@@
     )
   )
+  (symbol (lib_id "power:GND") (at 62.23 30.48 90) (unit 1)
+    (in_bom yes) (on_board yes) (dnp no) (fields_autoplaced)
+    (property "Reference" "#PWR048" (at 68.58 30.48 0)
+      (effects (font (size 1.27 1.27)) hide)
+    )
+    (property "Value" "GND" (at 66.04 30.48 90)
+      (effects (font (size 1.27 1.27)) (justify right))
+    )
+    (property "Footprint" "" (at 62.23 30.48 0)
+      (effects (font (size 1.27 1.27)) hide)
+    )
+    (property "Datasheet" "" (at 62.23 30.48 0)
+      (effects (font (size 1.27 1.27)) hide)
+    )
+    (pin "1")
+    (instances
+      (project "main"
+        (path "/cb08c644-d155-44e5-86e1-31645eace055"
+          (reference "#PWR048") (unit 1)
+        )
+      )
+    )
+  )
   (symbol (lib_id "power:GND") (at 231.14 137.16 270) (unit 1)
     (in_bom yes) (on_board yes) (dnp no) (fields_autoplaced)
@@
         (path "/cb08c644-d155-44e5-86e1-31645eace055"
           (reference "#PWR038") (unit 1)
+        )
+      )
+    )
+  )
+  (symbol (lib_id "Connector:Conn_01x05_Pin") (at 57.15 35.56 0) (unit 1)
+    (in_bom yes) (on_board yes) (dnp no)
+    (property "Reference" "J6" (at 57.785 25.4 0)
+      (effects (font (size 1.27 1.27)))
+    )
+    (property "Value" "Conn_01x05_Pin" (at 57.785 27.94 0)
+      (effects (font (size 1.27 1.27)))
+    )
+    (property "Footprint" "" (at 57.15 35.56 0)
+      (effects (font (size 1.27 1.27)) hide)
+    )
+    (property "Datasheet" "~" (at 57.15 35.56 0)
+      (effects (font (size 1.27 1.27)) hide)
+    )
+    (property "name" "swd conn" (at 58.42 22.86 0)
+      (effects (font (size 1.27 1.27)))
+    )
+    (pin "1")
+    (pin "5")
+    (pin "2")
+    (pin "4")
+    (pin "3")
+    (instances
+      (project "main"
+        (path "/cb08c644-d155-44e5-86e1-31645eace055"
+          (reference "J6") (unit 1)
         )
       )
@@
         )
       )
+    )
+  )
+  (symbol (lib_id "power:+3.3V") (at 62.23 33.02 270) (unit 1)
+    (in_bom yes) (on_board yes) (dnp no) (fields_autoplaced)
+    (property "Reference" "#PWR049" (at 58.42 33.02 0)
+      (effects (font (size 1.27 1.27)) hide)
+    )
+    (property "Value" "+3.3V" (at 66.04 33.02 90)
+      (effects (font (size 1.27 1.27)) (justify left))
+    )
+    (property "Footprint" "" (at 62.23 33.02 0)
+      (effects (font (size 1.27 1.27)) hide)
+    )
+    (property "Datasheet" "" (at 62.23 33.02 0)
+      (effects (font (size 1.27 1.27)) hide)
+    )
+    (pin "1")
+    (instances
+      (project "main"
+        (path "/cb08c644-d155-44e5-86e1-31645eace055"
+          (reference "#PWR049") (unit 1)
+        )
+      )

Commit message: Filters added
Other:
- added sheet Filters (filters.kicad_sch)
Changed lines of the file:
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@@
+    )
+  )
+  (sheet (at 104.14 173.99) (size 25.4 12.7) (fields_autoplaced)
+    (stroke (width 0.1524) (type solid))
+    (fill (color 0 0 0 0.0000))
+    (property "Sheetname" "Filters" (at 104.14 173.2784 0)
+      (effects (font (size 1.27 1.27)) (justify left bottom))
+    )
+    (property "Sheetfile" "filters.kicad_sch" (at 104.14 187.2746 0)
+      (effects (font (size 1.27 1.27)) (justify left top))
+    )
+    (pin "BPF2_OUT" output (at 129.54 179.07 0)
+      (effects (font (size 1.27 1.27)) (justify right))
+    )
+    (pin "BPF1_IN" input (at 104.14 176.53 180)
+      (effects (font (size 1.27 1.27)) (justify left))
+    )
+    (pin "BPF2_IN" input (at 104.14 179.07 180)
+      (effects (font (size 1.27 1.27)) (justify left))
+    )
+    (pin "BPF1_OUT" output (at 129.54 176.53 0)
+      (effects (font (size 1.27 1.27)) (justify right))
+    )
+    (pin "BPF3_IN" input (at 104.14 181.61 180)
+      (effects (font (size 1.27 1.27)) (justify left))
+    )
+    (pin "BPF3_OUT" output (at 129.54 181.61 0)
+      (effects (font (size 1.27 1.27)) (justify right))
+    )
+    (pin "BPF4_IN" input (at 104.14 184.15 180)
+      (effects (font (size 1.27 1.27)) (justify left))
+    )
+    (pin "BPF4_OUT" output (at 129.54 184.15 0)
+      (effects (font (size 1.27 1.27)) (justify right))
+    )
+    (instances
+      (project "main"
+        (path "/cb08c644-d155-44e5-86e1-31645eace055" (page "8"))
+      )
     )
   )

Commit message: Filter selector added
Other:
- removed sheet Filters
- added sheet Filter selector (filter_selector.kicad_sch)
Changed lines of the file:
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@@
+    )
+  )
+  (sheet (at 60.96 176.53) (size 13.97 7.62) (fields_autoplaced)
+    (stroke (width 0.1524) (type solid))
+    (fill (color 0 0 0 0.0000))
+    (property "Sheetname" "Filter selector" (at 60.96 175.8184 0)
+      (effects (font (size 1.27 1.27)) (justify left bottom))
+    )
+    (property "Sheetfile" "filter_selector.kicad_sch" (at 60.96 184.7346 0)
+      (effects (font (size 1.27 1.27)) (justify left top))
+    )
+    (pin "S2" input (at 60.96 181.61 180)
+      (effects (font (size 1.27 1.27)) (justify left))
+    )
+    (pin "S1" input (at 60.96 179.07 180)
+      (effects (font (size 1.27 1.27)) (justify left))
+    )
+    (pin "filtered" output (at 74.93 179.07 0)
+      (effects (font (size 1.27 1.27)) (justify right))
+    )
+    (instances
+      (project "main"
+        (path "/cb08c644-d155-44e5-86e1-31645eace055" (page "9"))
+      )
     )
   )
@@
       )
     )
-  )
-  (sheet (at 104.14 173.99) (size 25.4 12.7) (fields_autoplaced)
-    (stroke (width 0.1524) (type solid))
-    (fill (color 0 0 0 0.0000))
-    (property "Sheetname" "Filters" (at 104.14 173.2784 0)
-      (effects (font (size 1.27 1.27)) (justify left bottom))
-    )
-    (property "Sheetfile" "filters.kicad_sch" (at 104.14 187.2746 0)
-      (effects (font (size 1.27 1.27)) (justify left top))
-    )
-    (pin "BPF2_OUT" output (at 129.54 179.07 0)
-      (effects (font (size 1.27 1.27)) (justify right))
-    )
-    (pin "BPF1_IN" input (at 104.14 176.53 180)
-      (effects (font (size 1.27 1.27)) (justify left))
-    )
-    (pin "BPF2_IN" input (at 104.14 179.07 180)
-      (effects (font (size 1.27 1.27)) (justify left))
-    )
-    (pin "BPF1_OUT" output (at 129.54 176.53 0)
-      (effects (font (size 1.27 1.27)) (justify right))
-    )
-    (pin "BPF3_IN" input (at 104.14 181.61 180)
-      (effects (font (size 1.27 1.27)) (justify left))
-    )
-    (pin "BPF3_OUT" output (at 129.54 181.61 0)
-      (effects (font (size 1.27 1.27)) (justify right))
-    )
-    (pin "BPF4_IN" input (at 104.14 184.15 180)
-      (effects (font (size 1.27 1.27)) (justify left))
-    )
-    (pin "BPF4_OUT" output (at 129.54 184.15 0)
-      (effects (font (size 1.27 1.27)) (justify right))
-    )
-    (instances
-      (project "main"
-        (path "/cb08c644-d155-44e5-86e1-31645eace055" (page "8"))
-      )
-    )

Commit message: Modulator and RF processing circuits added
Other:
- removed sheet Filter selector
- added sheet RF Processing (rf_processing.kicad_sch)
Changed lines of the file:
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@@
-    )
-  )
-  (sheet (at 60.96 176.53) (size 13.97 7.62) (fields_autoplaced)
-    (stroke (width 0.1524) (type solid))
-    (fill (color 0 0 0 0.0000))
-    (property "Sheetname" "Filter selector" (at 60.96 175.8184 0)
-      (effects (font (size 1.27 1.27)) (justify left bottom))
-    )
-    (property "Sheetfile" "filter_selector.kicad_sch" (at 60.96 184.7346 0)
-      (effects (font (size 1.27 1.27)) (justify left top))
-    )
-    (pin "S2" input (at 60.96 181.61 180)
-      (effects (font (size 1.27 1.27)) (justify left))
-    )
-    (pin "S1" input (at 60.96 179.07 180)
-      (effects (font (size 1.27 1.27)) (justify left))
-    )
-    (pin "filtered" output (at 74.93 179.07 0)
-      (effects (font (size 1.27 1.27)) (justify right))
-    )
-    (instances
-      (project "main"
-        (path "/cb08c644-d155-44e5-86e1-31645eace055" (page "9"))
-      )
     )
   )
@@
       )
     )
+  )
+  (sheet (at 123.19 179.07) (size 21.59 11.43) (fields_autoplaced)
+    (stroke (width 0.1524) (type solid))
+    (fill (color 0 0 0 0.0000))
+    (property "Sheetname" "RF Processing" (at 123.19 178.3584 0)
+      (effects (font (size 1.27 1.27)) (justify left bottom))
+    )
+    (property "Sheetfile" "rf_processing.kicad_sch" (at 123.19 191.0846 0)
+      (effects (font (size 1.27 1.27)) (justify left top))
+    )
+    (instances
+      (project "main"
+        (path "/cb08c644-d155-44e5-86e1-31645eace055" (page "10"))
+      )
+    )

Commit message: mixer connected, MCU wiring changed
Connections:
- net RF Processing/filter_selector2: now reaches U1.11 (PA1)
- net RF Processing/QSD_EN: now reaches U1.14 (PA4)
- net QSE_EN: now reaches U1.42 (PB6)
- net filter_sel1: now reaches U1.43 (PB7)
- no-connect marks 11 -> 10
Other:
- sheet RF Processing ports: added L+, L-, QSD_EN, QSE_EN, R+, R-, SDR_I, SDR_Q, filter_selector1, filter_selector2, phase0, phase1; removed none
- moved on the sheet: C2, C3, L1, U4

Commit message: TODO text removed
Other:
- note removed: "TODO: PA0 is WKUP pin and will be used in the future, leave it unused"
Changed lines of the file:
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@@
-    (effects (font (size 1.27 1.27)) (justify left bottom))
-  )
-  (text "TODO: PA0 is WKUP pin and will be used in the\nfuture, leave it unused"
-    (at 95.25 20.32 0)
     (effects (font (size 1.27 1.27)) (justify left bottom))
   )
@@
     (effects (font (size 1.27 1.27)) (justify right bottom))
   )
-  (label "MISO" (at 129.54 73.66 0)
+  (label "MISO" (at 129.54 73.66 0) (fields_autoplaced)
     (effects (font (size 1.27 1.27)) (justify left bottom))
   )
-  (label "sda" (at 175.26 138.43 180)
+  (label "sda" (at 175.26 138.43 180) (fields_autoplaced)
     (effects (font (size 1.27 1.27)) (justify right bottom))
   )
@@
     (effects (font (size 1.27 1.27)) (justify right bottom))
   )
-  (label "MOSI" (at 129.54 76.2 0)
+  (label "MOSI" (at 129.54 76.2 0) (fields_autoplaced)
     (effects (font (size 1.27 1.27)) (justify left bottom))
   )
@@
     (effects (font (size 1.27 1.27)) (justify right bottom))
   )
-  (label "scl" (at 175.26 140.97 180)
+  (label "scl" (at 175.26 140.97 180) (fields_autoplaced)
     (effects (font (size 1.27 1.27)) (justify right bottom))
   )
@@
     (effects (font (size 1.27 1.27)) (justify right bottom))
   )
-  (label "MISO" (at 252.73 81.28 180)
+  (label "MISO" (at 252.73 81.28 180) (fields_autoplaced)
     (effects (font (size 1.27 1.27)) (justify right bottom))
   )
@@
     (effects (font (size 1.27 1.27)) (justify right bottom))
   )
-  (label "MOSI" (at 252.73 83.82 180)
+  (label "MOSI" (at 252.73 83.82 180) (fields_autoplaced)
     (effects (font (size 1.27 1.27)) (justify right bottom))
   )
-  (label "mck" (at 129.54 66.04 0)
+  (label "mck" (at 129.54 66.04 0) (fields_autoplaced)
     (effects (font (size 1.27 1.27)) (justify left bottom))
   )
@@
     (effects (font (size 1.27 1.27)) (justify right bottom))
   )
-  (label "SCLK" (at 252.73 86.36 180)
+  (label "SCLK" (at 252.73 86.36 180) (fields_autoplaced)
     (effects (font (size 1.27 1.27)) (justify right bottom))
   )
@@
     (effects (font (size 1.27 1.27)) (justify right bottom))
   )
-  (label "SCLK" (at 129.54 71.12 0)
+  (label "SCLK" (at 129.54 71.12 0) (fields_autoplaced)
     (effects (font (size 1.27 1.27)) (justify left bottom))
   )
