File: main/main.kicad_sch (KiCad schematic)
At the start: 21 parts, among them J6 Conn_01x05_Pin, SW6 RotaryEncoder, U1 STM32F411CEU6, U100 AP1117-33, U4 AT24CS64-SSHM, Y1 32768kHz

Commit message: Revire MCU to add swr_fwd and swr_rvs signals
Connections:
- net RF Processing/QSD_EN is gone; now on net Keyboard/keyb: U1.14 (PA4)
- net Keyboard/keyb: no longer U1.12 (PA2)
- net filter_sel1: now also U1.45 (PB8); no longer U1.43 (PB7)
- net LED: now reaches U1.10 (PA0)
- net filter_sel2: now reaches U1.46 (PB9)
- net RF Processing/filter_selector2 renamed RF Processing/swr_fwd
- new net QSD_EN: U1.43 (PB7)
- new net RF Processing/swr_rvs: U1.12 (PA2)
- no-connect marks 10 -> 8
Other:
- sheet RF Processing ports: added swr_fwd, swr_rvs; removed none
Changed lines of the file:
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@@
   (junction (at 195.58 143.51) (diameter 0) (color 0 0 0 0)
   )
-  (no_connect (at 96.52 109.22))
   (no_connect (at 252.73 107.95))
   (no_connect (at 252.73 100.33))
-  (no_connect (at 129.54 58.42))
+  (no_connect (at 135.255 58.42))
   (no_connect (at 252.73 110.49))
   (no_connect (at 252.73 102.87))
   (no_connect (at 96.52 71.12))
   (no_connect (at 252.73 105.41))
-  (no_connect (at 96.52 106.68))
   (no_connect (at 96.52 76.2))
   (bus_entry (at 67.31 114.3) (size -2.54 -2.54)
@@
     (stroke (width 0) (type default))
   )
+  (wire (pts (xy 136.525 55.245) (xy 136.525 60.96))
+    (stroke (width 0) (type default))
+  )
   (wire (pts (xy 226.06 49.53) (xy 226.06 68.58))
     (stroke (width 0) (type default))
   )
+  (wire (pts (xy 185.42 55.245) (xy 136.525 55.245))
+    (stroke (width 0) (type default))
+  )
   (wire (pts (xy 129.54 76.2) (xy 162.56 76.2))
     (stroke (width 0) (type default))
   )
-  (wire (pts (xy 139.065 60.96) (xy 139.065 63.5))
-    (stroke (width 0) (type default))
-  )
   (wire (pts (xy 114.3 143.51) (xy 114.3 138.43))
     (stroke (width 0) (type default))
@@
     (stroke (width 0) (type default))
   )
+  (wire (pts (xy 231.14 76.2) (xy 231.14 44.45))
+    (stroke (width 0) (type default))
+  )
   (bus (pts (xy 157.48 127) (xy 157.48 154.94))
     (stroke (width 0) (type default))
@@
     (stroke (width 0) (type default))
   )
+  (wire (pts (xy 129.54 63.5) (xy 137.795 63.5))
+    (stroke (width 0) (type default))
+  )
   (bus (pts (xy 157.48 110.49) (xy 175.26 110.49))
     (stroke (width 0) (type default))
   )
-  (wire (pts (xy 137.16 60.96) (xy 137.16 55.245))
-    (stroke (width 0) (type default))
-  )
-  (wire (pts (xy 137.16 55.245) (xy 193.04 55.245))
-    (stroke (width 0) (type default))
-  )
   (wire (pts (xy 129.54 73.66) (xy 162.56 73.66))
     (stroke (width 0) (type default))
@@
     (stroke (width 0) (type default))
   )
-  (wire (pts (xy 140.335 60.96) (xy 139.065 60.96))
+  (wire (pts (xy 141.605 65.405) (xy 140.335 65.405))
     (stroke (width 0) (type default))
   )
@@
     (stroke (width 0) (type default))
   )
-  (wire (pts (xy 129.54 68.58) (xy 195.58 68.58))
-    (stroke (width 0) (type default))
-  )
   (bus (pts (xy 168.91 135.89) (xy 168.91 127))
     (stroke (width 0) (type default))
@@
     (stroke (width 0) (type default))
   )
-  (wire (pts (xy 129.54 63.5) (xy 139.065 63.5))
-    (stroke (width 0) (type default))
-  )
   (wire (pts (xy 91.44 96.52) (xy 96.52 96.52))
     (stroke (width 0) (type default))
@@
     (stroke (width 0) (type default))
   )
-  (wire (pts (xy 158.75 80.01) (xy 158.75 66.04))
+  (wire (pts (xy 158.75 59.69) (xy 158.75 80.01))
     (stroke (width 0) (type default))
   )
@@
     (stroke (width 0) (type default))
   )
+  (wire (pts (xy 139.065 59.69) (xy 158.75 59.69))
+    (stroke (width 0) (type default))
+  )
   (wire (pts (xy 87.63 121.92) (xy 96.52 121.92))
     (stroke (width 0) (type default))
@@
     (stroke (width 0) (type default))
   )
+  (wire (pts (xy 129.54 58.42) (xy 135.255 58.42))
+    (stroke (width 0) (type default))
+  )
   (wire (pts (xy 111.76 50.8) (xy 111.76 53.34))
     (stroke (width 0) (type default))
@@
     (stroke (width 0) (type default))
   )
+  (wire (pts (xy 229.87 78.74) (xy 223.52 78.74))
+    (stroke (width 0) (type default))
+  )
   (wire (pts (xy 195.58 148.59) (xy 185.42 148.59))
     (stroke (width 0) (type default))
@@
     (stroke (width 0) (type default))
   )
+  (wire (pts (xy 139.065 66.04) (xy 139.065 59.69))
+    (stroke (width 0) (type default))
+  )
   (wire (pts (xy 242.57 83.82) (xy 252.73 83.82))
     (stroke (width 0) (type default))
@@
     (stroke (width 0) (type default))
   )
-  (wire (pts (xy 193.04 62.23) (xy 204.47 62.23))
-    (stroke (width 0) (type default))
-  )
   (bus (pts (xy 85.09 116.84) (xy 85.09 119.38))
     (stroke (width 0) (type default))
@@
     (stroke (width 0) (type default))
   )
+  (wire (pts (xy 137.795 63.5) (xy 137.795 57.15))
+    (stroke (width 0) (type default))
+  )
   (wire (pts (xy 200.66 113.03) (xy 200.66 91.44))
     (stroke (width 0) (type default))
   )
+  (wire (pts (xy 139.065 66.04) (xy 129.54 66.04))
+    (stroke (width 0) (type default))
+  )
+  (wire (pts (xy 140.335 65.405) (xy 140.335 68.58))
+    (stroke (width 0) (type default))
+  )
   (bus (pts (xy 78.74 151.13) (xy 161.29 151.13))
     (stroke (width 0) (type default))
@@
     (stroke (width 0) (type default))
   )
-  (wire (pts (xy 193.04 55.245) (xy 193.04 62.23))
+  (wire (pts (xy 231.14 44.45) (xy 185.42 44.45))
     (stroke (width 0) (type default))
   )
@@
     (stroke (width 0) (type default))
   )
+  (wire (pts (xy 129.54 68.58) (xy 140.335 68.58))
+    (stroke (width 0) (type default))
+  )
   (wire (pts (xy 114.3 50.8) (xy 114.3 53.34))
     (stroke (width 0) (type default))
@@
     (stroke (width 0) (type default))
   )
-  (wire (pts (xy 129.54 60.96) (xy 137.16 60.96))
+  (wire (pts (xy 136.525 60.96) (xy 129.54 60.96))
     (stroke (width 0) (type default))
   )
@@
     (stroke (width 0) (type default))
   )
+  (wire (pts (xy 223.52 76.2) (xy 231.14 76.2))
+    (stroke (width 0) (type default))
+  )
   (wire (pts (xy 87.63 99.06) (xy 96.52 99.06))
     (stroke (width 0) (type default))
@@
     (stroke (width 0) (type default))
   )
+  (wire (pts (xy 185.42 44.45) (xy 185.42 55.245))
+    (stroke (width 0) (type default))
+  )
   (wire (pts (xy 72.39 68.58) (xy 63.5 68.58))
     (stroke (width 0) (type default))
   )
+  (wire (pts (xy 186.69 57.15) (xy 186.69 45.72))
+    (stroke (width 0) (type default))
+  )
   (wire (pts (xy 187.96 46.99) (xy 228.6 46.99))
     (stroke (width 0) (type default))
@@
     (stroke (width 0) (type default))
   )
+  (wire (pts (xy 137.795 57.15) (xy 186.69 57.15))
+    (stroke (width 0) (type default))
+  )
+  (wire (pts (xy 229.87 45.72) (xy 229.87 78.74))
+    (stroke (width 0) (type default))
+  )
   (wire (pts (xy 195.58 143.51) (xy 195.58 148.59))
     (stroke (width 0) (type default))
   )
-  (wire (pts (xy 158.75 66.04) (xy 129.54 66.04))
-    (stroke (width 0) (type default))
-  )
   (wire (pts (xy 190.5 49.53) (xy 226.06 49.53))
     (stroke (width 0) (type default))
@@
     (stroke (width 0) (type default))
   )
-  (wire (pts (xy 195.58 71.12) (xy 204.47 71.12))
-    (stroke (width 0) (type default))
-  )
-  (wire (pts (xy 195.58 68.58) (xy 195.58 71.12))
-    (stroke (width 0) (type default))
-  )
   (bus (pts (xy 240.03 78.74) (xy 240.03 81.28))
     (stroke (width 0) (type default))
@@
   )
   (wire (pts (xy 87.63 116.84) (xy 96.52 116.84))
+    (stroke (width 0) (type default))
+  )
+  (wire (pts (xy 186.69 45.72) (xy 229.87 45.72))
     (stroke (width 0) (type default))
   )
@@
     (effects (font (size 1.27 1.27)) (justify left bottom))
   )
+  (label "QSD_EN" (at 96.52 104.14 180) (fields_autoplaced)
+    (effects (font (size 1.27 1.27)) (justify right bottom))
+  )
   (label "displ_RESET" (at 96.52 91.44 180) (fields_autoplaced)
     (effects (font (size 1.27 1.27)) (justify right bottom))
@@
     (effects (font (size 1.27 1.27)) (justify left bottom))
   )
+  (label "QSD_EN" (at 204.47 71.12 180) (fields_autoplaced)
+    (effects (font (size 1.27 1.27)) (justify right bottom))
+  )
   (label "scl" (at 64.77 110.49 0) (fields_autoplaced)
     (effects (font (size 1.27 1.27)) (justify left bottom))
@@
     (effects (font (size 1.27 1.27)) (justify right bottom))
   )
-  (label "filter_sel1" (at 96.52 104.14 180) (fields_autoplaced)
+  (label "filter_sel1" (at 96.52 106.68 180) (fields_autoplaced)
     (effects (font (size 1.27 1.27)) (justify right bottom))
   )
@@
     (effects (font (size 1.27 1.27)) (justify right bottom))
   )
+  (label "LED" (at 130.175 58.42 0) (fields_autoplaced)
+    (effects (font (size 1.27 1.27)) (justify left bottom))
+  )
   (label "MOSI" (at 252.73 83.82 180) (fields_autoplaced)
     (effects (font (size 1.27 1.27)) (justify right bottom))
@@
     (effects (font (size 1.27 1.27)) (justify right bottom))
   )
+  (label "filter_sel2" (at 204.47 62.23 180) (fields_autoplaced)
+    (effects (font (size 1.27 1.27)) (justify right bottom))
+  )
   (label "ws" (at 96.52 114.3 180) (fields_autoplaced)
+    (effects (font (size 1.27 1.27)) (justify right bottom))
+  )
+  (label "filter_sel2" (at 96.52 109.22 180) (fields_autoplaced)
     (effects (font (size 1.27 1.27)) (justify right bottom))
   )
@@
     )
   )
-  (sheet (at 140.335 58.42) (size 13.97 5.08) (fields_autoplaced)
+  (sheet (at 141.605 62.865) (size 13.97 5.08) (fields_autoplaced)
     (stroke (width 0.1524) (type solid))
     (fill (color 0 0 0 0.0000))
-    (property "Sheetname" "Keyboard" (at 140.335 57.7084 0)
+    (property "Sheetname" "Keyboard" (at 141.605 62.1534 0)
       (effects (font (size 1.27 1.27)) (justify left bottom))
     )
-    (property "Sheetfile" "keyboard.kicad_sch" (at 140.335 64.0846 0)
+    (property "Sheetfile" "keyboard.kicad_sch" (at 141.605 68.5296 0)
       (effects (font (size 1.27 1.27)) (justify left top))
     )
-    (pin "keyb" output (at 140.335 60.96 180)
+    (pin "keyb" output (at 141.605 65.405 180)
       (effects (font (size 1.27 1.27)) (justify left))
     )
@@
       (effects (font (size 1.27 1.27)) (justify left))
     )
-    (instances
+    (pin "swr_fwd" output (at 223.52 76.2 0)
+      (effects (font (size 1.27 1.27)) (justify right))
+    )
+    (pin "swr_rvs" output (at 223.52 78.74 0)
+      (effects (font (size 1.27 1.27)) (justify right))
+    )
+    (instances
