File: main/main.kicad_sch (KiCad schematic)
At the start: 23 parts, among them J6 Conn_01x05_Pin, SW6 RotaryEncoder, U1 STM32F411CEU6, U100 AP1117-33, U4 AT24CS64-SSHM, Y1 32768kHz

Commit message: FIXME comment added
Other:
- note added: "FIXME: использовать инвертор чтобы избежать одновременного включения"
Changed lines of the file:
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@@
     (stroke (width 0) (type default))
+  )
+  (arc (start 205.1048 69.85) (mid 199.3183 55.88) (end 205.1048 41.91)
+    (stroke (width 0) (type default))
+    (fill (type none))
   )
   (text "TODO: rewire to SWD standard" (at 41.91 44.45 0)
     (effects (font (size 1.27 1.27)) (justify left bottom))
   )
+  (text "FIXME: использовать инвертор чтобы\nизбежать одновременного включения"
+    (at 200.025 41.275 0)
+    (effects (font (size 1.27 1.27)) (justify left bottom))
+  )

Commit message: tkey moved to main
Parts:
- added J1: AudioJack5, symbol Connector_Audio:AudioJack5
Connections:
- net GND: now also J1.R3, J1.S, J1.T
- net Telegraph key/KEY_DAH renamed KEY_DAH
- net KEY_DAH: now also J1.R2
- net Telegraph key/KEY_DIT renamed KEY_DIT
- net KEY_DIT: now also J1.R1
Other:
- removed sheet Telegraph key
- moved on the sheet: SW6

Commit message: Key name fixed, PDF updated
Parts:
- J1: purpose Headset -> Telegraph key
Changed lines of the file:
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@@
       (effects (font (size 1.27 1.27)) hide)
     )
-    (property "purpose" "Headset" (at 267.335 160.655 0)
+    (property "purpose" "Telegraph key" (at 267.335 160.655 0)
       (effects (font (size 1.27 1.27)))
     )

Commit message: EEPROM TODO added
Other:
- note added: "TODO: Переподключить EEPROM как на Black Pill Заменить на FRAM"
Changed lines of the file:
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@@
+    (effects (font (size 1.27 1.27)) (justify left bottom))
+  )
+  (text "TODO:\nПереподключить EEPROM как на Black Pill\nЗаменить на FRAM"
+    (at 164.465 159.385 0)
     (effects (font (size 1.27 1.27)) (justify left bottom))
   )

Commit message: Key jack changed
Parts:
- removed J1: AudioJack5, symbol Connector_Audio:AudioJack5
- added J5: Telegraph key, Connector_Audio:Jack_3.5mm_CUI_SJ1-3525N_Horizontal, symbol Connector_Audio:AudioJack3_SwitchTR
Connections:
- net GND: now also J5.S
- net KEY_DAH: now also J5.R, J5.RN
- net KEY_DIT: now also J5.T, J5.TN
Changed lines of the file:
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@@
   (junction (at 128.27 38.1) (diameter 0) (color 0 0 0 0)
-  )
-  (junction (at 255.905 151.765) (diameter 0) (color 0 0 0 0)
   )
   (junction (at 162.56 57.15) (diameter 0) (color 0 0 0 0)
@@
     (stroke (width 0) (type default))
   )
+  (wire (pts (xy 255.905 146.685) (xy 258.445 146.685))
+    (stroke (width 0) (type default))
+  )
   (wire (pts (xy 187.96 115.57) (xy 199.39 115.57))
     (stroke (width 0) (type default))
@@
     (stroke (width 0) (type default))
   )
+  (wire (pts (xy 255.905 144.145) (xy 258.445 144.145))
+    (stroke (width 0) (type default))
+  )
   (bus (pts (xy 168.91 135.89) (xy 168.91 127))
     (stroke (width 0) (type default))
@@
     (stroke (width 0) (type default))
   )
+  (wire (pts (xy 255.905 146.685) (xy 255.905 149.225))
+    (stroke (width 0) (type default))
+  )
   (wire (pts (xy 87.63 121.92) (xy 96.52 121.92))
     (stroke (width 0) (type default))
@@
     (stroke (width 0) (type default))
   )
+  (wire (pts (xy 255.905 141.605) (xy 258.445 141.605))
+    (stroke (width 0) (type default))
+  )
   (wire (pts (xy 54.61 77.47) (xy 54.61 78.74))
     (stroke (width 0) (type default))
@@
     (stroke (width 0) (type default))
   )
-  (wire (pts (xy 255.905 135.255) (xy 255.905 141.605))
-    (stroke (width 0) (type default))
-  )
   (wire (pts (xy 109.22 50.8) (xy 109.22 53.34))
     (stroke (width 0) (type default))
@@
     (stroke (width 0) (type default))
   )
-  (wire (pts (xy 255.905 149.225) (xy 255.905 151.765))
-    (stroke (width 0) (type default))
-  )
   (bus (pts (xy 85.09 116.84) (xy 85.09 119.38))
     (stroke (width 0) (type default))
@@
     (stroke (width 0) (type default))
   )
+  (wire (pts (xy 255.905 141.605) (xy 255.905 144.145))
+    (stroke (width 0) (type default))
+  )
   (wire (pts (xy 119.38 26.67) (xy 119.38 29.21))
     (stroke (width 0) (type default))
@@
   )
   (wire (pts (xy 135.89 38.1) (xy 139.7 38.1))
-    (stroke (width 0) (type default))
-  )
-  (wire (pts (xy 255.905 141.605) (xy 258.445 141.605))
     (stroke (width 0) (type default))
   )
@@
     (effects (font (size 1.27 1.27)) (justify right bottom))
   )
-  (label "KEY_DIT" (at 258.445 144.145 180) (fields_autoplaced)
+  (label "KEY_DIT" (at 255.905 143.51 180) (fields_autoplaced)
     (effects (font (size 1.27 1.27)) (justify right bottom))
   )
@@
     (effects (font (size 1.27 1.27)) (justify left bottom))
   )
-  (label "KEY_DAH" (at 258.445 146.685 180) (fields_autoplaced)
+  (label "KEY_DAH" (at 255.905 148.59 180) (fields_autoplaced)
     (effects (font (size 1.27 1.27)) (justify right bottom))
   )
@@
     )
   )
-  (symbol (lib_id "power:GND") (at 255.905 135.255 270) (unit 1)
-    (in_bom yes) (on_board yes) (dnp no) (fields_autoplaced)
-    (property "Reference" "#PWR046" (at 249.555 135.255 0)
-      (effects (font (size 1.27 1.27)) hide)
-    )
-    (property "Value" "GND" (at 252.095 135.255 90)
-      (effects (font (size 1.27 1.27)) (justify right))
-    )
-    (property "Footprint" "" (at 255.905 135.255 0)
-      (effects (font (size 1.27 1.27)) hide)
-    )
-    (property "Datasheet" "" (at 255.905 135.255 0)
-      (effects (font (size 1.27 1.27)) hide)
-    )
-    (pin "1")
-    (instances
-      (project "main"
-        (path "/cb08c644-d155-44e5-86e1-31645eace055"
-          (reference "#PWR046") (unit 1)
-        )
-      )
-    )
-  )
   (symbol (lib_id "Device:R") (at 76.2 57.15 90) (unit 1)
     (in_bom yes) (on_board yes) (dnp no) (fields_autoplaced)
@@
     )
   )
+  (symbol (lib_id "Connector_Audio:AudioJack3_SwitchTR") (at 263.525 149.225 180) (unit 1)
+    (in_bom yes) (on_board yes) (dnp no) (fields_autoplaced)
+    (property "Reference" "J5" (at 271.78 144.78 0)
+      (effects (font (size 1.27 1.27)) (justify right))
+    )
+    (property "Value" "Telegraph key" (at 271.78 147.32 0)
+      (effects (font (size 1.27 1.27)) (justify right))
+    )
+    (property "Footprint" "Connector_Audio:Jack_3.5mm_CUI_SJ1-3525N_Horizontal" (at 263.525 149.225 0)
+      (effects (font (size 1.27 1.27)) hide)
+    )
+    (property "Datasheet" "~" (at 263.525 149.225 0)
+      (effects (font (size 1.27 1.27)) hide)
+    )
+    (pin "TN")
+    (pin "S")
+    (pin "RN")
+    (pin "R")
+    (pin "T")
+    (instances
+      (project "main"
+        (path "/cb08c644-d155-44e5-86e1-31645eace055"
+          (reference "J5") (unit 1)
+        )
+      )
+    )
+  )
   (symbol (lib_id "power:GND") (at 262.89 119.38 0) (unit 1)
     (in_bom yes) (on_board yes) (dnp no) (fields_autoplaced)
@@
         )
       )
-    )
-  )
-  (symbol (lib_id "Connector_Audio:AudioJack5") (at 263.525 146.685 180) (unit 1)
-    (in_bom yes) (on_board yes) (dnp no)
-    (property "Reference" "J1" (at 267.335 158.115 0)
-      (effects (font (size 1.27 1.27)))
-    )
-    (property "Value" "AudioJack5" (at 267.335 155.575 0)
-      (effects (font (size 1.27 1.27)))
-    )
-    (property "Footprint" "" (at 263.525 146.685 0)
-      (effects (font (size 1.27 1.27)) hide)
-    )
-    (property "Datasheet" "~" (at 263.525 146.685 0)
-      (effects (font (size 1.27 1.27)) hide)
-    )
-    (property "purpose" "Telegraph key" (at 267.335 160.655 0)
-      (effects (font (size 1.27 1.27)))
-    )
-    (pin "R3")
-    (pin "S")
-    (pin "R1")
-    (pin "T")
-    (pin "R2")
-    (instances
-      (project "main"
-        (path "/cb08c644-d155-44e5-86e1-31645eace055/e511764a-2dd7-4601-8d00-331d6dbffa9f"
-          (reference "J1") (unit 1)
-        )
-        (path "/cb08c644-d155-44e5-86e1-31645eace055"
-          (reference "J5") (unit 1)
-        )
-      )

Commit message: bridget jumpers added to key
Parts:
- added JP1, JP2: SolderJumper_2_Bridged, symbol Jumper:SolderJumper_2_Bridged
Connections:
- net KEY_DAH: now also JP2.1 (A); no longer J5.RN
- net KEY_DIT: now also JP1.1 (A); no longer J5.TN
- new net: J5.RN, JP2.2 (B)
- new net: J5.TN, JP1.2 (B)
Other:
- moved on the sheet: J5
Changed lines of the file:
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@@
   (junction (at 109.22 50.8) (diameter 0) (color 0 0 0 0)
   )
+  (junction (at 245.11 148.59) (diameter 0) (color 0 0 0 0)
+  )
   (junction (at 157.48 110.49) (diameter 0) (color 0 0 0 0)
   )
@@
   )
   (junction (at 162.56 57.15) (diameter 0) (color 0 0 0 0)
+  )
+  (junction (at 245.11 136.525) (diameter 0) (color 0 0 0 0)
   )
   (junction (at 114.3 50.8) (diameter 0) (color 0 0 0 0)
@@
     (stroke (width 0) (type default))
   )
-  (wire (pts (xy 255.905 151.765) (xy 255.905 155.575))
+  (wire (pts (xy 253.365 151.13) (xy 253.365 153.67))
     (stroke (width 0) (type default))
   )
@@
     (stroke (width 0) (type default))
   )
+  (wire (pts (xy 245.11 146.05) (xy 245.11 148.59))
+    (stroke (width 0) (type default))
+  )
   (wire (pts (xy 168.91 60.96) (xy 187.96 60.96))
     (stroke (width 0) (type default))
@@
     (stroke (width 0) (type default))
   )
-  (wire (pts (xy 255.905 146.685) (xy 258.445 146.685))
+  (wire (pts (xy 245.11 146.05) (xy 246.38 146.05))
     (stroke (width 0) (type default))
   )
@@
     (stroke (width 0) (type default))
   )
-  (wire (pts (xy 255.905 144.145) (xy 258.445 144.145))
+  (wire (pts (xy 253.365 143.51) (xy 253.365 136.525))
+    (stroke (width 0) (type default))
+  )
+  (wire (pts (xy 253.365 143.51) (xy 255.905 143.51))
     (stroke (width 0) (type default))
   )
@@
     (stroke (width 0) (type default))
   )
-  (wire (pts (xy 255.905 146.685) (xy 255.905 149.225))
-    (stroke (width 0) (type default))
-  )
   (wire (pts (xy 87.63 121.92) (xy 96.52 121.92))
     (stroke (width 0) (type default))
@@
     (stroke (width 0) (type default))
   )
+  (wire (pts (xy 255.27 140.97) (xy 255.905 140.97))
+    (stroke (width 0) (type default))
+  )
   (wire (pts (xy 129.54 58.42) (xy 135.255 58.42))
     (stroke (width 0) (type default))
@@
     (stroke (width 0) (type default))
   )
-  (wire (pts (xy 255.905 141.605) (xy 258.445 141.605))
+  (wire (pts (xy 245.11 133.35) (xy 245.745 133.35))
     (stroke (width 0) (type default))
   )
@@
     (stroke (width 0) (type default))
   )
-  (wire (pts (xy 255.905 141.605) (xy 255.905 144.145))
+  (wire (pts (xy 245.11 133.35) (xy 245.11 136.525))
     (stroke (width 0) (type default))
   )
@@
     (stroke (width 0) (type default))
   )
+  (wire (pts (xy 255.27 133.35) (xy 255.27 140.97))
+    (stroke (width 0) (type default))
+  )
   (wire (pts (xy 87.63 114.3) (xy 96.52 114.3))
     (stroke (width 0) (type default))
@@
     (stroke (width 0) (type default))
   )
+  (wire (pts (xy 253.365 133.35) (xy 255.27 133.35))
+    (stroke (width 0) (type default))
+  )
   (wire (pts (xy 185.42 44.45) (xy 185.42 55.245))
     (stroke (width 0) (type default))
@@
     (stroke (width 0) (type default))
   )
+  (wire (pts (xy 243.205 136.525) (xy 245.11 136.525))
+    (stroke (width 0) (type default))
+  )
   (wire (pts (xy 194.31 76.2) (xy 204.47 76.2))
     (stroke (width 0) (type default))
@@
     (stroke (width 0) (type default))
   )
+  (wire (pts (xy 243.205 148.59) (xy 245.11 148.59))
+    (stroke (width 0) (type default))
+  )
   (wire (pts (xy 54.61 88.9) (xy 54.61 87.63))
     (stroke (width 0) (type default))
@@
     (stroke (width 0) (type default))
   )
-  (wire (pts (xy 258.445 149.225) (xy 255.905 149.225))
+  (wire (pts (xy 255.905 148.59) (xy 245.11 148.59))
     (stroke (width 0) (type default))
   )
@@
     (stroke (width 0) (type default))
   )
-  (wire (pts (xy 255.905 151.765) (xy 258.445 151.765))
+  (wire (pts (xy 253.365 151.13) (xy 255.905 151.13))
+    (stroke (width 0) (type default))
+  )
+  (wire (pts (xy 253.365 136.525) (xy 245.11 136.525))
+    (stroke (width 0) (type default))
+  )
+  (wire (pts (xy 254 146.05) (xy 255.905 146.05))
     (stroke (width 0) (type default))
   )
@@
     (effects (font (size 1.27 1.27)) (justify right bottom))
   )
-  (label "KEY_DIT" (at 255.905 143.51 180) (fields_autoplaced)
+  (label "KEY_DIT" (at 243.205 136.525 180) (fields_autoplaced)
     (effects (font (size 1.27 1.27)) (justify right bottom))
   )
@@
     (effects (font (size 1.27 1.27)) (justify left bottom))
   )
-  (label "KEY_DAH" (at 255.905 148.59 180) (fields_autoplaced)
+  (label "KEY_DAH" (at 243.205 148.59 180) (fields_autoplaced)
     (effects (font (size 1.27 1.27)) (justify right bottom))
   )
@@
     )
   )
+  (symbol (lib_id "Jumper:SolderJumper_2_Bridged") (at 250.19 146.05 0) (unit 1)
+    (in_bom yes) (on_board yes) (dnp no) (fields_autoplaced)
+    (property "Reference" "JP2" (at 250.19 142.875 0)
+      (effects (font (size 1.27 1.27)))
+    )
+    (property "Value" "SolderJumper_2_Bridged" (at 250.19 142.875 0)
+      (effects (font (size 1.27 1.27)) hide)
+    )
+    (property "Footprint" "" (at 250.19 146.05 0)
+      (effects (font (size 1.27 1.27)) hide)
+    )
+    (property "Datasheet" "~" (at 250.19 146.05 0)
+      (effects (font (size 1.27 1.27)) hide)
+    )
+    (pin "1")
+    (pin "2")
+    (instances
+      (project "main"
+        (path "/cb08c644-d155-44e5-86e1-31645eace055"
+          (reference "JP2") (unit 1)
+        )
+      )
+    )
+  )
   (symbol (lib_id "power:+VDC") (at 262.89 68.58 0) (unit 1)
     (in_bom yes) (on_board yes) (dnp no) (fields_autoplaced)
@@
     )
   )
-  (symbol (lib_id "Connector_Audio:AudioJack3_SwitchTR") (at 263.525 149.225 180) (unit 1)
-    (in_bom yes) (on_board yes) (dnp no) (fields_autoplaced)
-    (property "Reference" "J5" (at 271.78 144.78 0)
+  (symbol (lib_id "Connector_Audio:AudioJack3_SwitchTR") (at 260.985 148.59 180) (unit 1)
+    (in_bom yes) (on_board yes) (dnp no) (fields_autoplaced)
+    (property "Reference" "J5" (at 268.605 144.145 0)
       (effects (font (size 1.27 1.27)) (justify right))
     )
-    (property "Value" "Telegraph key" (at 271.78 147.32 0)
+    (property "Value" "Telegraph key" (at 268.605 146.685 0)
       (effects (font (size 1.27 1.27)) (justify right))
     )
-    (property "Footprint" "Connector_Audio:Jack_3.5mm_CUI_SJ1-3525N_Horizontal" (at 263.525 149.225 0)
-      (effects (font (size 1.27 1.27)) hide)
-    )
-    (property "Datasheet" "~" (at 263.525 149.225 0)
+    (property "Footprint" "Connector_Audio:Jack_3.5mm_CUI_SJ1-3525N_Horizontal" (at 260.985 148.59 0)
+      (effects (font (size 1.27 1.27)) hide)
+    )
+    (property "Datasheet" "~" (at 260.985 148.59 0)
       (effects (font (size 1.27 1.27)) hide)
     )
@@
     )
   )
+  (symbol (lib_id "Jumper:SolderJumper_2_Bridged") (at 249.555 133.35 0) (unit 1)
+    (in_bom yes) (on_board yes) (dnp no) (fields_autoplaced)
+    (property "Reference" "JP1" (at 249.555 130.175 0)
+      (effects (font (size 1.27 1.27)))
+    )
+    (property "Value" "SolderJumper_2_Bridged" (at 249.555 130.175 0)
+      (effects (font (size 1.27 1.27)) hide)
+    )
+    (property "Footprint" "" (at 249.555 133.35 0)
+      (effects (font (size 1.27 1.27)) hide)
+    )
+    (property "Datasheet" "~" (at 249.555 133.35 0)
+      (effects (font (size 1.27 1.27)) hide)
+    )
+    (pin "1")
+    (pin "2")
+    (instances
+      (project "main"
+        (path "/cb08c644-d155-44e5-86e1-31645eace055"
+          (reference "JP1") (unit 1)
+        )
+      )
+    )
+  )
   (symbol (lib_id "power:GND") (at 190.5 36.83 0) (unit 1)
     (in_bom yes) (on_board yes) (dnp no) (fields_autoplaced)
@@
     )
   )
-  (symbol (lib_id "power:GND") (at 255.905 155.575 0) (unit 1)
-    (in_bom yes) (on_board yes) (dnp no) (fields_autoplaced)
-    (property "Reference" "#PWR047" (at 255.905 161.925 0)
-      (effects (font (size 1.27 1.27)) hide)
-    )
-    (property "Value" "GND" (at 255.905 160.655 0)
-      (effects (font (size 1.27 1.27)))
-    )
-    (property "Footprint" "" (at 255.905 155.575 0)
-      (effects (font (size 1.27 1.27)) hide)
-    )
-    (property "Datasheet" "" (at 255.905 155.575 0)
-      (effects (font (size 1.27 1.27)) hide)
-    )
+  (symbol (lib_id "power:GND") (at 253.365 153.67 0) (unit 1)
+    (in_bom yes) (on_board yes) (dnp no) (fields_autoplaced)
+    (property "Reference" "#PWR047" (at 253.365 160.02 0)
+      (effects (font (size 1.27 1.27)) hide)
+    )
+    (property "Value" "GND" (at 253.365 158.75 0)
+      (effects (font (size 1.27 1.27)))
+    )
+    (property "Footprint" "" (at 253.365 153.67 0)
+      (effects (font (size 1.27 1.27)) hide)
+    )
+    (property "Datasheet" "" (at 253.365 153.67 0)
+      (effects (font (size 1.27 1.27)) hide)
+    )

Commit message: Key connector changed, can be used as PTT
Parts:
- removed J5: Telegraph key, Connector_Audio:Jack_3.5mm_CUI_SJ1-3525N_Horizontal, symbol Connector_Audio:AudioJack3_SwitchTR
- removed JP1, JP2: SolderJumper_2_Bridged, symbol Jumper:SolderJumper_2_Bridged
- added J7: PTT / Key, symbol Connector_Audio:AudioJack4
- added JP1, JP9: Jumper_2_Bridged, symbol Jumper:Jumper_2_Bridged
- added JP2: Jumper_3_Open, symbol Jumper:Jumper_3_Open
Connections:
- net GND: now also JP9.1 (A)
- net KEY_DAH: now also JP2.2 (C)
- net KEY_DIT: now also JP1.1 (A)
- new net: J7.R1, JP2.1 (A)
- new net: J7.R2, JP2.3 (B)
- new net: J7.S, JP9.2 (B)
- new net: J7.T, JP1.2 (B)

Commit message: jumper changed to closed
Parts:
- removed JP2: Jumper_3_Open, symbol Jumper:Jumper_3_Open
- added JP2: Jumper_3_Bridged12, symbol Jumper:Jumper_3_Bridged12
Connections:
- net KEY_DAH: now also JP2.2 (C)
- net at J7.R1: now also JP2.1 (A)
- net at J7.R2: now also JP2.3 (B)
Changed lines of the file:
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@@
+    )
+  )
+  (symbol (lib_id "Jumper:Jumper_3_Bridged12") (at 248.285 147.32 270) (unit 1)
+    (in_bom yes) (on_board yes) (dnp no)
+    (property "Reference" "JP2" (at 242.57 150.495 90)
+      (effects (font (size 1.27 1.27)) (justify left))
+    )
+    (property "Value" "Jumper_3_Bridged12" (at 250.825 148.59 90)
+      (effects (font (size 1.27 1.27)) (justify left) hide)
+    )
+    (property "Footprint" "" (at 248.285 147.32 0)
+      (effects (font (size 1.27 1.27)) hide)
+    )
+    (property "Datasheet" "~" (at 248.285 147.32 0)
+      (effects (font (size 1.27 1.27)) hide)
+    )
+    (pin "2")
+    (pin "1")
+    (pin "3")
+    (instances
+      (project "main"
+        (path "/cb08c644-d155-44e5-86e1-31645eace055"
+          (reference "JP2") (unit 1)
+        )
+      )
     )
   )
@@
     )
   )
-  (symbol (lib_id "Jumper:Jumper_3_Open") (at 248.285 147.32 270) (unit 1)
-    (in_bom yes) (on_board yes) (dnp no)
-    (property "Reference" "JP2" (at 243.205 150.495 90)
-      (effects (font (size 1.27 1.27)) (justify left))
-    )
-    (property "Value" "Jumper_3_Open" (at 250.825 148.59 90)
-      (effects (font (size 1.27 1.27)) (justify left) hide)
-    )
-    (property "Footprint" "" (at 248.285 147.32 0)
-      (effects (font (size 1.27 1.27)) hide)
-    )
-    (property "Datasheet" "~" (at 248.285 147.32 0)
-      (effects (font (size 1.27 1.27)) hide)
-    )
-    (pin "3")
-    (pin "1")
-    (pin "2")
-    (instances
-      (project "main"
-        (path "/cb08c644-d155-44e5-86e1-31645eace055"
-          (reference "JP2") (unit 1)
-        )
-      )
-    )
-  )
   (symbol (lib_id "power:GND") (at 254 153.67 0) (unit 1)
     (in_bom yes) (on_board yes) (dnp no) (fields_autoplaced)
@@
   (symbol (lib_id "Jumper:Jumper_2_Bridged") (at 260.985 151.13 0) (unit 1)
     (in_bom yes) (on_board yes) (dnp no) (fields_autoplaced)
-    (property "Reference" "JP9" (at 260.985 146.05 0)
-      (effects (font (size 1.27 1.27)))
-    )
+    (property "Reference" "JP9" (at 260.985 153.67 0)
+      (effects (font (size 1.27 1.27)))
+    )
