File: main/mixer.kicad_sch (KiCad schematic)
At the start: 23 parts, among them U7 74CBTLV3253PW, U8 TS972IDT

Commit message: Mixer: numbers assigned
Parts:
- renumbered C58 to C40, U7 to U5
Changed lines of the file:
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@@
   (symbol (lib_id "Analog_Switch:SN74CBT3253") (at 98.425 85.725 0) (unit 1)
     (in_bom yes) (on_board yes) (dnp no) (fields_autoplaced)
-    (property "Reference" "U7" (at 98.0791 67.945 0)
-      (effects (font (size 1.27 1.27)) (justify right))
-    )
-    (property "Value" "74CBTLV3253PW" (at 98.0791 70.485 0)
-      (effects (font (size 1.27 1.27)) (justify right))
+    (property "Reference" "U5" (at 100.6191 68.58 0)
+      (effects (font (size 1.27 1.27)) (justify left))
+    )
+    (property "Value" "74CBTLV3253PW" (at 100.6191 71.12 0)
+      (effects (font (size 1.27 1.27)) (justify left))
     )
     (property "Footprint" "" (at 98.425 85.725 0)
@@
   (symbol (lib_id "Device:C") (at 203.2 81.915 0) (unit 1)
     (in_bom yes) (on_board yes) (dnp no) (fields_autoplaced)
-    (property "Reference" "C58" (at 206.375 80.645 0)
+    (property "Reference" "C40" (at 206.375 80.645 0)
       (effects (font (size 1.27 1.27)) (justify left))
     )
@@
   (symbol (lib_id "Device:C") (at 203.2 116.84 0) (unit 1)
     (in_bom yes) (on_board yes) (dnp no) (fields_autoplaced)
-    (property "Reference" "C58" (at 206.375 115.57 0)
+    (property "Reference" "C40" (at 206.375 115.57 0)
       (effects (font (size 1.27 1.27)) (justify left))
     )
@@
   (symbol (lib_id "power:+3.3V") (at 168.91 47.625 0) (mirror y) (unit 1)
     (in_bom yes) (on_board yes) (dnp no) (fields_autoplaced)
-    (property "Reference" "#PWR059" (at 168.91 51.435 0)
+    (property "Reference" "#PWR066" (at 168.91 51.435 0)
       (effects (font (size 1.27 1.27)) hide)
     )
@@
   (symbol (lib_id "Device:C") (at 133.985 138.43 0) (unit 1)
     (in_bom yes) (on_board yes) (dnp no)
-    (property "Reference" "C58" (at 132.715 132.715 0)
+    (property "Reference" "C40" (at 132.715 132.715 0)
       (effects (font (size 1.27 1.27)) (justify right))
     )
@@
   (symbol (lib_id "Device:C") (at 149.86 55.245 0) (mirror y) (unit 1)
     (in_bom yes) (on_board yes) (dnp no) (fields_autoplaced)
-    (property "Reference" "C58" (at 146.05 53.975 0)
+    (property "Reference" "C40" (at 146.05 53.975 0)
       (effects (font (size 1.27 1.27)) (justify left))
     )
@@
   (symbol (lib_id "Device:C") (at 143.51 138.43 0) (unit 1)
     (in_bom yes) (on_board yes) (dnp no)
-    (property "Reference" "C58" (at 142.24 132.715 0)
+    (property "Reference" "C40" (at 142.24 132.715 0)
       (effects (font (size 1.27 1.27)) (justify right))
     )
@@
   (symbol (lib_id "Device:C") (at 93.345 51.435 0) (mirror y) (unit 1)
     (in_bom yes) (on_board yes) (dnp no) (fields_autoplaced)
-    (property "Reference" "C58" (at 96.52 50.165 0)
-      (effects (font (size 1.27 1.27)) (justify right))
-    )
-    (property "Value" "100nF" (at 96.52 52.705 0)
-      (effects (font (size 1.27 1.27)) (justify right))
+    (property "Reference" "C40" (at 90.17 50.165 0)
+      (effects (font (size 1.27 1.27)) (justify left))
+    )
+    (property "Value" "100nF" (at 90.17 52.705 0)
+      (effects (font (size 1.27 1.27)) (justify left))
     )
     (property "Footprint" "" (at 92.3798 55.245 0)
@@
   (symbol (lib_id "power:+3.3V") (at 98.425 45.085 0) (mirror y) (unit 1)
     (in_bom yes) (on_board yes) (dnp no) (fields_autoplaced)
-    (property "Reference" "#PWR059" (at 98.425 48.895 0)
+    (property "Reference" "#PWR066" (at 98.425 48.895 0)
       (effects (font (size 1.27 1.27)) hide)
     )
@@
   (symbol (lib_id "Device:C") (at 114.935 138.43 0) (unit 1)
     (in_bom yes) (on_board yes) (dnp no)
-    (property "Reference" "C58" (at 113.665 132.715 0)
+    (property "Reference" "C40" (at 113.665 132.715 0)
       (effects (font (size 1.27 1.27)) (justify right))
     )
@@
   (symbol (lib_id "Device:C") (at 124.46 138.43 0) (unit 1)
     (in_bom yes) (on_board yes) (dnp no)
-    (property "Reference" "C58" (at 123.19 132.715 0)
+    (property "Reference" "C40" (at 123.19 132.715 0)
       (effects (font (size 1.27 1.27)) (justify right))
     )
@@
   (symbol (lib_id "Device:C") (at 163.195 55.245 0) (mirror y) (unit 1)
     (in_bom yes) (on_board yes) (dnp no) (fields_autoplaced)
-    (property "Reference" "C58" (at 159.385 53.975 0)
-      (effects (font (size 1.27 1.27)) (justify left))
-    )
+    (property "Reference" "C40" (at 159.385 53.975 0)
+      (effects (font (size 1.27 1.27)) (justify left))
+    )
