File: main/mixer.kicad_sch (KiCad schematic)
At the start: 23 parts, among them U5 74CBTLV3253PW, U8 TS972IDT

Commit message: mixer: comments, labels
Parts:
- added C40 (x2): 10u, symbol Device:C
Connections:
- net 180°: now reaches C40.1, U5.10 (2B1), U5.3 (1B4)
- net 180°: now also C40.1; no longer R22.1
- net 270°: now reaches C40.1, U5.11 (2B2), U5.4 (1B3)
- net 270°: now also C40.1; no longer R23.1
- net 90°: now reaches C40.1, R24.1, U5.12 (2B3), U5.5 (1B2)
- net 0°: now reaches C40.1, R21.1, U5.13 (2B4), U5.6 (1B1)
- new net: C40.2, R22.1
- new net: C40.2, R23.1
Other:
- note added: "Double Balanced "Tayloe" Detector (by Dan Tayloe)"
- note added: "TODO: C43 и C44 не нужны?"
- note added: "TODO: C57 не факт что нужен"
- note added: "TODO: R27 и R28 не нужны?"
- note added: "TODO: Не факт что эти резисторы здесь нужны Похоже, тут вылезла какая-то несогласованность входного сопротивления"
- note removed: "Based on "Tayloe detector" (by Dan Tayloe)"
- note removed: "TODO: Не факт что эти резисторы здесь нужны"
- moved on the sheet: C40
