File: main/mixer.kicad_sch (KiCad schematic)
At the start: 25 parts, among them U5 74CBTLV3253PW, U8 TS972IDT

Commit message: QSD_EN->RX_EN, QSE_EN->TX_EN, FIXME removed
Connections:
- net QSD_EN renamed ENABLE
Changed lines of the file:
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@@
     (effects (font (size 1.27 1.27)) (justify left))
   )
-  (hierarchical_label "QSD_EN" (shape input) (at 83.185 95.885 180) (fields_autoplaced)
+  (hierarchical_label "ENABLE" (shape input) (at 83.185 95.885 180) (fields_autoplaced)
     (effects (font (size 1.27 1.27)) (justify right))
   )
