File: main/filters.kicad_sch (KiCad schematic)
At the start: 24 parts

Commit message: Filters annotated
Parts:
- renumbered L13 to L10, L16 to L11, L15 to L13, L5 to L2, L8 to L3, L7 to L4, L10 to L5, L9 to L7, L11 to L8, L14 to L9
Changed lines of the file:
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@@
   (symbol (lib_id "Device:L") (at 184.15 83.82 90) (unit 1)
     (in_bom yes) (on_board yes) (dnp no) (fields_autoplaced)
-    (property "Reference" "L15" (at 184.15 78.74 90)
+    (property "Reference" "L13" (at 184.15 78.74 90)
       (effects (font (size 1.27 1.27)))
     )
@@
   (symbol (lib_id "Device:L") (at 66.04 48.26 90) (unit 1)
     (in_bom yes) (on_board yes) (dnp no) (fields_autoplaced)
-    (property "Reference" "L5" (at 66.04 43.18 90)
+    (property "Reference" "L2" (at 66.04 43.18 90)
       (effects (font (size 1.27 1.27)))
     )
@@
   (symbol (lib_id "Device:L") (at 149.86 83.82 90) (unit 1)
     (in_bom yes) (on_board yes) (dnp no) (fields_autoplaced)
-    (property "Reference" "L14" (at 149.86 78.74 90)
+    (property "Reference" "L9" (at 149.86 78.74 90)
       (effects (font (size 1.27 1.27)))
     )
@@
   (symbol (lib_id "Device:L") (at 100.33 83.82 90) (unit 1)
     (in_bom yes) (on_board yes) (dnp no) (fields_autoplaced)
-    (property "Reference" "L9" (at 100.33 78.74 90)
+    (property "Reference" "L7" (at 100.33 78.74 90)
       (effects (font (size 1.27 1.27)))
     )
@@
   (symbol (lib_id "Device:L") (at 157.48 57.15 0) (mirror x) (unit 1)
     (in_bom yes) (on_board yes) (dnp no)
-    (property "Reference" "L13" (at 156.21 55.88 0)
+    (property "Reference" "L10" (at 156.21 55.88 0)
       (effects (font (size 1.27 1.27)) (justify right))
     )
@@
   (symbol (lib_id "Device:L") (at 73.66 92.71 0) (mirror x) (unit 1)
     (in_bom yes) (on_board yes) (dnp no)
-    (property "Reference" "L10" (at 72.39 91.44 0)
+    (property "Reference" "L5" (at 72.39 91.44 0)
       (effects (font (size 1.27 1.27)) (justify right))
     )
@@
   (symbol (lib_id "Device:L") (at 73.66 57.15 0) (mirror x) (unit 1)
     (in_bom yes) (on_board yes) (dnp no)
-    (property "Reference" "L7" (at 72.39 55.88 0)
+    (property "Reference" "L4" (at 72.39 55.88 0)
       (effects (font (size 1.27 1.27)) (justify right))
     )
@@
   (symbol (lib_id "Device:L") (at 66.04 83.82 90) (unit 1)
     (in_bom yes) (on_board yes) (dnp no) (fields_autoplaced)
-    (property "Reference" "L8" (at 66.04 78.74 90)
+    (property "Reference" "L3" (at 66.04 78.74 90)
       (effects (font (size 1.27 1.27)))
     )
@@
   (symbol (lib_id "Device:L") (at 157.48 92.71 0) (mirror x) (unit 1)
     (in_bom yes) (on_board yes) (dnp no)
-    (property "Reference" "L16" (at 156.21 91.44 0)
+    (property "Reference" "L11" (at 156.21 91.44 0)
       (effects (font (size 1.27 1.27)) (justify right))
     )
@@
   (symbol (lib_id "Device:L") (at 149.86 48.26 90) (unit 1)
     (in_bom yes) (on_board yes) (dnp no) (fields_autoplaced)
-    (property "Reference" "L11" (at 149.86 43.18 90)
-      (effects (font (size 1.27 1.27)))
-    )
+    (property "Reference" "L8" (at 149.86 43.18 90)
+      (effects (font (size 1.27 1.27)))
+    )
