File: main/codec.kicad_sch (KiCad schematic)
At the start: 17 parts, among them J1 AudioJack5, U2 TLV320AIC3104IRHBR, U200 AP2120N-1.8TRG1

Commit message: GND and power rewired for codec
Parts:
- added C1 (x3): 100n, symbol Device:C
- added C1 (x3): 1u, symbol Device:C
- added C1: 10u, symbol Device:C
Connections:
- net +3.3V: no longer U2.18 (DRVDD1), U2.24 (DRVDD2), U2.25 (AVDD)
- net GND: now also C1.2, C1.2, C1.2, C1.2, C1.2, C1.2, C1.2
- new net VDDA: C1.1, C1.1, C1.1, C1.1, C1.1, C1.1, C1.1, U2.18 (DRVDD1), U2.24 (DRVDD2), U2.25 (AVDD)
Other:
- note added: "Decided to not separate analog and digital grounds"
- note added: "Разводить в соответствии с рекомендациями из даташита"

Commit message: comment about mic
Other:
- note added: "FIXME: Полная фигня с подключением микрофона Переделать!"
Changed lines of the file:
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@@
     (fill (type none))
+  )
+  (text "FIXME: Полная фигня с\nподключением микрофона\nПеределать!"
+    (at 48.26 146.05 0)
+    (effects (font (size 1.27 1.27)) (justify left bottom))
   )
   (text "TODO: задействовать кнопку гарнитуры" (at 199.39 88.9 0)

Commit message: FIXME comment about headphones
Other:
- note added: "FIXME: Полная фигня с подключением наушников Переделать!"
Changed lines of the file:
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@@
     (fill (type none))
+  )
+  (text "FIXME: Полная фигня с\nподключением наушников\nПеределать!"
+    (at 203.2 122.555 0)
+    (effects (font (size 1.27 1.27)) (justify left bottom))
   )
   (text "FIXME: Полная фигня с\nподключением микрофона\nПеределать!"

Commit message: Headset layout redrawn, PDF generated
Parts:
- removed C30: 10uF, symbol Device:C
- removed C31, C32: 100n, symbol Device:C
- removed J1: AudioJack5, symbol Connector_Audio:AudioJack5
- added J1: Headset, 16 Ohm, symbol Connector_Audio:AudioJack4
- added NT1: NetTie_2, symbol Device:NetTie_2
- C29: value 10uF -> 2n
- R1: value 10k -> 2.2k
Connections:
- net GND: now also C29.2
- net reset: now also C29.1
- net at U2.20 (HPLCOM): now also NT1.1
- net at U2.23 (HPROUT): now also J1.R1
- net at U2.22 (HPRCOM): now also J1.S, NT1.2
- net MIC_DET: now reaches C28.2
- net MIC_DET: now also R1.1, U2.14 (MIC2L/LINE2L/MICDET), J1.R2; no longer U2.16 (MIC2R/LINE2R)
- net at U2.19 (HPLOUT): now also J1.T; no longer C29.1
- removed net mic: C28.1, R1.1, U2.14 (MIC2L/LINE2L/MICDET)
- new net MIC_INPUT: C28.1, U2.16 (MIC2R/LINE2R)
Other:
- note added: "In cases where the ESD events generate a device reset, it is recommended to add at least a 1-nF capacitor connected between the RESET pin and DVSS. This capacitor avoids ESD events that could place the codec in default state."
- note removed: "FIXME: Полная фигня с подключением микрофона Переделать!"
- note removed: "FIXME: Полная фигня с подключением наушников Переделать!"
- note removed: "TODO: задействовать кнопку гарнитуры"
- note removed: "TODO: может лучше для мощного аудиовыхода использовать отдельный разъём?"
- note removed: "Вопрос: Эти конденсаторы (C31 и C32) точно нужны? Автор: Технологические для установки шлейфа для проверки звукового устройства USB"
- moved on the sheet: C1, C2, C24, C28, C33, C34, C35, C36, R1, U2, U200

Commit message: Audiojack rewired to Samsung standard
Connections:
- net MIC_DET: now also J1.S; no longer J1.R2
- net at NT1.2, U2.22 (HPRCOM): now also J1.R2; no longer J1.S
Changed lines of the file:
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@@
   (junction (at 147.955 34.925) (diameter 0) (color 0 0 0 0)
   )
-  (junction (at 181.61 102.87) (diameter 0) (color 0 0 0 0)
-  )
   (junction (at 160.02 132.08) (diameter 0) (color 0 0 0 0)
   )
@@
   (junction (at 215.9 48.26) (diameter 0) (color 0 0 0 0)
   )
+  (junction (at 177.165 104.14) (diameter 0) (color 0 0 0 0)
+  )
   (junction (at 203.2 30.48) (diameter 0) (color 0 0 0 0)
   )
@@
     (stroke (width 0) (type default))
   )
-  (wire (pts (xy 181.61 102.87) (xy 181.61 104.14))
+  (wire (pts (xy 177.165 102.87) (xy 177.165 104.14))
     (stroke (width 0) (type default))
   )
@@
     (stroke (width 0) (type default))
   )
-  (wire (pts (xy 151.13 104.14) (xy 181.61 104.14))
+  (wire (pts (xy 151.13 104.14) (xy 177.165 104.14))
     (stroke (width 0) (type default))
   )
@@
     (stroke (width 0) (type default))
   )
-  (wire (pts (xy 175.895 102.87) (xy 181.61 102.87))
+  (wire (pts (xy 175.895 102.87) (xy 177.165 102.87))
     (stroke (width 0) (type default))
   )
@@
     (stroke (width 0) (type default))
   )
+  (wire (pts (xy 177.165 104.14) (xy 177.165 105.41))
+    (stroke (width 0) (type default))
+  )
   (wire (pts (xy 59.69 128.27) (xy 59.69 118.11))
     (stroke (width 0) (type default))
@@
     (stroke (width 0) (type default))
   )
-  (wire (pts (xy 185.42 105.41) (xy 185.42 118.11))
+  (wire (pts (xy 185.42 102.87) (xy 185.42 118.11))
     (stroke (width 0) (type default))
   )
@@
     (stroke (width 0) (type default))
   )
-  (wire (pts (xy 181.61 102.87) (xy 188.595 102.87))
-    (stroke (width 0) (type default))
-  )
   (bus (pts (xy 72.39 105.41) (xy 72.39 128.27))
     (stroke (width 0) (type default))
@@
     (stroke (width 0) (type default))
   )
-  (wire (pts (xy 188.595 105.41) (xy 185.42 105.41))
-    (stroke (width 0) (type default))
-  )
   (bus (pts (xy 72.39 100.33) (xy 72.39 102.87))
     (stroke (width 0) (type default))
@@
     (stroke (width 0) (type default))
   )
+  (wire (pts (xy 188.595 105.41) (xy 177.165 105.41))
+    (stroke (width 0) (type default))
+  )
   (wire (pts (xy 55.88 90.17) (xy 69.85 90.17))
     (stroke (width 0) (type default))
@@
     (stroke (width 0) (type default))
   )
+  (wire (pts (xy 185.42 102.87) (xy 188.595 102.87))
+    (stroke (width 0) (type default))
+  )

Commit message: Mic input added
Parts:
- added J7: Mic, symbol Connector_Audio:AudioJack4
- added JP3, JP4, JP5, JP6: Jumper_2_Bridged, symbol Jumper:Jumper_2_Bridged
Connections:
- net MIC_DET: now also JP4.1 (A), JP5.1 (A), JP6.1 (A)
- net at J1.R2, NT1.2, U2.22 (HPRCOM): now also JP3.1 (A)
- new net: J7.T, JP6.2 (B)
- new net: J7.R1, JP5.2 (B)
- new net: J7.R2, JP4.2 (B)
- new net: J7.S, JP3.2 (B)
Changed lines of the file:
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@@
   (junction (at 240.03 48.26) (diameter 0) (color 0 0 0 0)
   )
+  (junction (at 187.325 105.41) (diameter 0) (color 0 0 0 0)
+  )
   (junction (at 215.9 55.88) (diameter 0) (color 0 0 0 0)
   )
@@
   (junction (at 227.965 43.815) (diameter 0) (color 0 0 0 0)
   )
+  (junction (at 185.42 137.16) (diameter 0) (color 0 0 0 0)
+  )
   (junction (at 161.925 34.925) (diameter 0) (color 0 0 0 0)
   )
   (junction (at 147.955 34.925) (diameter 0) (color 0 0 0 0)
   )
+  (junction (at 185.42 124.46) (diameter 0) (color 0 0 0 0)
+  )
   (junction (at 160.02 132.08) (diameter 0) (color 0 0 0 0)
   )
   (junction (at 185.42 118.11) (diameter 0) (color 0 0 0 0)
   )
+  (junction (at 185.42 131.445) (diameter 0) (color 0 0 0 0)
+  )
   (junction (at 215.9 48.26) (diameter 0) (color 0 0 0 0)
   )
@@
     (stroke (width 0) (type default))
   )
+  (wire (pts (xy 199.39 134.62) (xy 201.93 134.62))
+    (stroke (width 0) (type default))
+  )
   (wire (pts (xy 215.9 48.26) (xy 219.71 48.26))
     (stroke (width 0) (type default))
@@
     (stroke (width 0) (type default))
   )
+  (wire (pts (xy 199.39 131.445) (xy 199.39 134.62))
+    (stroke (width 0) (type default))
+  )
   (wire (pts (xy 215.9 59.69) (xy 227.965 59.69))
     (stroke (width 0) (type default))
@@
     (stroke (width 0) (type default))
   )
+  (wire (pts (xy 198.12 137.16) (xy 201.93 137.16))
+    (stroke (width 0) (type default))
+  )
+  (wire (pts (xy 198.12 139.7) (xy 201.93 139.7))
+    (stroke (width 0) (type default))
+  )
   (wire (pts (xy 59.69 128.27) (xy 55.88 128.27))
     (stroke (width 0) (type default))
   )
+  (wire (pts (xy 185.42 139.7) (xy 187.96 139.7))
+    (stroke (width 0) (type default))
+  )
+  (wire (pts (xy 187.325 105.41) (xy 187.325 126.365))
+    (stroke (width 0) (type default))
+  )
   (wire (pts (xy 80.01 133.35) (xy 82.55 133.35))
     (stroke (width 0) (type default))
@@
     (stroke (width 0) (type default))
   )
+  (wire (pts (xy 185.42 124.46) (xy 185.42 131.445))
+    (stroke (width 0) (type default))
+  )
   (wire (pts (xy 148.59 87.63) (xy 153.67 87.63))
     (stroke (width 0) (type default))
   )
+  (wire (pts (xy 185.42 137.16) (xy 185.42 139.7))
+    (stroke (width 0) (type default))
+  )
   (wire (pts (xy 215.9 48.26) (xy 215.9 43.815))
     (stroke (width 0) (type default))
@@
     (stroke (width 0) (type default))
   )
+  (wire (pts (xy 185.42 131.445) (xy 185.42 137.16))
+    (stroke (width 0) (type default))
+  )
   (wire (pts (xy 148.59 110.49) (xy 153.035 110.49))
     (stroke (width 0) (type default))
@@
     (stroke (width 0) (type default))
   )
+  (wire (pts (xy 185.42 137.16) (xy 187.96 137.16))
+    (stroke (width 0) (type default))
+  )
   (wire (pts (xy 160.02 129.54) (xy 160.02 132.08))
     (stroke (width 0) (type default))
@@
     (stroke (width 0) (type default))
   )
+  (wire (pts (xy 187.325 126.365) (xy 189.865 126.365))
+    (stroke (width 0) (type default))
+  )
   (wire (pts (xy 153.035 107.95) (xy 188.595 107.95))
     (stroke (width 0) (type default))
@@
     (stroke (width 0) (type default))
   )
+  (wire (pts (xy 185.42 131.445) (xy 188.595 131.445))
+    (stroke (width 0) (type default))
+  )
   (wire (pts (xy 236.22 48.26) (xy 240.03 48.26))
     (stroke (width 0) (type default))
   )
+  (wire (pts (xy 201.93 126.365) (xy 200.025 126.365))
+    (stroke (width 0) (type default))
+  )
   (bus (pts (xy 72.39 100.33) (xy 72.39 102.87))
     (stroke (width 0) (type default))
@@
     (stroke (width 0) (type default))
   )
+  (wire (pts (xy 201.93 132.08) (xy 201.93 126.365))
+    (stroke (width 0) (type default))
+  )
   (wire (pts (xy 148.59 77.47) (xy 148.59 82.55))
     (stroke (width 0) (type default))
@@
     (stroke (width 0) (type default))
   )
+  (wire (pts (xy 198.755 131.445) (xy 199.39 131.445))
+    (stroke (width 0) (type default))
+  )
   (wire (pts (xy 212.09 55.88) (xy 215.9 55.88))
     (stroke (width 0) (type default))
@@
     (stroke (width 0) (type default))
   )
-  (wire (pts (xy 188.595 105.41) (xy 177.165 105.41))
+  (wire (pts (xy 177.165 105.41) (xy 187.325 105.41))
     (stroke (width 0) (type default))
   )
@@
   )
   (wire (pts (xy 74.93 107.95) (xy 82.55 107.95))
+    (stroke (width 0) (type default))
+  )
+  (wire (pts (xy 187.325 105.41) (xy 188.595 105.41))
     (stroke (width 0) (type default))
   )
@@
     )
   )
+  (symbol (lib_id "Jumper:Jumper_2_Bridged") (at 193.04 139.7 0) (unit 1)
+    (in_bom yes) (on_board yes) (dnp no)
+    (property "Reference" "JP6" (at 193.04 141.605 0)
+      (effects (font (size 1.27 1.27)))
+    )
+    (property "Value" "Jumper_2_Bridged" (at 193.04 137.16 0)
+      (effects (font (size 1.27 1.27)) hide)
+    )
+    (property "Footprint" "" (at 193.04 139.7 0)
+      (effects (font (size 1.27 1.27)) hide)
+    )
+    (property "Datasheet" "~" (at 193.04 139.7 0)
+      (effects (font (size 1.27 1.27)) hide)
+    )
+    (pin "1")
+    (pin "2")
+    (instances
+      (project "main"
+        (path "/cb08c644-d155-44e5-86e1-31645eace055/e511764a-2dd7-4601-8d00-331d6dbffa9f"
+          (reference "JP6") (unit 1)
+        )
+      )
+    )
+  )
+  (symbol (lib_id "Jumper:Jumper_2_Bridged") (at 193.04 137.16 0) (unit 1)
+    (in_bom yes) (on_board yes) (dnp no) (fields_autoplaced)
+    (property "Reference" "JP5" (at 193.04 134.62 0)
+      (effects (font (size 1.27 1.27)))
+    )
+    (property "Value" "Jumper_2_Bridged" (at 193.04 134.62 0)
+      (effects (font (size 1.27 1.27)) hide)
+    )
+    (property "Footprint" "" (at 193.04 137.16 0)
+      (effects (font (size 1.27 1.27)) hide)
+    )
+    (property "Datasheet" "~" (at 193.04 137.16 0)
+      (effects (font (size 1.27 1.27)) hide)
+    )
+    (pin "1")
+    (pin "2")
+    (instances
+      (project "main"
+        (path "/cb08c644-d155-44e5-86e1-31645eace055/e511764a-2dd7-4601-8d00-331d6dbffa9f"
+          (reference "JP5") (unit 1)
+        )
+      )
+    )
+  )
   (symbol (lib_id "power:GND") (at 120.015 45.085 0) (unit 1)
     (in_bom yes) (on_board yes) (dnp no) (fields_autoplaced)
@@
     )
   )
+  (symbol (lib_id "Connector_Audio:AudioJack4") (at 207.01 134.62 0) (mirror y) (unit 1)
+    (in_bom yes) (on_board yes) (dnp no)
+    (property "Reference" "J7" (at 209.55 125.73 0)
+      (effects (font (size 1.27 1.27)))
+    )
+    (property "Value" "Mic" (at 209.55 128.27 0)
+      (effects (font (size 1.27 1.27)))
+    )
+    (property "Footprint" "" (at 207.01 134.62 0)
+      (effects (font (size 1.27 1.27)) hide)
+    )
+    (property "Datasheet" "~" (at 207.01 134.62 0)
+      (effects (font (size 1.27 1.27)) hide)
+    )
+    (pin "S")
+    (pin "R1")
+    (pin "T")
+    (pin "R2")
+    (instances
+      (project "main"
+        (path "/cb08c644-d155-44e5-86e1-31645eace055/e511764a-2dd7-4601-8d00-331d6dbffa9f"
+          (reference "J7") (unit 1)
+        )
+      )
+    )
+  )
   (symbol (lib_id "Device:C") (at 52.07 128.27 90) (unit 1)
     (in_bom yes) (on_board yes) (dnp no) (fields_autoplaced)
@@
         (path "/cb08c644-d155-44e5-86e1-31645eace055/e511764a-2dd7-4601-8d00-331d6dbffa9f"
           (reference "#PWR019") (unit 1)
+        )
+      )
+    )
+  )
+  (symbol (lib_id "Jumper:Jumper_2_Bridged") (at 193.675 131.445 0) (unit 1)
+    (in_bom yes) (on_board yes) (dnp no) (fields_autoplaced)
+    (property "Reference" "JP4" (at 193.675 128.27 0)
+      (effects (font (size 1.27 1.27)))
+    )
+    (property "Value" "Jumper_2_Bridged" (at 193.675 128.905 0)
+      (effects (font (size 1.27 1.27)) hide)
+    )
+    (property "Footprint" "" (at 193.675 131.445 0)
+      (effects (font (size 1.27 1.27)) hide)
+    )
+    (property "Datasheet" "~" (at 193.675 131.445 0)
+      (effects (font (size 1.27 1.27)) hide)
+    )
+    (pin "1")
+    (pin "2")
+    (instances
+      (project "main"
+        (path "/cb08c644-d155-44e5-86e1-31645eace055/e511764a-2dd7-4601-8d00-331d6dbffa9f"
+          (reference "JP4") (unit 1)
         )
       )
@@
         )
       )
+    )
+  )
+  (symbol (lib_id "Jumper:Jumper_2_Bridged") (at 194.945 126.365 0) (unit 1)
+    (in_bom yes) (on_board yes) (dnp no) (fields_autoplaced)
+    (property "Reference" "JP3" (at 194.945 123.19 0)
+      (effects (font (size 1.27 1.27)))
+    )
+    (property "Value" "Jumper_2_Bridged" (at 194.945 123.825 0)
+      (effects (font (size 1.27 1.27)) hide)
+    )
+    (property "Footprint" "" (at 194.945 126.365 0)
+      (effects (font (size 1.27 1.27)) hide)
+    )
+    (property "Datasheet" "~" (at 194.945 126.365 0)
+      (effects (font (size 1.27 1.27)) hide)
+    )
+    (pin "1")
+    (pin "2")
+    (instances
+      (project "main"
+        (path "/cb08c644-d155-44e5-86e1-31645eace055/e511764a-2dd7-4601-8d00-331d6dbffa9f"
+          (reference "JP3") (unit 1)
+        )
+      )

Commit message: headset circuit redrawn
Other:
- moved on the sheet: J1
Changed lines of the file:
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@@
   (junction (at 240.03 48.26) (diameter 0) (color 0 0 0 0)
   )
-  (junction (at 187.325 105.41) (diameter 0) (color 0 0 0 0)
+  (junction (at 189.23 107.95) (diameter 0) (color 0 0 0 0)
   )
   (junction (at 215.9 55.88) (diameter 0) (color 0 0 0 0)
@@
   (junction (at 185.42 137.16) (diameter 0) (color 0 0 0 0)
   )
+  (junction (at 177.165 107.95) (diameter 0) (color 0 0 0 0)
+  )
   (junction (at 161.925 34.925) (diameter 0) (color 0 0 0 0)
   )
@@
   (junction (at 215.9 48.26) (diameter 0) (color 0 0 0 0)
   )
-  (junction (at 177.165 104.14) (diameter 0) (color 0 0 0 0)
-  )
   (junction (at 203.2 30.48) (diameter 0) (color 0 0 0 0)
   )
@@
     (stroke (width 0) (type default))
   )
-  (wire (pts (xy 177.165 102.87) (xy 177.165 104.14))
-    (stroke (width 0) (type default))
-  )
   (wire (pts (xy 55.88 102.87) (xy 66.04 102.87))
     (stroke (width 0) (type default))
@@
     (stroke (width 0) (type default))
   )
+  (wire (pts (xy 189.23 107.95) (xy 193.675 107.95))
+    (stroke (width 0) (type default))
+  )
   (wire (pts (xy 215.9 59.69) (xy 227.965 59.69))
     (stroke (width 0) (type default))
@@
     (stroke (width 0) (type default))
   )
+  (wire (pts (xy 177.165 102.87) (xy 177.165 107.95))
+    (stroke (width 0) (type default))
+  )
   (bus (pts (xy 72.39 78.105) (xy 72.39 97.79))
     (stroke (width 0) (type default))
@@
     (stroke (width 0) (type default))
   )
-  (wire (pts (xy 151.13 104.14) (xy 177.165 104.14))
+  (wire (pts (xy 148.59 107.95) (xy 177.165 107.95))
     (stroke (width 0) (type default))
   )
@@
     (stroke (width 0) (type default))
   )
-  (wire (pts (xy 187.325 105.41) (xy 187.325 126.365))
+  (wire (pts (xy 189.23 107.95) (xy 189.23 126.365))
     (stroke (width 0) (type default))
   )
@@
     (stroke (width 0) (type default))
   )
-  (wire (pts (xy 177.165 104.14) (xy 177.165 105.41))
-    (stroke (width 0) (type default))
-  )
   (wire (pts (xy 59.69 128.27) (xy 59.69 118.11))
     (stroke (width 0) (type default))
@@
     (stroke (width 0) (type default))
   )
-  (wire (pts (xy 148.59 110.49) (xy 153.035 110.49))
+  (wire (pts (xy 148.59 110.49) (xy 193.675 110.49))
     (stroke (width 0) (type default))
   )
@@
     (stroke (width 0) (type default))
   )
-  (wire (pts (xy 185.42 102.87) (xy 185.42 118.11))
+  (wire (pts (xy 185.42 105.41) (xy 185.42 118.11))
     (stroke (width 0) (type default))
   )
@@
     (stroke (width 0) (type default))
   )
-  (wire (pts (xy 187.325 126.365) (xy 189.865 126.365))
-    (stroke (width 0) (type default))
-  )
-  (wire (pts (xy 153.035 107.95) (xy 188.595 107.95))
+  (wire (pts (xy 189.23 126.365) (xy 189.865 126.365))
     (stroke (width 0) (type default))
   )
@@
     (stroke (width 0) (type default))
   )
-  (wire (pts (xy 171.45 110.49) (xy 188.595 110.49))
+  (wire (pts (xy 171.45 113.03) (xy 193.675 113.03))
     (stroke (width 0) (type default))
   )
@@
     (stroke (width 0) (type default))
   )
-  (wire (pts (xy 148.59 107.95) (xy 151.13 107.95))
-    (stroke (width 0) (type default))
-  )
   (wire (pts (xy 120.015 45.085) (xy 120.015 42.545))
     (stroke (width 0) (type default))
@@
     (stroke (width 0) (type default))
   )
-  (wire (pts (xy 171.45 105.41) (xy 171.45 110.49))
+  (wire (pts (xy 171.45 105.41) (xy 171.45 113.03))
     (stroke (width 0) (type default))
   )
@@
     (stroke (width 0) (type default))
   )
-  (wire (pts (xy 153.035 107.95) (xy 153.035 110.49))
-    (stroke (width 0) (type default))
-  )
-  (wire (pts (xy 177.165 105.41) (xy 187.325 105.41))
-    (stroke (width 0) (type default))
-  )
   (wire (pts (xy 55.88 90.17) (xy 69.85 90.17))
     (stroke (width 0) (type default))
@@
     (stroke (width 0) (type default))
   )
-  (wire (pts (xy 185.42 102.87) (xy 188.595 102.87))
+  (wire (pts (xy 185.42 105.41) (xy 193.675 105.41))
     (stroke (width 0) (type default))
   )
@@
     (stroke (width 0) (type default))
   )
-  (wire (pts (xy 187.325 105.41) (xy 188.595 105.41))
+  (wire (pts (xy 177.165 107.95) (xy 189.23 107.95))
     (stroke (width 0) (type default))
   )
@@
   )
   (wire (pts (xy 148.59 138.43) (xy 160.02 138.43))
-    (stroke (width 0) (type default))
-  )
-  (wire (pts (xy 151.13 104.14) (xy 151.13 107.95))
     (stroke (width 0) (type default))
   )
@@
     )
   )
-  (symbol (lib_id "Connector_Audio:AudioJack4") (at 193.675 105.41 0) (mirror y) (unit 1)
+  (symbol (lib_id "Connector_Audio:AudioJack4") (at 198.755 107.95 0) (mirror y) (unit 1)
     (in_bom yes) (on_board yes) (dnp no)
-    (property "Reference" "J1" (at 196.215 96.52 0)
-      (effects (font (size 1.27 1.27)))
-    )
-    (property "Value" "Headset, 16 Ohm" (at 196.215 99.06 0)
-      (effects (font (size 1.27 1.27)))
-    )
-    (property "Footprint" "" (at 193.675 105.41 0)
-      (effects (font (size 1.27 1.27)) hide)
-    )
-    (property "Datasheet" "~" (at 193.675 105.41 0)
-      (effects (font (size 1.27 1.27)) hide)
-    )
+    (property "Reference" "J1" (at 201.295 99.06 0)
+      (effects (font (size 1.27 1.27)))
+    )
+    (property "Value" "Headset, 16 Ohm" (at 201.295 101.6 0)
+      (effects (font (size 1.27 1.27)))
+    )
+    (property "Footprint" "" (at 198.755 107.95 0)
+      (effects (font (size 1.27 1.27)) hide)
+    )
+    (property "Datasheet" "~" (at 198.755 107.95 0)
+      (effects (font (size 1.27 1.27)) hide)
+    )
