File: main/rf_processing.kicad_sch (KiCad schematic)
At the start: 5 parts, among them T1 Transformer_1P_SS

Commit message: 50 Ohm resistors moved from modulator
Parts:
- removed T1: Transformer_1P_SS, symbol Device:Transformer_1P_SS
- added R1 (x2): 50, symbol Device:R
- added TR1: ADT16-1T, RF_Mini-Circuits:Mini-Circuits_CD542_H2.84mm, symbol Transformer:ADT16-1T
Connections:
- net Filter selector/filtered: now also TR1.3
- net GND: now also TR1.1
- net Modulator/SDR_NEG: now also R1.1
- net Modulator/SDR_POS: now also R1.1
- net QSE_BIAS: now also TR1.5
- net SDR_NEG: now also R1.2, TR1.4
- net SDR_POS: now also R1.2, TR1.6
Other:
- note added: "TODO: Зачем здесь нужны резисторы?"
Changed lines of the file:
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@@
   (junction (at 207.01 119.38) (diameter 0) (color 0 0 0 0)
   )
+  (wire (pts (xy 163.83 85.09) (xy 163.83 57.15))
+    (stroke (width 0) (type default))
+  )
+  (wire (pts (xy 175.26 62.23) (xy 175.26 95.25))
+    (stroke (width 0) (type default))
+  )
   (wire (pts (xy 129.54 85.09) (xy 139.7 85.09))
     (stroke (width 0) (type default))
   )
+  (wire (pts (xy 149.86 85.09) (xy 163.83 85.09))
+    (stroke (width 0) (type default))
+  )
+  (wire (pts (xy 142.24 62.23) (xy 144.78 62.23))
+    (stroke (width 0) (type default))
+  )
+  (wire (pts (xy 152.4 62.23) (xy 175.26 62.23))
+    (stroke (width 0) (type default))
+  )
   (wire (pts (xy 207.01 121.92) (xy 207.01 119.38))
     (stroke (width 0) (type default))
@@
     (stroke (width 0) (type default))
   )
+  (wire (pts (xy 163.83 57.15) (xy 152.4 57.15))
+    (stroke (width 0) (type default))
+  )
   (wire (pts (xy 207.01 119.38) (xy 193.04 119.38))
     (stroke (width 0) (type default))
   )
+  (wire (pts (xy 132.08 57.15) (xy 144.78 57.15))
+    (stroke (width 0) (type default))
+  )
   (wire (pts (xy 180.34 90.17) (xy 180.34 119.38))
     (stroke (width 0) (type default))
   )
+  (wire (pts (xy 142.24 59.69) (xy 142.24 62.23))
+    (stroke (width 0) (type default))
+  )
   (wire (pts (xy 193.04 119.38) (xy 193.04 121.92))
     (stroke (width 0) (type default))
@@
     (stroke (width 0) (type default))
   )
-  (wire (pts (xy 160.02 90.17) (xy 180.34 90.17))
+  (wire (pts (xy 149.86 90.17) (xy 180.34 90.17))
     (stroke (width 0) (type default))
   )
@@
     (stroke (width 0) (type default))
   )
+  (wire (pts (xy 132.08 59.69) (xy 142.24 59.69))
+    (stroke (width 0) (type default))
+  )
+  (wire (pts (xy 149.86 95.25) (xy 175.26 95.25))
+    (stroke (width 0) (type default))
+  )
   (wire (pts (xy 180.34 119.38) (xy 193.04 119.38))
     (stroke (width 0) (type default))
+  )
+  (text "TODO: Зачем здесь нужны резисторы?" (at 138.43 46.99 0)
+    (effects (font (size 1.27 1.27)) (justify left bottom))
+  )
+  (label "SDR_NEG" (at 152.4 85.09 0) (fields_autoplaced)
+    (effects (font (size 1.27 1.27)) (justify left bottom))
+  )
+  (label "SDR_POS" (at 152.4 95.25 0) (fields_autoplaced)
+    (effects (font (size 1.27 1.27)) (justify left bottom))
   )
   (label "QSE_BIAS" (at 165.1 90.17 0) (fields_autoplaced)
     (effects (font (size 1.27 1.27)) (justify left bottom))
   )
-  (hierarchical_label "f0" (shape input) (at 115.57 57.15 180) (fields_autoplaced)
+  (hierarchical_label "phase0" (shape input) (at 115.57 57.15 180) (fields_autoplaced)
     (effects (font (size 1.27 1.27)) (justify right))
   )
@@
     (effects (font (size 1.27 1.27)) (justify right))
   )
-  (hierarchical_label "f1" (shape input) (at 115.57 59.69 180) (fields_autoplaced)
+  (hierarchical_label "phase1" (shape input) (at 115.57 59.69 180) (fields_autoplaced)
     (effects (font (size 1.27 1.27)) (justify right))
-  )
-  (hierarchical_label "SDR_NEG" (shape bidirectional) (at 160.02 95.25 0) (fields_autoplaced)
-    (effects (font (size 1.27 1.27)) (justify left))
-  )
-  (hierarchical_label "SDR_POS" (shape bidirectional) (at 160.02 85.09 0) (fields_autoplaced)
-    (effects (font (size 1.27 1.27)) (justify left))
   )
   (hierarchical_label "filter_selector1" (shape bidirectional) (at 115.57 85.09 180) (fields_autoplaced)
     (effects (font (size 1.27 1.27)) (justify right))
+  )
+  (symbol (lib_id "Transformer:ADT16-1T") (at 144.78 90.17 0) (unit 1)
+    (in_bom yes) (on_board yes) (dnp no) (fields_autoplaced)
+    (property "Reference" "TR1" (at 144.78 80.01 0)
+      (effects (font (size 1.27 1.27)))
+    )
+    (property "Value" "ADT16-1T" (at 144.78 82.55 0)
+      (effects (font (size 1.27 1.27)))
+    )
+    (property "Footprint" "RF_Mini-Circuits:Mini-Circuits_CD542_H2.84mm" (at 144.78 99.06 0)
+      (effects (font (size 1.27 1.27)) hide)
+    )
+    (property "Datasheet" "https://www.minicircuits.com/pdfs/ADT16-1T+.pdf" (at 144.78 90.17 0)
+      (effects (font (size 1.27 1.27)) hide)
+    )
+    (pin "4")
+    (pin "1")
+    (pin "2")
+    (pin "3")
+    (pin "5")
+    (pin "6")
+    (instances
+      (project "main"
+        (path "/cb08c644-d155-44e5-86e1-31645eace055/f348e705-e1f2-401a-94bd-812b815f83a8"
+          (reference "TR1") (unit 1)
+        )
+      )
+    )
   )
   (symbol (lib_id "Device:R") (at 193.04 125.73 0) (mirror y) (unit 1)
@@
     )
   )
+  (symbol (lib_id "Device:R") (at 148.59 57.15 90) (unit 1)
+    (in_bom yes) (on_board yes) (dnp no) (fields_autoplaced)
+    (property "Reference" "R1" (at 148.59 50.8 90)
+      (effects (font (size 1.27 1.27)))
+    )
+    (property "Value" "50" (at 148.59 53.34 90)
+      (effects (font (size 1.27 1.27)))
+    )
+    (property "Footprint" "" (at 148.59 58.928 90)
+      (effects (font (size 1.27 1.27)) hide)
+    )
+    (property "Datasheet" "~" (at 148.59 57.15 0)
+      (effects (font (size 1.27 1.27)) hide)
+    )
+    (pin "2")
+    (pin "1")
+    (instances
+      (project "main"
+        (path "/cb08c644-d155-44e5-86e1-31645eace055"
+          (reference "R1") (unit 1)
+        )
+        (path "/cb08c644-d155-44e5-86e1-31645eace055/f348e705-e1f2-401a-94bd-812b815f83a8/6911640e-2f8b-4689-850c-33e2fd821898"
+          (reference "R4") (unit 1)
+        )
+        (path "/cb08c644-d155-44e5-86e1-31645eace055/f348e705-e1f2-401a-94bd-812b815f83a8"
+          (reference "R33") (unit 1)
+        )
+        (path "/cb08c644-d155-44e5-86e1-31645eace055/f348e705-e1f2-401a-94bd-812b815f83a8/071bf193-b8ce-446c-a6f0-4f73f2e6bcab"
+          (reference "R33") (unit 1)
+        )
+      )
+    )
+  )
   (symbol (lib_id "power:GND") (at 222.25 129.54 0) (mirror y) (unit 1)
     (in_bom yes) (on_board yes) (dnp no) (fields_autoplaced)
@@
         (path "/cb08c644-d155-44e5-86e1-31645eace055/f348e705-e1f2-401a-94bd-812b815f83a8"
           (reference "#PWR073") (unit 1)
-        )
-      )
-    )
-  )
-  (symbol (lib_id "Device:Transformer_1P_SS") (at 149.86 90.17 0) (unit 1)
-    (in_bom yes) (on_board yes) (dnp no) (fields_autoplaced)
-    (property "Reference" "T1" (at 149.8727 80.01 0)
-      (effects (font (size 1.27 1.27)))
-    )
-    (property "Value" "Transformer_1P_SS" (at 149.8727 82.55 0)
-      (effects (font (size 1.27 1.27)))
-    )
-    (property "Footprint" "" (at 149.86 90.17 0)
-      (effects (font (size 1.27 1.27)) hide)
-    )
-    (property "Datasheet" "~" (at 149.86 90.17 0)
-      (effects (font (size 1.27 1.27)) hide)
-    )
-    (pin "4")
-    (pin "5")
-    (pin "1")
-    (pin "2")
-    (pin "3")
-    (instances
-      (project "main"
-        (path "/cb08c644-d155-44e5-86e1-31645eace055"
-          (reference "T1") (unit 1)
-        )
-        (path "/cb08c644-d155-44e5-86e1-31645eace055/f348e705-e1f2-401a-94bd-812b815f83a8"
-          (reference "T1") (unit 1)
         )
       )
@@
         )
       )
+    )
+  )
+  (symbol (lib_id "Device:R") (at 148.59 62.23 90) (unit 1)
+    (in_bom yes) (on_board yes) (dnp no) (fields_autoplaced)
+    (property "Reference" "R1" (at 148.59 66.04 90)
+      (effects (font (size 1.27 1.27)))
+    )
+    (property "Value" "50" (at 148.59 68.58 90)
+      (effects (font (size 1.27 1.27)))
+    )
+    (property "Footprint" "" (at 148.59 64.008 90)
+      (effects (font (size 1.27 1.27)) hide)
+    )
+    (property "Datasheet" "~" (at 148.59 62.23 0)
+      (effects (font (size 1.27 1.27)) hide)
+    )
+    (pin "2")
+    (pin "1")
+    (instances
+      (project "main"
+        (path "/cb08c644-d155-44e5-86e1-31645eace055"
+          (reference "R1") (unit 1)
+        )
+        (path "/cb08c644-d155-44e5-86e1-31645eace055/f348e705-e1f2-401a-94bd-812b815f83a8/6911640e-2f8b-4689-850c-33e2fd821898"
+          (reference "R4") (unit 1)
+        )
+        (path "/cb08c644-d155-44e5-86e1-31645eace055/f348e705-e1f2-401a-94bd-812b815f83a8"
+          (reference "R34") (unit 1)
+        )
+        (path "/cb08c644-d155-44e5-86e1-31645eace055/f348e705-e1f2-401a-94bd-812b815f83a8/071bf193-b8ce-446c-a6f0-4f73f2e6bcab"
+          (reference "R34") (unit 1)
+        )
+      )

Commit message: Moving components
Parts:
- added R1 (x2): 10, symbol Device:R
Connections:
- net SDR_NEG: now also TR1.6, R1.1; no longer TR1.4
- net SDR_POS: now also TR1.4, R1.1; no longer TR1.6
Other:
- note added: "TODO: Зачем здесь нужны эти резисторы?"
- note removed: "TODO: Зачем здесь нужны резисторы?"

Commit message: Mixer added
Parts:
- removed R1 (x2): 10, symbol Device:R
Other:
- added sheet Mixer (Detector) (mixer.kicad_sch)
Changed lines of the file:
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@@
-    )
-  )
-  (symbol (lib_id "Device:R") (at 193.04 57.15 90) (unit 1)
-    (in_bom yes) (on_board yes) (dnp no) (fields_autoplaced)
-    (property "Reference" "R1" (at 193.04 50.8 90)
-      (effects (font (size 1.27 1.27)))
-    )
-    (property "Value" "10" (at 193.04 53.34 90)
-      (effects (font (size 1.27 1.27)))
-    )
-    (property "Footprint" "" (at 193.04 58.928 90)
-      (effects (font (size 1.27 1.27)) hide)
-    )
-    (property "Datasheet" "~" (at 193.04 57.15 0)
-      (effects (font (size 1.27 1.27)) hide)
-    )
-    (pin "2")
-    (pin "1")
-    (instances
-      (project "main"
-        (path "/cb08c644-d155-44e5-86e1-31645eace055"
-          (reference "R1") (unit 1)
-        )
-        (path "/cb08c644-d155-44e5-86e1-31645eace055/f348e705-e1f2-401a-94bd-812b815f83a8/6911640e-2f8b-4689-850c-33e2fd821898"
-          (reference "R4") (unit 1)
-        )
-        (path "/cb08c644-d155-44e5-86e1-31645eace055/f348e705-e1f2-401a-94bd-812b815f83a8"
-          (reference "R19") (unit 1)
-        )
-        (path "/cb08c644-d155-44e5-86e1-31645eace055/f348e705-e1f2-401a-94bd-812b815f83a8/071bf193-b8ce-446c-a6f0-4f73f2e6bcab"
-          (reference "R33") (unit 1)
-        )
-      )
     )
   )
@@
         (path "/cb08c644-d155-44e5-86e1-31645eace055/f348e705-e1f2-401a-94bd-812b815f83a8"
           (reference "C53") (unit 1)
-        )
-      )
-    )
-  )
-  (symbol (lib_id "Device:R") (at 193.04 62.23 90) (mirror x) (unit 1)
-    (in_bom yes) (on_board yes) (dnp no) (fields_autoplaced)
-    (property "Reference" "R1" (at 193.04 66.04 90)
-      (effects (font (size 1.27 1.27)))
-    )
-    (property "Value" "10" (at 193.04 68.58 90)
-      (effects (font (size 1.27 1.27)))
-    )
-    (property "Footprint" "" (at 193.04 60.452 90)
-      (effects (font (size 1.27 1.27)) hide)
-    )
-    (property "Datasheet" "~" (at 193.04 62.23 0)
-      (effects (font (size 1.27 1.27)) hide)
-    )
-    (pin "2")
-    (pin "1")
-    (instances
-      (project "main"
-        (path "/cb08c644-d155-44e5-86e1-31645eace055"
-          (reference "R1") (unit 1)
-        )
-        (path "/cb08c644-d155-44e5-86e1-31645eace055/f348e705-e1f2-401a-94bd-812b815f83a8/6911640e-2f8b-4689-850c-33e2fd821898"
-          (reference "R4") (unit 1)
-        )
-        (path "/cb08c644-d155-44e5-86e1-31645eace055/f348e705-e1f2-401a-94bd-812b815f83a8"
-          (reference "R20") (unit 1)
-        )
-        (path "/cb08c644-d155-44e5-86e1-31645eace055/f348e705-e1f2-401a-94bd-812b815f83a8/071bf193-b8ce-446c-a6f0-4f73f2e6bcab"
-          (reference "R34") (unit 1)
         )
       )
@@
       )
     )
+  )
+  (sheet (at 235.585 70.485) (size 26.67 25.4) (fields_autoplaced)
+    (stroke (width 0.1524) (type solid))
+    (fill (color 0 0 0 0.0000))
+    (property "Sheetname" "Mixer (Detector)" (at 235.585 69.7734 0)
+      (effects (font (size 1.27 1.27)) (justify left bottom))
+    )
+    (property "Sheetfile" "mixer.kicad_sch" (at 235.585 96.4696 0)
+      (effects (font (size 1.27 1.27)) (justify left top))
+    )
+    (instances
+      (project "main"
+        (path "/cb08c644-d155-44e5-86e1-31645eace055/f348e705-e1f2-401a-94bd-812b815f83a8" (page "12"))
+      )
+    )

Commit message: mixer connected, MCU wiring changed
Other:
- sheet Mixer (Detector) ports: added QSD_EN, SDR_I, SDR_NEG, SDR_POS, SDR_Q, f0, f1; removed none
- moved on the sheet: C64, R1, TR1

Commit message: assigns
Parts:
- renumbered C64 to C38
Changed lines of the file:
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@@
   (symbol (lib_id "Device:C") (at 184.15 130.81 0) (mirror x) (unit 1)
     (in_bom yes) (on_board yes) (dnp no)
-    (property "Reference" "C64" (at 180.34 129.54 0)
+    (property "Reference" "C38" (at 180.34 129.54 0)
       (effects (font (size 1.27 1.27)) (justify right))
     )
@@
   (symbol (lib_id "power:+3.3V") (at 170.18 114.3 0) (mirror y) (unit 1)
     (in_bom yes) (on_board yes) (dnp no) (fields_autoplaced)
-    (property "Reference" "#PWR065" (at 170.18 118.11 0)
+    (property "Reference" "#PWR061" (at 170.18 118.11 0)
       (effects (font (size 1.27 1.27)) hide)
     )
@@
   (symbol (lib_id "Device:C") (at 199.39 130.81 0) (mirror x) (unit 1)
     (in_bom yes) (on_board yes) (dnp no)
-    (property "Reference" "C64" (at 195.58 129.54 0)
-      (effects (font (size 1.27 1.27)) (justify right))
-    )
+    (property "Reference" "C38" (at 195.58 129.54 0)
+      (effects (font (size 1.27 1.27)) (justify right))
+    )

Commit message: R37 bias supply removed
Connections:
- net GND: no longer TR1.1
- net QSE_BIAS: now also TR1.1
Changed lines of the file:
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@@
   (junction (at 184.15 124.46) (diameter 0) (color 0 0 0 0)
   )
+  (junction (at 157.48 111.76) (diameter 0) (color 0 0 0 0)
+  )
   (wire (pts (xy 140.97 90.17) (xy 140.97 57.15))
     (stroke (width 0) (type default))
@@
     (stroke (width 0) (type default))
   )
+  (wire (pts (xy 116.84 111.76) (xy 157.48 111.76))
+    (stroke (width 0) (type default))
+  )
   (wire (pts (xy 115.57 57.15) (xy 121.92 57.15))
     (stroke (width 0) (type default))
   )
+  (wire (pts (xy 116.84 100.33) (xy 116.84 111.76))
+    (stroke (width 0) (type default))
+  )
   (wire (pts (xy 172.72 54.61) (xy 166.37 54.61))
     (stroke (width 0) (type default))
@@
     (stroke (width 0) (type default))
   )
-  (wire (pts (xy 157.48 95.25) (xy 157.48 124.46))
+  (wire (pts (xy 157.48 95.25) (xy 157.48 111.76))
     (stroke (width 0) (type default))
   )
@@
   )
   (wire (pts (xy 157.48 124.46) (xy 170.18 124.46))
+    (stroke (width 0) (type default))
+  )
+  (wire (pts (xy 157.48 111.76) (xy 157.48 124.46))
     (stroke (width 0) (type default))
   )
@@
         )
       )
-    )
-  )
-  (symbol (lib_id "power:GND") (at 116.84 100.33 0) (unit 1)
-    (in_bom yes) (on_board yes) (dnp no) (fields_autoplaced)
-    (property "Reference" "#PWR069" (at 116.84 106.68 0)
-      (effects (font (size 1.27 1.27)) hide)
-    )
-    (property "Value" "GND" (at 116.84 105.41 0)
-      (effects (font (size 1.27 1.27)))
-    )
-    (property "Footprint" "" (at 116.84 100.33 0)
-      (effects (font (size 1.27 1.27)) hide)
-    )
-    (property "Datasheet" "" (at 116.84 100.33 0)
-      (effects (font (size 1.27 1.27)) hide)
-    )
-    (pin "1")
-    (instances
-      (project "main"
-        (path "/cb08c644-d155-44e5-86e1-31645eace055"
-          (reference "#PWR069") (unit 1)
-        )
-        (path "/cb08c644-d155-44e5-86e1-31645eace055/f348e705-e1f2-401a-94bd-812b815f83a8"
-          (reference "#PWR069") (unit 1)
-        )
-      )

Commit message: Power SWR Bridge used as input ANT connection
Parts:
- added C63, C65: 100nF, symbol Device:C
- added R1: 100k, symbol Device:R
- added R1 (x2): 2.2k, symbol Device:R
Connections:
- net +3.3V: now also R1.1
- net GND: now also C63.1, R1.2
- new net: C63.2, R1.1, R1.1, R1.2
- new net: C65.2, R1.2
- new net Filter selector/filter_in: C65.1
Other:
- added sheet Power SWR Bridge (power_swr_bridge.kicad_sch)
- sheet Filter selector ports: added filter_in; removed none
