File: main/rf_processing.kicad_sch (KiCad schematic)
At the start: 12 parts

Commit message: comment about mic
Connections:
- net GND: now also TR1.1
- net QSE_BIAS: no longer TR1.1
Changed lines of the file:
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@@
   (junction (at 52.07 54.61) (diameter 0) (color 0 0 0 0)
   )
-  (junction (at 157.48 111.76) (diameter 0) (color 0 0 0 0)
-  )
   (wire (pts (xy 45.72 106.045) (xy 45.72 95.25))
     (stroke (width 0) (type default))
@@
     (stroke (width 0) (type default))
   )
-  (wire (pts (xy 116.84 111.76) (xy 157.48 111.76))
-    (stroke (width 0) (type default))
-  )
-  (wire (pts (xy 115.57 57.15) (xy 121.92 57.15))
-    (stroke (width 0) (type default))
-  )
-  (wire (pts (xy 116.84 100.33) (xy 116.84 111.76))
-    (stroke (width 0) (type default))
-  )
   (wire (pts (xy 44.45 57.15) (xy 44.45 54.61))
     (stroke (width 0) (type default))
   )
-  (wire (pts (xy 172.72 54.61) (xy 166.37 54.61))
-    (stroke (width 0) (type default))
-  )
   (wire (pts (xy 104.14 90.17) (xy 116.84 90.17))
     (stroke (width 0) (type default))
@@
     (stroke (width 0) (type default))
   )
-  (wire (pts (xy 140.97 57.15) (xy 166.37 57.15))
+  (wire (pts (xy 140.97 57.15) (xy 172.72 57.15))
     (stroke (width 0) (type default))
   )
@@
     (stroke (width 0) (type default))
   )
-  (wire (pts (xy 157.48 95.25) (xy 157.48 111.76))
-    (stroke (width 0) (type default))
-  )
-  (wire (pts (xy 166.37 54.61) (xy 166.37 57.15))
-    (stroke (width 0) (type default))
-  )
   (wire (pts (xy 47.625 92.71) (xy 47.625 103.505))
     (stroke (width 0) (type default))
@@
     (stroke (width 0) (type default))
   )
-  (wire (pts (xy 115.57 54.61) (xy 115.57 57.15))
-    (stroke (width 0) (type default))
-  )
   (wire (pts (xy 170.18 124.46) (xy 170.18 127))
     (stroke (width 0) (type default))
@@
     (stroke (width 0) (type default))
   )
-  (wire (pts (xy 104.14 54.61) (xy 115.57 54.61))
+  (wire (pts (xy 104.14 57.15) (xy 121.92 57.15))
     (stroke (width 0) (type default))
   )
@@
     (stroke (width 0) (type default))
   )
-  (wire (pts (xy 157.48 111.76) (xy 157.48 124.46))
+  (wire (pts (xy 157.48 95.25) (xy 157.48 124.46))
     (stroke (width 0) (type default))
   )
@@
     (effects (font (size 1.27 1.27)) (justify right))
   )
-  (hierarchical_label "L-" (shape input) (at 87.63 59.69 180) (fields_autoplaced)
-    (effects (font (size 1.27 1.27)) (justify right))
-  )
-  (hierarchical_label "R+" (shape input) (at 87.63 67.31 180) (fields_autoplaced)
+  (hierarchical_label "L-" (shape input) (at 87.63 60.325 180) (fields_autoplaced)
+    (effects (font (size 1.27 1.27)) (justify right))
+  )
+  (hierarchical_label "R+" (shape input) (at 87.63 67.945 180) (fields_autoplaced)
     (effects (font (size 1.27 1.27)) (justify right))
   )
@@
     (effects (font (size 1.27 1.27)) (justify right))
   )
-  (hierarchical_label "QSE_EN" (shape input) (at 87.63 71.12 180) (fields_autoplaced)
+  (hierarchical_label "QSE_EN" (shape input) (at 87.63 71.755 180) (fields_autoplaced)
     (effects (font (size 1.27 1.27)) (justify right))
   )
@@
     (effects (font (size 1.27 1.27)) (justify right))
   )
-  (hierarchical_label "R-" (shape input) (at 87.63 64.77 180) (fields_autoplaced)
-    (effects (font (size 1.27 1.27)) (justify right))
-  )
-  (hierarchical_label "L+" (shape input) (at 87.63 62.23 180) (fields_autoplaced)
+  (hierarchical_label "R-" (shape input) (at 87.63 65.405 180) (fields_autoplaced)
+    (effects (font (size 1.27 1.27)) (justify right))
+  )
+  (hierarchical_label "L+" (shape input) (at 87.63 62.865 180) (fields_autoplaced)
     (effects (font (size 1.27 1.27)) (justify right))
   )
@@
     )
   )
+  (symbol (lib_id "power:GND") (at 116.84 100.33 0) (unit 1)
+    (in_bom yes) (on_board yes) (dnp no) (fields_autoplaced)
+    (property "Reference" "#PWR0105" (at 116.84 106.68 0)
+      (effects (font (size 1.27 1.27)) hide)
+    )
+    (property "Value" "GND" (at 116.84 105.41 0)
+      (effects (font (size 1.27 1.27)))
+    )
+    (property "Footprint" "" (at 116.84 100.33 0)
+      (effects (font (size 1.27 1.27)) hide)
+    )
+    (property "Datasheet" "" (at 116.84 100.33 0)
+      (effects (font (size 1.27 1.27)) hide)
+    )
+    (pin "1")
+    (instances
+      (project "main"
+        (path "/cb08c644-d155-44e5-86e1-31645eace055/f348e705-e1f2-401a-94bd-812b815f83a8"
+          (reference "#PWR0105") (unit 1)
+        )
+      )
+    )
+  )
   (symbol (lib_id "Device:C") (at 44.45 60.96 0) (mirror x) (unit 1)
     (in_bom yes) (on_board yes) (dnp no) (fields_autoplaced)
@@
     )
   )
-  (sheet (at 87.63 49.53) (size 16.51 24.13) (fields_autoplaced)
+  (sheet (at 87.63 49.53) (size 16.51 24.765) (fields_autoplaced)
     (stroke (width 0.1524) (type solid))
     (fill (color 0 0 0 0.0000))
@@
       (effects (font (size 1.27 1.27)) (justify left bottom))
     )
-    (property "Sheetfile" "modulator.kicad_sch" (at 87.63 74.2446 0)
+    (property "Sheetfile" "modulator.kicad_sch" (at 87.63 74.8796 0)
       (effects (font (size 1.27 1.27)) (justify left top))
     )
-    (pin "QSE_EN" input (at 87.63 71.12 180)
+    (pin "QSE_EN" input (at 87.63 71.755 180)
       (effects (font (size 1.27 1.27)) (justify left))
     )
@@
       (effects (font (size 1.27 1.27)) (justify right))
     )
-    (pin "SDR_POS" output (at 104.14 54.61 0)
-      (effects (font (size 1.27 1.27)) (justify right))
-    )
-    (pin "VOUTR_POS" input (at 87.63 67.31 180)
-      (effects (font (size 1.27 1.27)) (justify left))
-    )
-    (pin "VOUTL_POS" input (at 87.63 62.23 180)
-      (effects (font (size 1.27 1.27)) (justify left))
-    )
-    (pin "VOUTR_NEG" input (at 87.63 64.77 180)
-      (effects (font (size 1.27 1.27)) (justify left))
-    )
-    (pin "VOUTL_NEG" input (at 87.63 59.69 180)
+    (pin "SDR_POS" output (at 104.14 57.15 0)
+      (effects (font (size 1.27 1.27)) (justify right))
+    )
+    (pin "VOUTR_POS" input (at 87.63 67.945 180)
+      (effects (font (size 1.27 1.27)) (justify left))
+    )
+    (pin "VOUTL_POS" input (at 87.63 62.865 180)
+      (effects (font (size 1.27 1.27)) (justify left))
+    )
+    (pin "VOUTR_NEG" input (at 87.63 65.405 180)
+      (effects (font (size 1.27 1.27)) (justify left))
+    )
+    (pin "VOUTL_NEG" input (at 87.63 60.325 180)
       (effects (font (size 1.27 1.27)) (justify left))
     )
@@
       (effects (font (size 1.27 1.27)) (justify left top))
     )
-    (pin "SDR_POS" input (at 172.72 54.61 180)
-      (effects (font (size 1.27 1.27)) (justify left))
-    )
+    (pin "SDR_POS" input (at 172.72 57.15 180)
+      (effects (font (size 1.27 1.27)) (justify left))
+    )

Commit message: capacitor added to ant bias
Parts:
- added C38: 10uF, symbol Device:C
Connections:
- net GND: now also C38.1
- net at C63.2, R1.1, R1.1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: now also C38.2
Other:
- moved on the sheet: C38, R1, TR1

Commit message: Amplifier added to circuit
Parts:
- removed C38: 10uF, symbol Device:C
- removed C63, C65: 100nF, symbol Device:C
- removed R1: 100k, symbol Device:R
- removed R1 (x2): 2.2k, symbol Device:R
- added C38: 100n, symbol Device:C
- added C38: 10n, symbol Device:C
- added L1: ~, symbol Device:L
- added Q10: 2N7002, Package_TO_SOT_SMD:SOT-23, symbol Transistor_FET:2N7002
Connections:
- net Filter selector/filter_in: now also Q10.2 (S)
- net GND: now also C38.1
- net QSD_EN: now also L1.1
- new net: C38.2, L1.2, Q10.1 (G)
- new net: C38.1, Q10.3 (D)
- new net Power Amplifier/out: C38.2
Other:
- added sheet Power Amplifier (transmitter.kicad_sch)
- note removed: "TODO: Зачем здесь нужны эти резисторы?"
- moved on the sheet: C38, R1, TR1

Commit message: inductor TODO added, PDF updated
Parts:
- L1: value ~ -> 0
Other:
- note added: "TODO: В peaberry/SchematicV2.pdf есть эта индуктивность, зачем она не ясно"
Changed lines of the file:
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@@
     (stroke (width 0) (type default))
+  )
+  (text "TODO: В peaberry/SchematicV2.pdf есть\nэта индуктивность, зачем она не ясно"
+    (at 53.34 59.055 0)
+    (effects (font (size 1.27 1.27)) (justify right bottom))
   )
   (label "SDR_NEG" (at 168.275 117.475 0) (fields_autoplaced)
@@
   (symbol (lib_id "Device:L") (at 58.42 55.88 0) (mirror y) (unit 1)
     (in_bom yes) (on_board yes) (dnp no) (fields_autoplaced)
-    (property "Reference" "L1" (at 57.15 55.88 0)
+    (property "Reference" "L1" (at 57.15 54.61 0)
       (effects (font (size 1.27 1.27)) (justify left))
     )
-    (property "Value" "~" (at 57.15 57.15 0)
+    (property "Value" "0" (at 57.15 57.15 0)
       (effects (font (size 1.27 1.27)) (justify left))
     )

Commit message: 30 MHz output LPF added
Connections:
- net Power Amplifier/out renamed 30 MHz LPF/lpf1
Other:
- added sheet 30 MHz LPF (30MHz_LPF.kicad_sch)
Changed lines of the file:
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@@
     (stroke (width 0) (type default))
   )
-  (wire (pts (xy 99.06 45.72) (xy 102.235 45.72))
+  (wire (pts (xy 129.54 45.72) (xy 132.715 45.72))
     (stroke (width 0) (type default))
   )
@@
     (stroke (width 0) (type default))
   )
+  (wire (pts (xy 99.695 43.18) (xy 116.84 43.18))
+    (stroke (width 0) (type default))
+  )
   (wire (pts (xy 128.27 88.9) (xy 130.81 88.9))
     (stroke (width 0) (type default))
@@
     (stroke (width 0) (type default))
   )
-  (wire (pts (xy 81.915 43.18) (xy 86.36 43.18))
+  (wire (pts (xy 81.915 43.18) (xy 86.995 43.18))
     (stroke (width 0) (type default))
   )
@@
     (stroke (width 0) (type default))
   )
-  (wire (pts (xy 99.06 48.26) (xy 102.235 48.26))
+  (wire (pts (xy 129.54 48.26) (xy 132.715 48.26))
     (stroke (width 0) (type default))
   )
@@
     (effects (font (size 1.27 1.27)) (justify left))
   )
-  (hierarchical_label "swr_rvs" (shape output) (at 102.235 48.26 0) (fields_autoplaced)
+  (hierarchical_label "swr_rvs" (shape output) (at 132.715 48.26 0) (fields_autoplaced)
     (effects (font (size 1.27 1.27)) (justify left))
   )
@@
     (effects (font (size 1.27 1.27)) (justify right))
   )
-  (hierarchical_label "swr_fwd" (shape output) (at 102.235 45.72 0) (fields_autoplaced)
+  (hierarchical_label "swr_fwd" (shape output) (at 132.715 45.72 0) (fields_autoplaced)
     (effects (font (size 1.27 1.27)) (justify left))
   )
@@
     )
   )
+  (sheet (at 86.995 41.275) (size 12.7 3.81) (fields_autoplaced)
+    (stroke (width 0.1524) (type solid))
+    (fill (color 0 0 0 0.0000))
+    (property "Sheetname" "30 MHz LPF" (at 86.995 40.5634 0)
+      (effects (font (size 1.27 1.27)) (justify left bottom))
+    )
+    (property "Sheetfile" "30MHz_LPF.kicad_sch" (at 86.995 45.6696 0)
+      (effects (font (size 1.27 1.27)) (justify left top))
+    )
+    (pin "lpf1" bidirectional (at 86.995 43.18 180)
+      (effects (font (size 1.27 1.27)) (justify left))
+    )
+    (pin "lpf2" bidirectional (at 99.695 43.18 0)
+      (effects (font (size 1.27 1.27)) (justify right))
+    )
+    (instances
+      (project "main"
+        (path "/cb08c644-d155-44e5-86e1-31645eace055/f348e705-e1f2-401a-94bd-812b815f83a8" (page "14"))
+      )
+    )
+  )
   (sheet (at 123.19 106.045) (size 19.685 8.89)
     (stroke (width 0.1524) (type solid))
@@
     )
   )
-  (sheet (at 86.36 41.275) (size 12.7 8.89) (fields_autoplaced)
+  (sheet (at 116.84 41.275) (size 12.7 8.89) (fields_autoplaced)
     (stroke (width 0.1524) (type solid))
     (fill (color 0 0 0 0.0000))
-    (property "Sheetname" "Power SWR Bridge" (at 86.36 40.5634 0)
+    (property "Sheetname" "Power SWR Bridge" (at 116.84 40.5634 0)
       (effects (font (size 1.27 1.27)) (justify left bottom))
     )
-    (property "Sheetfile" "power_swr_bridge.kicad_sch" (at 86.36 50.7496 0)
+    (property "Sheetfile" "power_swr_bridge.kicad_sch" (at 116.84 50.7496 0)
       (effects (font (size 1.27 1.27)) (justify left top))
     )
-    (pin "rvs" output (at 99.06 48.26 0)
-      (effects (font (size 1.27 1.27)) (justify right))
-    )
-    (pin "fwd" output (at 99.06 45.72 0)
-      (effects (font (size 1.27 1.27)) (justify right))
-    )
-    (pin "ANT" passive (at 86.36 43.18 180)
-      (effects (font (size 1.27 1.27)) (justify left))
-    )
+    (pin "rvs" output (at 129.54 48.26 0)
+      (effects (font (size 1.27 1.27)) (justify right))
+    )
+    (pin "fwd" output (at 129.54 45.72 0)
+      (effects (font (size 1.27 1.27)) (justify right))
+    )
+    (pin "ANT" passive (at 116.84 43.18 180)
+      (effects (font (size 1.27 1.27)) (justify left))
+    )

Commit message: QSD_EN->RX_EN, QSE_EN->TX_EN, FIXME removed
Connections:
- net QSD_EN renamed RX_EN
Other:
- sheet Mixer (Detector) ports: added ENABLE; removed QSD_EN
- sheet Modulator ports: added ENABLE; removed QSE_EN
Changed lines of the file:
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@@
     (effects (font (size 1.27 1.27)) (justify right))
   )
-  (hierarchical_label "QSD_EN" (shape input) (at 57.15 48.895 180) (fields_autoplaced)
+  (hierarchical_label "RX_EN" (shape input) (at 57.15 48.895 180) (fields_autoplaced)
     (effects (font (size 1.27 1.27)) (justify right))
   )
@@
     (effects (font (size 1.27 1.27)) (justify right))
   )
-  (hierarchical_label "QSE_EN" (shape input) (at 79.375 86.36 180) (fields_autoplaced)
+  (hierarchical_label "TX_EN" (shape input) (at 79.375 86.36 180) (fields_autoplaced)
     (effects (font (size 1.27 1.27)) (justify right))
   )
@@
     (effects (font (size 1.27 1.27)) (justify right))
   )
-  (hierarchical_label "QSD_EN" (shape input) (at 211.455 84.455 180) (fields_autoplaced)
+  (hierarchical_label "RX_EN" (shape input) (at 211.455 84.455 180) (fields_autoplaced)
     (effects (font (size 1.27 1.27)) (justify right))
   )
@@
       (effects (font (size 1.27 1.27)) (justify left top))
     )
-    (pin "QSE_EN" input (at 130.81 88.9 180)
-      (effects (font (size 1.27 1.27)) (justify left))
-    )
     (pin "f0" input (at 130.81 69.215 180)
       (effects (font (size 1.27 1.27)) (justify left))
@@
     )
     (pin "VOUTL_NEG" input (at 130.81 77.47 180)
+      (effects (font (size 1.27 1.27)) (justify left))
+    )
+    (pin "ENABLE" input (at 130.81 88.9 180)
       (effects (font (size 1.27 1.27)) (justify left))
     )
@@
       (effects (font (size 1.27 1.27)) (justify left))
     )
-    (pin "QSD_EN" input (at 211.455 84.455 180)
-      (effects (font (size 1.27 1.27)) (justify left))
-    )
     (pin "f0" input (at 211.455 78.105 180)
       (effects (font (size 1.27 1.27)) (justify left))
@@
       (effects (font (size 1.27 1.27)) (justify right))
     )
-    (instances
+    (pin "ENABLE" input (at 211.455 84.455 180)
+      (effects (font (size 1.27 1.27)) (justify left))
+    )
+    (instances
