File: main/filter_selector.kicad_sch (KiCad schematic)
At the start: 13 parts, among them J7 Conn_Coaxial, U7 74CBTLV3253PW

Commit message: filter selector: elements number assigned as in original circuit
Parts:
- renumbered C58 to C59, C23 to C63
Changed lines of the file:
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@@
   (symbol (lib_id "Device:C") (at 143.51 62.23 0) (unit 1)
     (in_bom yes) (on_board yes) (dnp no) (fields_autoplaced)
-    (property "Reference" "C58" (at 147.32 60.96 0)
+    (property "Reference" "C59" (at 147.32 60.96 0)
       (effects (font (size 1.27 1.27)) (justify left))
     )
@@
   (symbol (lib_id "power:+3.3V") (at 138.43 55.88 0) (unit 1)
     (in_bom yes) (on_board yes) (dnp no) (fields_autoplaced)
-    (property "Reference" "#PWR059" (at 138.43 59.69 0)
+    (property "Reference" "#PWR066" (at 138.43 59.69 0)
       (effects (font (size 1.27 1.27)) hide)
     )
@@
   (symbol (lib_id "power:+3.3V") (at 97.79 114.3 0) (unit 1)
     (in_bom yes) (on_board yes) (dnp no) (fields_autoplaced)
-    (property "Reference" "#PWR066" (at 97.79 118.11 0)
+    (property "Reference" "#PWR063" (at 97.79 118.11 0)
       (effects (font (size 1.27 1.27)) hide)
     )
@@
   (symbol (lib_id "Device:C") (at 90.17 130.81 0) (mirror x) (unit 1)
     (in_bom yes) (on_board yes) (dnp no)
-    (property "Reference" "C23" (at 86.36 129.54 0)
+    (property "Reference" "C63" (at 86.36 129.54 0)
       (effects (font (size 1.27 1.27)) (justify right))
     )
@@
   (symbol (lib_id "power:+3.3V") (at 97.79 44.45 0) (unit 1)
     (in_bom yes) (on_board yes) (dnp no) (fields_autoplaced)
-    (property "Reference" "#PWR065" (at 97.79 48.26 0)
-      (effects (font (size 1.27 1.27)) hide)
-    )
+    (property "Reference" "#PWR061" (at 97.79 48.26 0)
+      (effects (font (size 1.27 1.27)) hide)
+    )

Commit message: R37 bias supply removed
Parts:
- removed C64, C66: 100nF, symbol Device:C
- removed R1: 100k, symbol Device:R
- removed R1 (x2): 2.2k, symbol Device:R
Connections:
- net filtered: now also U7.7 (1A)
Other:
- note removed: "TODO: Probably, this circuit isn't necessary"

Commit message: Power SWR Bridge used as input ANT connection
Parts:
- removed C63, C65: 100nF, symbol Device:C
- removed J7: Conn_Coaxial, symbol Connector:Conn_Coaxial
- removed R1 (x2): 2.2k, symbol Device:R
- removed R1: 100k, symbol Device:R
Connections:
- net filter_in: now reaches U7.9 (2A)

Commit message: Amplifier added to circuit
Parts:
- added C63, C65: 100nF, symbol Device:C
- added R1 (x4): 2.2k, symbol Device:R
- added R1 (x2): 100k, symbol Device:R
Connections:
- net +3.3V: now also R1.1, R1.1
- net GND: now also C63.1, C65.1, R1.2, R1.2
- net filter_in: now also R1.1
- net filtered: now also R1.2
- new net: C63.2, R1.1, R1.2, R1.2
- new net: C65.2, R1.1, R1.1, R1.2
