File: main/transmitter.kicad_sch (KiCad schematic)
At the start: 35 parts, among them Q1 PZT2222A, Q2 BS170, Q3 BS170, Q4 BS170, Q5 BS170, Q6 MMBT3904, Q7 BSS84, Q8 BS170, Q9 MMBT3904

Commit message: Amplifier added to circuit
Other:
- note added: "TODO: Может не нужно устанавливать или это тонкая подстройка?"
Changed lines of the file:
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@@
     (effects (font (size 2.5 2.5)) (justify left bottom))
+  )
+  (text "TODO: Может не нужно устанавливать\nили это тонкая подстройка?"
+    (at 76.2 104.14 0)
+    (effects (font (size 1.27 1.27)) (justify left bottom))
   )
   (text "Здесь можно использовать любые транзисторы" (at 55.245 120.015 0)
