File: main/power_swr_bridge.kicad_sch (KiCad schematic)
At the start: 15 parts, among them J7 Conn_Coaxial

Commit message: swr bridge mirrored for better look
Other:
- moved on the sheet: C61, C62, C64, C66, D4, D5, J7, L14, L15, R4, R5, R6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

Commit message: SWR bridge: TODO comment added, PDF updated
Other:
- note added: "From (tr)uSDX RF board"
- note added: "TODO: Мощные компоненты! Уточнить при назначении посадочных мест!"
Changed lines of the file:
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@@
     (stroke (width 0) (type default))
+  )
+  (text "TODO: Мощные компоненты!\nУточнить при назначении посадочных мест!"
+    (at 131.445 45.72 0)
+    (effects (font (size 1.27 1.27)) (justify left bottom))
+  )
+  (text "From (tr)uSDX RF board" (at 129.54 23.495 0)
+    (effects (font (size 2.5 2.5)) (justify left bottom))
   )
   (label "ANT_OUT" (at 95.25 113.665 180) (fields_autoplaced)

Commit message: SWR meter: comments added
Other:
- note added: ""Stockton bridge" from (tr)uSDX RF board"
- note added: "TODO: Для точности можно использовать сдвоенное кольцо ("бинокль")"
- note removed: "From (tr)uSDX RF board"
Changed lines of the file:
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@@
     (stroke (width 0) (type default))
+  )
+  (text "TODO: Для точности можно использовать\nсдвоенное кольцо (\"бинокль\")"
+    (at 67.31 83.82 0)
+    (effects (font (size 1.27 1.27)) (justify left bottom))
   )
   (text "TODO: Мощные компоненты!\nУточнить при назначении посадочных мест!"
@@
     (effects (font (size 1.27 1.27)) (justify left bottom))
   )
-  (text "From (tr)uSDX RF board" (at 129.54 23.495 0)
+  (text "\"Stockton bridge\"\nfrom (tr)uSDX RF board" (at 129.54 23.495 0)
     (effects (font (size 2.5 2.5)) (justify left bottom))
   )

Commit message: SWR meter: TODO removed
Other:
- note removed: "TODO: Мощные компоненты! Уточнить при назначении посадочных мест!"
Changed lines of the file:
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@@
-    (effects (font (size 1.27 1.27)) (justify left bottom))
-  )
-  (text "TODO: Мощные компоненты!\nУточнить при назначении посадочных мест!"
-    (at 131.445 45.72 0)
     (effects (font (size 1.27 1.27)) (justify left bottom))
   )

Commit message: SWR meter: inductors added, PDF updated
Parts:
- added L1 (x2): 47uH, symbol Device:L
Connections:
- net fwd: now also L1.1; no longer C64.1, R7.1
- net rvs: now also L1.1; no longer C61.1, R4.1
- new net: C61.1, L1.2, R4.1
- new net: C64.1, L1.2, R7.1
Changed lines of the file:
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@@
+    (stroke (width 0) (type default))
+  )
+  (wire (pts (xy 182.88 85.09) (xy 176.53 85.09))
     (stroke (width 0) (type default))
   )
@@
     (stroke (width 0) (type default))
   )
-  (wire (pts (xy 184.15 65.405) (xy 176.53 65.405))
+  (wire (pts (xy 182.88 65.405) (xy 176.53 65.405))
+    (stroke (width 0) (type default))
+  )
+  (wire (pts (xy 193.675 65.405) (xy 190.5 65.405))
     (stroke (width 0) (type default))
   )
@@
     (stroke (width 0) (type default))
   )
-  (wire (pts (xy 184.15 85.09) (xy 176.53 85.09))
+  (wire (pts (xy 193.675 85.09) (xy 190.5 85.09))
     (stroke (width 0) (type default))
   )
@@
     (effects (font (size 1.27 1.27)) (justify right))
   )
-  (hierarchical_label "rvs" (shape output) (at 184.15 85.09 0) (fields_autoplaced)
+  (hierarchical_label "rvs" (shape output) (at 193.675 85.09 0) (fields_autoplaced)
     (effects (font (size 1.27 1.27)) (justify left))
   )
-  (hierarchical_label "fwd" (shape output) (at 184.15 65.405 0) (fields_autoplaced)
+  (hierarchical_label "fwd" (shape output) (at 193.675 65.405 0) (fields_autoplaced)
     (effects (font (size 1.27 1.27)) (justify left))
   )
@@
     )
   )
-  (symbol (lib_id "Device:C") (at 176.53 93.98 0) (mirror y) (unit 1)
-    (in_bom yes) (on_board yes) (dnp no) (fields_autoplaced)
-    (property "Reference" "C61" (at 173.355 92.71 0)
-      (effects (font (size 1.27 1.27)) (justify left))
-    )
-    (property "Value" "10n" (at 173.355 95.25 0)
-      (effects (font (size 1.27 1.27)) (justify left))
-    )
-    (property "Footprint" "" (at 175.5648 97.79 0)
+  (symbol (lib_id "Device:C") (at 176.53 93.98 0) (unit 1)
+    (in_bom yes) (on_board yes) (dnp no)
+    (property "Reference" "C61" (at 179.705 92.71 0)
+      (effects (font (size 1.27 1.27)) (justify left))
+    )
+    (property "Value" "10n" (at 179.705 95.25 0)
+      (effects (font (size 1.27 1.27)) (justify left))
+    )
+    (property "Footprint" "" (at 177.4952 97.79 0)
       (effects (font (size 1.27 1.27)) hide)
     )
@@
     )
   )
+  (symbol (lib_id "Device:L") (at 186.69 65.405 270) (mirror x) (unit 1)
+    (in_bom yes) (on_board yes) (dnp no) (fields_autoplaced)
+    (property "Reference" "L1" (at 186.69 59.69 90)
+      (effects (font (size 1.27 1.27)))
+    )
+    (property "Value" "47uH" (at 186.69 62.23 90)
+      (effects (font (size 1.27 1.27)))
+    )
+    (property "Footprint" "" (at 186.69 65.405 0)
+      (effects (font (size 1.27 1.27)) hide)
+    )
+    (property "Datasheet" "~" (at 186.69 65.405 0)
+      (effects (font (size 1.27 1.27)) hide)
+    )
+    (pin "1")
+    (pin "2")
+    (instances
+      (project "main"
+        (path "/cb08c644-d155-44e5-86e1-31645eace055"
+          (reference "L1") (unit 1)
+        )
+        (path "/cb08c644-d155-44e5-86e1-31645eace055/f348e705-e1f2-401a-94bd-812b815f83a8/83cdc139-f19f-4702-871a-4a75f5a0616b"
+          (reference "L16") (unit 1)
+        )
+        (path "/cb08c644-d155-44e5-86e1-31645eace055/f348e705-e1f2-401a-94bd-812b815f83a8"
+          (reference "L17") (unit 1)
+        )
+        (path "/cb08c644-d155-44e5-86e1-31645eace055/f348e705-e1f2-401a-94bd-812b815f83a8/8653829a-ea60-4c18-8b01-1eb920d43d9e"
+          (reference "L18") (unit 1)
+        )
+      )
+    )
+  )
+  (symbol (lib_id "Device:L") (at 186.69 85.09 270) (mirror x) (unit 1)
+    (in_bom yes) (on_board yes) (dnp no) (fields_autoplaced)
+    (property "Reference" "L1" (at 186.69 79.375 90)
+      (effects (font (size 1.27 1.27)))
+    )
+    (property "Value" "47uH" (at 186.69 81.915 90)
+      (effects (font (size 1.27 1.27)))
+    )
+    (property "Footprint" "" (at 186.69 85.09 0)
+      (effects (font (size 1.27 1.27)) hide)
+    )
+    (property "Datasheet" "~" (at 186.69 85.09 0)
+      (effects (font (size 1.27 1.27)) hide)
+    )
+    (pin "1")
+    (pin "2")
+    (instances
+      (project "main"
+        (path "/cb08c644-d155-44e5-86e1-31645eace055"
+          (reference "L1") (unit 1)
+        )
+        (path "/cb08c644-d155-44e5-86e1-31645eace055/f348e705-e1f2-401a-94bd-812b815f83a8/83cdc139-f19f-4702-871a-4a75f5a0616b"
+          (reference "L16") (unit 1)
+        )
+        (path "/cb08c644-d155-44e5-86e1-31645eace055/f348e705-e1f2-401a-94bd-812b815f83a8"
+          (reference "L17") (unit 1)
+        )
+        (path "/cb08c644-d155-44e5-86e1-31645eace055/f348e705-e1f2-401a-94bd-812b815f83a8/8653829a-ea60-4c18-8b01-1eb920d43d9e"
+          (reference "L19") (unit 1)
+        )
+      )
+    )
+  )
   (symbol (lib_id "Device:C") (at 176.53 56.515 180) (unit 1)
     (in_bom yes) (on_board yes) (dnp no) (fields_autoplaced)
@@
     )
   )
-  (symbol (lib_id "Device:C") (at 163.195 93.98 0) (mirror y) (unit 1)
-    (in_bom yes) (on_board yes) (dnp no) (fields_autoplaced)
-    (property "Reference" "C62" (at 159.385 92.71 0)
-      (effects (font (size 1.27 1.27)) (justify left))
-    )
-    (property "Value" "10n" (at 159.385 95.25 0)
-      (effects (font (size 1.27 1.27)) (justify left))
-    )
-    (property "Footprint" "" (at 162.2298 97.79 0)
-      (effects (font (size 1.27 1.27)) hide)
-    )
+  (symbol (lib_id "Device:C") (at 163.195 93.98 0) (unit 1)
+    (in_bom yes) (on_board yes) (dnp no)
+    (property "Reference" "C62" (at 167.005 92.71 0)
+      (effects (font (size 1.27 1.27)) (justify left))
+    )
+    (property "Value" "10n" (at 167.005 95.25 0)
+      (effects (font (size 1.27 1.27)) (justify left))
+    )
+    (property "Footprint" "" (at 164.1602 97.79 0)
+      (effects (font (size 1.27 1.27)) hide)
+    )

Commit message: SWR meter TODO additions
Other:
- note added: "TODO: Для точности можно использовать сдвоенное кольцо ("бинокль") Amidon BN61-202"
- note removed: "TODO: Для точности можно использовать сдвоенное кольцо ("бинокль")"
Changed lines of the file:
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@@
     (stroke (width 0) (type default))
   )
-  (text "TODO: Для точности можно использовать\nсдвоенное кольцо (\"бинокль\")"
-    (at 67.31 83.82 0)
+  (text "TODO: Для точности можно использовать\nсдвоенное кольцо (\"бинокль\") Amidon BN61-202"
+    (at 65.405 81.28 0)
     (effects (font (size 1.27 1.27)) (justify left bottom))
   )

Commit message: SWR meter circuit updated
Parts:
- removed C61, C62, C64, C66: 10n, symbol Device:C
- removed D4, D5: 1N4148W, Diode_SMD:D_SOD-123, symbol Diode:1N4148W
- removed L1 (x2): 47uH, symbol Device:L
- removed L14: 1:7 ratio, symbol Device:L_Ferrite_Coupled
- removed L15: 3:21 ratio, symbol Device:L_Ferrite_Coupled
- removed R4, R7: 68k, symbol Device:R
- removed R5, R6, R8, R9: 100, symbol Device:R
- added C? (x2): 0.1u, Capacitor_SMD:C_0805_2012Metric_Pad1.15x1.40mm_HandSolder, symbol Device:C
- added C? (x2): 0.01u, Capacitor_SMD:C_0805_2012Metric_Pad1.15x1.40mm_HandSolder, symbol Device:C
- added D4, D5: 1N34/D311/1N4148W, symbol Device:D
- added L1, L2: 1000u, Diode_THT:D_DO-41_SOD81_P2.54mm_Vertical_AnodeUp, symbol Device:L
- added L25: 1:7 ratio, symbol Device:L_Ferrite_Coupled
- added L26: 3:21 ratio, symbol Device:L_Ferrite_Coupled
- added R? (x4): 100, Resistor_SMD:R_0805_2012Metric_Pad1.15x1.40mm_HandSolder, symbol Device:R
- added R? (x2): 300, Resistor_SMD:R_0805_2012Metric_Pad1.15x1.40mm_HandSolder, symbol Device:R
- added R? (x2): 680, Resistor_SMD:R_0805_2012Metric_Pad1.15x1.40mm_HandSolder, symbol Device:R
Connections:
- net ANT: now also L25.1, L26.3
- net ANT_OUT: now also L25.2
- net GND: now also C?.2, C?.2, C?.2, C?.2, L25.3, L26.4, R?.2, R?.2, R?.2, R?.2, R?.2, R?.2
- net fwd: now also C?.1, R?.1, R?.2
- net rvs: now also C?.1, R?.1, R?.2
- new net: C?.1, D4.1 (K), L1.2
- new net: D4.2 (A), L25.4, L26.1, R?.1, R?.1
- new net: D5.2 (A), L26.2, R?.1, R?.1
- new net: L2.1, R?.1
- new net: C?.1, D5.1 (K), L2.2
- new net: L1.1, R?.1
Other:
- note added: ""Stockton bridge" copied from AYN/4B («All You Need / 4 Bands») - Aleksander Alekseev's Portable QRP CW Transceiver"
- note added: "BN61-202"
- note added: "Tandem match / Stockton bridge @ BN61-202 Primary windings: RG-174 coax cable Secondary windings: enameled copper wire Fore more details see: https://eax.me/stockton-bridge/ Windings ratio is copied from (tr)uSDX. (FIXME: I don't know how to wind 3T of RG-174 cable)"
- note added: "The SWR bridge works as a static bleeder too. For DC “ANT” is shorted to ground."
- note added: "The diodes should be matched by the voltage drop. Germanium is preferred."
- note removed: ""Stockton bridge" from (tr)uSDX RF board"
- note removed: "TODO: Для точности можно использовать сдвоенное кольцо ("бинокль") Amidon BN61-202"
- moved on the sheet: J7

Commit message: SWR symbols reference numbers reassigned
Parts:
- renumbered L25 to L14, L26 to L15
Changed lines of the file:
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@@
       (project "main"
         (path "/cb08c644-d155-44e5-86e1-31645eace055/f348e705-e1f2-401a-94bd-812b815f83a8/8653829a-ea60-4c18-8b01-1eb920d43d9e"
-          (reference "D6") (unit 1)
+          (reference "D5") (unit 1)
         )
       )
@@
       (project "main"
         (path "/cb08c644-d155-44e5-86e1-31645eace055/f348e705-e1f2-401a-94bd-812b815f83a8/8653829a-ea60-4c18-8b01-1eb920d43d9e"
-          (reference "#PWR0145") (unit 1)
+          (reference "#PWR061") (unit 1)
         )
       )
@@
       (project "main"
         (path "/cb08c644-d155-44e5-86e1-31645eace055/f348e705-e1f2-401a-94bd-812b815f83a8/8653829a-ea60-4c18-8b01-1eb920d43d9e"
-          (reference "R61") (unit 1)
+          (reference "R6") (unit 1)
         )
       )
@@
   (symbol (lib_id "power:GND") (at 100.965 67.31 0) (mirror y) (unit 1)
     (in_bom yes) (on_board yes) (dnp no) (fields_autoplaced)
-    (property "Reference" "#PWR0148" (at 100.965 73.66 0)
+    (property "Reference" "#PWR062" (at 100.965 73.66 0)
       (effects (font (size 1.27 1.27)) hide)
     )
@@
       (project "main"
         (path "/cb08c644-d155-44e5-86e1-31645eace055/f348e705-e1f2-401a-94bd-812b815f83a8/8653829a-ea60-4c18-8b01-1eb920d43d9e"
-          (reference "#PWR0148") (unit 1)
+          (reference "#PWR062") (unit 1)
         )
       )
@@
       (project "main"
         (path "/cb08c644-d155-44e5-86e1-31645eace055/f348e705-e1f2-401a-94bd-812b815f83a8/8653829a-ea60-4c18-8b01-1eb920d43d9e"
-          (reference "#PWR0140") (unit 1)
+          (reference "#PWR0139") (unit 1)
         )
       )
@@
       (project "main"
         (path "/cb08c644-d155-44e5-86e1-31645eace055/f348e705-e1f2-401a-94bd-812b815f83a8/8653829a-ea60-4c18-8b01-1eb920d43d9e"
-          (reference "#PWR0143") (unit 1)
+          (reference "#PWR0135") (unit 1)
         )
       )
@@
       (project "main"
         (path "/cb08c644-d155-44e5-86e1-31645eace055/f348e705-e1f2-401a-94bd-812b815f83a8/8653829a-ea60-4c18-8b01-1eb920d43d9e"
-          (reference "L23") (unit 1)
+          (reference "L18") (unit 1)
         )
       )
@@
       (project "main"
         (path "/cb08c644-d155-44e5-86e1-31645eace055/f348e705-e1f2-401a-94bd-812b815f83a8/8653829a-ea60-4c18-8b01-1eb920d43d9e"
-          (reference "#PWR0134") (unit 1)
+          (reference "#PWR0145") (unit 1)
         )
       )
@@
       (project "main"
         (path "/cb08c644-d155-44e5-86e1-31645eace055/f348e705-e1f2-401a-94bd-812b815f83a8/8653829a-ea60-4c18-8b01-1eb920d43d9e"
-          (reference "C31") (unit 1)
+          (reference "C32") (unit 1)
         )
       )
@@
   (symbol (lib_id "Device:L_Ferrite_Coupled") (at 111.125 64.77 0) (unit 1)
     (in_bom yes) (on_board yes) (dnp no) (fields_autoplaced)
-    (property "Reference" "L25" (at 110.871 56.515 0)
+    (property "Reference" "L14" (at 110.871 56.515 0)
       (effects (font (size 1.27 1.27)))
     )
@@
       (project "main"
         (path "/cb08c644-d155-44e5-86e1-31645eace055/f348e705-e1f2-401a-94bd-812b815f83a8/8653829a-ea60-4c18-8b01-1eb920d43d9e"
-          (reference "L25") (unit 1)
+          (reference "L14") (unit 1)
         )
       )
@@
       (project "main"
         (path "/cb08c644-d155-44e5-86e1-31645eace055/f348e705-e1f2-401a-94bd-812b815f83a8/8653829a-ea60-4c18-8b01-1eb920d43d9e"
-          (reference "L22") (unit 1)
+          (reference "L19") (unit 1)
         )
       )
@@
       (project "main"
         (path "/cb08c644-d155-44e5-86e1-31645eace055/f348e705-e1f2-401a-94bd-812b815f83a8/8653829a-ea60-4c18-8b01-1eb920d43d9e"
-          (reference "#PWR0142") (unit 1)
+          (reference "#PWR0136") (unit 1)
         )
       )
@@
       (project "main"
         (path "/cb08c644-d155-44e5-86e1-31645eace055/f348e705-e1f2-401a-94bd-812b815f83a8/8653829a-ea60-4c18-8b01-1eb920d43d9e"
-          (reference "C32") (unit 1)
+          (reference "C31") (unit 1)
         )
       )
@@
       (project "main"
         (path "/cb08c644-d155-44e5-86e1-31645eace055/f348e705-e1f2-401a-94bd-812b815f83a8/8653829a-ea60-4c18-8b01-1eb920d43d9e"
-          (reference "#PWR0147") (unit 1)
+          (reference "#PWR0134") (unit 1)
         )
       )
@@
       (project "main"
         (path "/cb08c644-d155-44e5-86e1-31645eace055/f348e705-e1f2-401a-94bd-812b815f83a8/8653829a-ea60-4c18-8b01-1eb920d43d9e"
-          (reference "R60") (unit 1)
+          (reference "R7") (unit 1)
         )
       )
@@
       (project "main"
         (path "/cb08c644-d155-44e5-86e1-31645eace055/f348e705-e1f2-401a-94bd-812b815f83a8/8653829a-ea60-4c18-8b01-1eb920d43d9e"
-          (reference "R58") (unit 1)
+          (reference "R8") (unit 1)
         )
       )
@@
       (project "main"
         (path "/cb08c644-d155-44e5-86e1-31645eace055/f348e705-e1f2-401a-94bd-812b815f83a8/8653829a-ea60-4c18-8b01-1eb920d43d9e"
-          (reference "#PWR0139") (unit 1)
+          (reference "#PWR0140") (unit 1)
         )
       )
@@
       (project "main"
         (path "/cb08c644-d155-44e5-86e1-31645eace055/f348e705-e1f2-401a-94bd-812b815f83a8/8653829a-ea60-4c18-8b01-1eb920d43d9e"
-          (reference "#PWR0136") (unit 1)
+          (reference "#PWR0143") (unit 1)
         )
       )
@@
       (project "main"
         (path "/cb08c644-d155-44e5-86e1-31645eace055/f348e705-e1f2-401a-94bd-812b815f83a8/8653829a-ea60-4c18-8b01-1eb920d43d9e"
-          (reference "C89") (unit 1)
+          (reference "C30") (unit 1)
         )
       )
@@
       (project "main"
         (path "/cb08c644-d155-44e5-86e1-31645eace055/f348e705-e1f2-401a-94bd-812b815f83a8/8653829a-ea60-4c18-8b01-1eb920d43d9e"
-          (reference "#PWR0137") (unit 1)
+          (reference "#PWR0142") (unit 1)
         )
       )
@@
       (project "main"
         (path "/cb08c644-d155-44e5-86e1-31645eace055/f348e705-e1f2-401a-94bd-812b815f83a8/8653829a-ea60-4c18-8b01-1eb920d43d9e"
-          (reference "#PWR0141") (unit 1)
+          (reference "#PWR0138") (unit 1)
         )
       )
@@
       (project "main"
         (path "/cb08c644-d155-44e5-86e1-31645eace055/f348e705-e1f2-401a-94bd-812b815f83a8/8653829a-ea60-4c18-8b01-1eb920d43d9e"
-          (reference "R62") (unit 1)
+          (reference "R5") (unit 1)
         )
       )
@@
   (symbol (lib_id "power:GND") (at 121.285 82.55 0) (mirror y) (unit 1)
     (in_bom yes) (on_board yes) (dnp no) (fields_autoplaced)
-    (property "Reference" "#PWR0149" (at 121.285 88.9 0)
+    (property "Reference" "#PWR069" (at 121.285 88.9 0)
       (effects (font (size 1.27 1.27)) hide)
     )
@@
       (project "main"
         (path "/cb08c644-d155-44e5-86e1-31645eace055/f348e705-e1f2-401a-94bd-812b815f83a8/8653829a-ea60-4c18-8b01-1eb920d43d9e"
-          (reference "#PWR0149") (unit 1)
+          (reference "#PWR069") (unit 1)
         )
       )
@@
       (project "main"
         (path "/cb08c644-d155-44e5-86e1-31645eace055/f348e705-e1f2-401a-94bd-812b815f83a8/8653829a-ea60-4c18-8b01-1eb920d43d9e"
-          (reference "R59") (unit 1)
+          (reference "R9") (unit 1)
         )
       )
@@
       (project "main"
         (path "/cb08c644-d155-44e5-86e1-31645eace055/f348e705-e1f2-401a-94bd-812b815f83a8/8653829a-ea60-4c18-8b01-1eb920d43d9e"
-          (reference "D7") (unit 1)
+          (reference "D4") (unit 1)
         )
       )
@@
       (project "main"
         (path "/cb08c644-d155-44e5-86e1-31645eace055/f348e705-e1f2-401a-94bd-812b815f83a8/8653829a-ea60-4c18-8b01-1eb920d43d9e"
-          (reference "R63") (unit 1)
+          (reference "R4") (unit 1)
         )
       )
@@
       (project "main"
         (path "/cb08c644-d155-44e5-86e1-31645eace055/f348e705-e1f2-401a-94bd-812b815f83a8/8653829a-ea60-4c18-8b01-1eb920d43d9e"
-          (reference "#PWR0138") (unit 1)
+          (reference "#PWR0141") (unit 1)
         )
       )
@@
   (symbol (lib_id "Device:L_Ferrite_Coupled") (at 111.125 85.09 0) (mirror x) (unit 1)
     (in_bom yes) (on_board yes) (dnp no)
-    (property "Reference" "L26" (at 111.125 76.835 0)
+    (property "Reference" "L15" (at 111.125 76.835 0)
       (effects (font (size 1.27 1.27)))
     )
@@
       (project "main"
         (path "/cb08c644-d155-44e5-86e1-31645eace055/f348e705-e1f2-401a-94bd-812b815f83a8/8653829a-ea60-4c18-8b01-1eb920d43d9e"
-          (reference "L26") (unit 1)
+          (reference "L15") (unit 1)
         )
       )
@@
       (project "main"
         (path "/cb08c644-d155-44e5-86e1-31645eace055/f348e705-e1f2-401a-94bd-812b815f83a8/8653829a-ea60-4c18-8b01-1eb920d43d9e"
-          (reference "#PWR0144") (unit 1)
+          (reference "#PWR059") (unit 1)
         )
       )
@@
       (project "main"
         (path "/cb08c644-d155-44e5-86e1-31645eace055/f348e705-e1f2-401a-94bd-812b815f83a8/8653829a-ea60-4c18-8b01-1eb920d43d9e"
-          (reference "C30") (unit 1)
+          (reference "C61") (unit 1)
         )
       )
@@
         )
         (path "/cb08c644-d155-44e5-86e1-31645eace055/f348e705-e1f2-401a-94bd-812b815f83a8/8653829a-ea60-4c18-8b01-1eb920d43d9e"
-          (reference "#PWR069") (unit 1)
+          (reference "#PWR0137") (unit 1)
         )
       )
@@
       (project "main"
         (path "/cb08c644-d155-44e5-86e1-31645eace055/f348e705-e1f2-401a-94bd-812b815f83a8/8653829a-ea60-4c18-8b01-1eb920d43d9e"
-          (reference "#PWR0146") (unit 1)
+          (reference "#PWR094") (unit 1)
         )
       )
@@
       (project "main"
         (path "/cb08c644-d155-44e5-86e1-31645eace055/f348e705-e1f2-401a-94bd-812b815f83a8/8653829a-ea60-4c18-8b01-1eb920d43d9e"
-          (reference "#PWR0135") (unit 1)
-        )
-      )
+          (reference "#PWR0144") (unit 1)
+        )
+      )
