File: main/power_swr_bridge.kicad_sch (KiCad schematic)
At the start: 19 parts, among them J7 Conn_Coaxial

Commit message: SWR meter phases fix
Connections:
- net ANT: no longer L15.3
- net ANT_OUT: now also L15.4
- net GND: now also L14.4, L15.3; no longer L14.3, L15.4
- net at D4.2 (A), L15.1, R?.1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: now also L14.3; no longer L14.4
- no-connect marks 0 -> 2
Changed lines of the file:
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@@
   (junction (at 156.21 72.39) (diameter 0) (color 0 0 0 0)
   )
-  (junction (at 87.63 62.23) (diameter 0) (color 0 0 0 0)
-  )
   (junction (at 156.21 116.205) (diameter 0) (color 0 0 0 0)
   )
+  (junction (at 128.905 62.23) (diameter 0) (color 0 0 0 0)
+  )
+  (no_connect (at 124.46 60.96))
+  (no_connect (at 124.46 88.9))
   (wire (pts (xy 147.32 87.63) (xy 147.32 83.82))
     (stroke (width 0) (type default))
@@
     (stroke (width 0) (type default))
   )
-  (wire (pts (xy 87.63 62.23) (xy 106.045 62.23))
+  (wire (pts (xy 128.905 62.23) (xy 147.955 62.23))
     (stroke (width 0) (type default))
   )
@@
     (stroke (width 0) (type default))
   )
-  (wire (pts (xy 100.965 67.31) (xy 106.045 67.31))
+  (wire (pts (xy 116.205 67.31) (xy 121.285 67.31))
     (stroke (width 0) (type default))
   )
@@
     (stroke (width 0) (type default))
   )
-  (wire (pts (xy 121.285 67.31) (xy 116.205 67.31))
+  (wire (pts (xy 93.345 67.31) (xy 106.045 67.31))
     (stroke (width 0) (type default))
   )
@@
     (stroke (width 0) (type default))
   )
+  (wire (pts (xy 116.205 82.55) (xy 128.905 82.55))
+    (stroke (width 0) (type default))
+  )
   (wire (pts (xy 147.32 76.2) (xy 147.32 72.39))
     (stroke (width 0) (type default))
@@
     (stroke (width 0) (type default))
   )
-  (wire (pts (xy 116.205 62.23) (xy 147.955 62.23))
+  (wire (pts (xy 116.205 62.23) (xy 128.905 62.23))
     (stroke (width 0) (type default))
   )
@@
     (stroke (width 0) (type default))
   )
-  (wire (pts (xy 87.63 82.55) (xy 106.045 82.55))
-    (stroke (width 0) (type default))
-  )
   (polyline (pts (xy 104.14 53.975) (xy 118.11 53.975))
     (stroke (width 0) (type default))
   )
-  (wire (pts (xy 121.285 67.31) (xy 121.285 74.295))
-    (stroke (width 0) (type default))
-  )
-  (wire (pts (xy 121.285 82.55) (xy 116.205 82.55))
+  (wire (pts (xy 100.965 82.55) (xy 106.045 82.55))
     (stroke (width 0) (type default))
   )
@@
     (stroke (width 0) (type default))
   )
-  (wire (pts (xy 93.345 74.295) (xy 93.345 87.63))
+  (wire (pts (xy 93.345 67.31) (xy 93.345 87.63))
     (stroke (width 0) (type default))
   )
@@
     (stroke (width 0) (type default))
   )
+  (wire (pts (xy 128.905 62.23) (xy 128.905 82.55))
+    (stroke (width 0) (type default))
+  )
   (polyline (pts (xy 104.14 53.975) (xy 104.14 90.805))
     (stroke (width 0) (type default))
@@
     (stroke (width 0) (type default))
   )
-  (wire (pts (xy 80.645 62.23) (xy 87.63 62.23))
+  (wire (pts (xy 80.645 62.23) (xy 106.045 62.23))
     (stroke (width 0) (type default))
   )
@@
     (stroke (width 0) (type default))
   )
-  (wire (pts (xy 87.63 62.23) (xy 87.63 82.55))
-    (stroke (width 0) (type default))
-  )
   (wire (pts (xy 176.53 116.205) (xy 172.72 116.205))
     (stroke (width 0) (type default))
@@
   )
   (wire (pts (xy 189.23 140.335) (xy 189.23 146.685))
-    (stroke (width 0) (type default))
-  )
-  (wire (pts (xy 121.285 74.295) (xy 93.345 74.295))
     (stroke (width 0) (type default))
   )
@@
     )
   )
-  (symbol (lib_id "power:GND") (at 100.965 67.31 0) (mirror y) (unit 1)
+  (symbol (lib_id "power:GND") (at 121.285 67.31 0) (unit 1)
     (in_bom yes) (on_board yes) (dnp no) (fields_autoplaced)
-    (property "Reference" "#PWR062" (at 100.965 73.66 0)
-      (effects (font (size 1.27 1.27)) hide)
-    )
-    (property "Value" "GND" (at 100.965 71.755 0)
-      (effects (font (size 1.27 1.27)))
-    )
-    (property "Footprint" "" (at 100.965 67.31 0)
-      (effects (font (size 1.27 1.27)) hide)
-    )
-    (property "Datasheet" "" (at 100.965 67.31 0)
+    (property "Reference" "#PWR062" (at 121.285 73.66 0)
+      (effects (font (size 1.27 1.27)) hide)
+    )
+    (property "Value" "GND" (at 121.285 71.755 0)
+      (effects (font (size 1.27 1.27)))
+    )
+    (property "Footprint" "" (at 121.285 67.31 0)
+      (effects (font (size 1.27 1.27)) hide)
+    )
+    (property "Datasheet" "" (at 121.285 67.31 0)
       (effects (font (size 1.27 1.27)) hide)
     )
@@
     )
   )
-  (symbol (lib_id "power:GND") (at 124.46 88.9 0) (unit 1)
-    (in_bom yes) (on_board yes) (dnp no) (fields_autoplaced)
-    (property "Reference" "#PWR0102" (at 124.46 95.25 0)
-      (effects (font (size 1.27 1.27)) hide)
-    )
-    (property "Value" "GND" (at 124.46 93.345 0)
-      (effects (font (size 1.27 1.27)))
-    )
-    (property "Footprint" "" (at 124.46 88.9 0)
-      (effects (font (size 1.27 1.27)) hide)
-    )
-    (property "Datasheet" "" (at 124.46 88.9 0)
-      (effects (font (size 1.27 1.27)) hide)
-    )
-    (pin "1")
-    (instances
-      (project "swr-bridge"
-        (path "/796eaa33-c177-43f1-9e4e-9ff4b4a4006e/00000000-0000-0000-0000-0000639cf678"
-          (reference "#PWR0102") (unit 1)
-        )
-        (path "/796eaa33-c177-43f1-9e4e-9ff4b4a4006e"
-          (reference "#PWR0102") (unit 1)
-        )
-      )
-      (project "main"
-        (path "/cb08c644-d155-44e5-86e1-31645eace055/f348e705-e1f2-401a-94bd-812b815f83a8/8653829a-ea60-4c18-8b01-1eb920d43d9e"
-          (reference "#PWR0134") (unit 1)
-        )
-      )
-    )
-  )
   (symbol (lib_id "Device:R") (at 189.23 136.525 0) (mirror y) (unit 1)
     (in_bom yes) (on_board yes) (dnp no)
@@
     )
   )
-  (symbol (lib_id "power:GND") (at 121.285 82.55 0) (mirror y) (unit 1)
+  (symbol (lib_id "power:GND") (at 100.965 82.55 0) (unit 1)
     (in_bom yes) (on_board yes) (dnp no) (fields_autoplaced)
-    (property "Reference" "#PWR069" (at 121.285 88.9 0)
-      (effects (font (size 1.27 1.27)) hide)
-    )
-    (property "Value" "GND" (at 121.285 81.28 0)
-      (effects (font (size 1.27 1.27)))
-    )
-    (property "Footprint" "" (at 121.285 82.55 0)
-      (effects (font (size 1.27 1.27)) hide)
-    )
-    (property "Datasheet" "" (at 121.285 82.55 0)
+    (property "Reference" "#PWR069" (at 100.965 88.9 0)
+      (effects (font (size 1.27 1.27)) hide)
+    )
+    (property "Value" "GND" (at 100.965 81.28 0)
+      (effects (font (size 1.27 1.27)))
+    )
+    (property "Footprint" "" (at 100.965 82.55 0)
+      (effects (font (size 1.27 1.27)) hide)
+    )
+    (property "Datasheet" "" (at 100.965 82.55 0)
       (effects (font (size 1.27 1.27)) hide)
     )
@@
         )
       )
-    )
-  )
-  (symbol (lib_id "power:GND") (at 124.46 60.96 0) (mirror x) (unit 1)
-    (in_bom yes) (on_board yes) (dnp no) (fields_autoplaced)
-    (property "Reference" "#PWR0102" (at 124.46 54.61 0)
-      (effects (font (size 1.27 1.27)) hide)
-    )
-    (property "Value" "GND" (at 124.46 56.515 0)
-      (effects (font (size 1.27 1.27)))
-    )
-    (property "Footprint" "" (at 124.46 60.96 0)
-      (effects (font (size 1.27 1.27)) hide)
-    )
-    (property "Datasheet" "" (at 124.46 60.96 0)
-      (effects (font (size 1.27 1.27)) hide)
-    )
-    (pin "1")
-    (instances
-      (project "swr-bridge"
-        (path "/796eaa33-c177-43f1-9e4e-9ff4b4a4006e/00000000-0000-0000-0000-0000639cf678"
-          (reference "#PWR0102") (unit 1)
-        )
-        (path "/796eaa33-c177-43f1-9e4e-9ff4b4a4006e"
-          (reference "#PWR0102") (unit 1)
-        )
-      )
-      (project "main"
-        (path "/cb08c644-d155-44e5-86e1-31645eace055/f348e705-e1f2-401a-94bd-812b815f83a8/8653829a-ea60-4c18-8b01-1eb920d43d9e"
-          (reference "#PWR094") (unit 1)
-        )
-      )
