File: main/modulator.kicad_sch (KiCad schematic)
At the start: 16 parts, among them U7 74CBTLV3253PW

Commit message: 50 Ohm resistors moved from modulator
Parts:
- removed R1 (x2): 50, symbol Device:R
Connections:
- net SDR_NEG: now also U7.7 (1A)
- net SDR_POS: now also U7.9 (2A)
Other:
- note removed: "TODO: Зачем здесь нужны резисторы?"
Changed lines of the file:
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@@
   (junction (at 130.81 96.52) (diameter 0) (color 0 0 0 0)
   )
-  (wire (pts (xy 153.67 91.44) (xy 158.75 91.44))
-    (stroke (width 0) (type default))
-  )
   (wire (pts (xy 110.49 129.54) (xy 110.49 101.6))
     (stroke (width 0) (type default))
@@
     (stroke (width 0) (type default))
   )
-  (wire (pts (xy 158.75 91.44) (xy 158.75 93.98))
-    (stroke (width 0) (type default))
-  )
   (wire (pts (xy 101.6 129.54) (xy 110.49 129.54))
     (stroke (width 0) (type default))
@@
     (stroke (width 0) (type default))
   )
-  (wire (pts (xy 180.34 88.9) (xy 171.45 88.9))
-    (stroke (width 0) (type default))
-  )
-  (wire (pts (xy 171.45 93.98) (xy 180.34 93.98))
-    (stroke (width 0) (type default))
-  )
   (wire (pts (xy 96.52 105.41) (xy 101.6 105.41))
     (stroke (width 0) (type default))
@@
     (stroke (width 0) (type default))
   )
-  (wire (pts (xy 163.83 88.9) (xy 153.67 88.9))
-    (stroke (width 0) (type default))
-  )
   (wire (pts (xy 143.51 58.42) (xy 143.51 60.96))
-    (stroke (width 0) (type default))
-  )
-  (wire (pts (xy 158.75 93.98) (xy 163.83 93.98))
     (stroke (width 0) (type default))
   )
@@
     (effects (font (size 1.27 1.27)) (justify left bottom))
   )
-  (text "TODO: Зачем здесь нужны резисторы?" (at 157.48 80.01 0)
-    (effects (font (size 1.27 1.27)) (justify left bottom))
-  )
   (hierarchical_label "VOUTR_NEG" (shape input) (at 73.66 105.41 180) (fields_autoplaced)
     (effects (font (size 1.27 1.27)) (justify right))
@@
     (effects (font (size 1.27 1.27)) (justify left))
   )
-  (hierarchical_label "SDR_POS" (shape output) (at 180.34 93.98 0) (fields_autoplaced)
+  (hierarchical_label "SDR_POS" (shape output) (at 153.67 91.44 0) (fields_autoplaced)
     (effects (font (size 1.27 1.27)) (justify left))
   )
@@
     (effects (font (size 1.27 1.27)) (justify right))
   )
-  (hierarchical_label "SDR_NEG" (shape output) (at 180.34 88.9 0) (fields_autoplaced)
+  (hierarchical_label "SDR_NEG" (shape output) (at 153.67 88.9 0) (fields_autoplaced)
     (effects (font (size 1.27 1.27)) (justify left))
   )
@@
     )
   )
-  (symbol (lib_id "Device:R") (at 167.64 88.9 90) (unit 1)
-    (in_bom yes) (on_board yes) (dnp no) (fields_autoplaced)
-    (property "Reference" "R1" (at 167.64 82.55 90)
-      (effects (font (size 1.27 1.27)))
-    )
-    (property "Value" "50" (at 167.64 85.09 90)
-      (effects (font (size 1.27 1.27)))
-    )
-    (property "Footprint" "" (at 167.64 90.678 90)
-      (effects (font (size 1.27 1.27)) hide)
-    )
-    (property "Datasheet" "~" (at 167.64 88.9 0)
-      (effects (font (size 1.27 1.27)) hide)
-    )
-    (pin "2")
-    (pin "1")
-    (instances
-      (project "main"
-        (path "/cb08c644-d155-44e5-86e1-31645eace055"
-          (reference "R1") (unit 1)
-        )
-        (path "/cb08c644-d155-44e5-86e1-31645eace055/f348e705-e1f2-401a-94bd-812b815f83a8/6911640e-2f8b-4689-850c-33e2fd821898"
-          (reference "R4") (unit 1)
-        )
-        (path "/cb08c644-d155-44e5-86e1-31645eace055/f348e705-e1f2-401a-94bd-812b815f83a8"
-          (reference "R17") (unit 1)
-        )
-        (path "/cb08c644-d155-44e5-86e1-31645eace055/f348e705-e1f2-401a-94bd-812b815f83a8/071bf193-b8ce-446c-a6f0-4f73f2e6bcab"
-          (reference "R33") (unit 1)
-        )
-      )
-    )
-  )
   (symbol (lib_id "power:GND") (at 101.6 140.97 0) (mirror y) (unit 1)
     (in_bom yes) (on_board yes) (dnp no) (fields_autoplaced)
@@
         )
       )
-    )
-  )
-  (symbol (lib_id "Device:R") (at 167.64 93.98 90) (mirror x) (unit 1)
-    (in_bom yes) (on_board yes) (dnp no) (fields_autoplaced)
-    (property "Reference" "R1" (at 167.64 97.79 90)
-      (effects (font (size 1.27 1.27)))
-    )
-    (property "Value" "50" (at 167.64 100.33 90)
-      (effects (font (size 1.27 1.27)))
-    )
-    (property "Footprint" "" (at 167.64 92.202 90)
-      (effects (font (size 1.27 1.27)) hide)
-    )
-    (property "Datasheet" "~" (at 167.64 93.98 0)
-      (effects (font (size 1.27 1.27)) hide)
-    )
-    (pin "2")
-    (pin "1")
-    (instances
-      (project "main"
-        (path "/cb08c644-d155-44e5-86e1-31645eace055"
-          (reference "R1") (unit 1)
-        )
-        (path "/cb08c644-d155-44e5-86e1-31645eace055/f348e705-e1f2-401a-94bd-812b815f83a8/6911640e-2f8b-4689-850c-33e2fd821898"
-          (reference "R4") (unit 1)
-        )
-        (path "/cb08c644-d155-44e5-86e1-31645eace055/f348e705-e1f2-401a-94bd-812b815f83a8"
-          (reference "R17") (unit 1)
-        )
-        (path "/cb08c644-d155-44e5-86e1-31645eace055/f348e705-e1f2-401a-94bd-812b815f83a8/071bf193-b8ce-446c-a6f0-4f73f2e6bcab"
-          (reference "R34") (unit 1)
-        )
-      )

Commit message: Phases table added
Other:
- note added: "Phases: 0 1 2 3 L- R- R+ L+ L+ R+ R- L-"
Changed lines of the file:
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@@
     (stroke (width 0) (type default))
+  )
+  (text "Phases:\n0	1	2	3\nL-	R-	R+	L+\nL+	R+	R-	L-" (at 123.19 140.335 0)
+    (effects (font (size 2.5 2.5)) (justify left bottom))
   )
   (text "TODO:\nВопрос:\nНужны ли разделительные конденсаторы\n(C46 и прочие) на большую ёмкость?"

Commit message: assigns
Parts:
- renumbered C58 to C40, U7 to U5
Changed lines of the file:
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@@
   (symbol (lib_id "Device:C") (at 101.6 87.63 0) (mirror y) (unit 1)
     (in_bom yes) (on_board yes) (dnp no)
-    (property "Reference" "C58" (at 97.79 86.36 0)
+    (property "Reference" "C40" (at 97.79 86.36 0)
       (effects (font (size 1.27 1.27)) (justify left))
     )
@@
   (symbol (lib_id "Device:C") (at 101.6 63.5 0) (mirror y) (unit 1)
     (in_bom yes) (on_board yes) (dnp no)
-    (property "Reference" "C58" (at 97.79 62.23 0)
+    (property "Reference" "C40" (at 97.79 62.23 0)
       (effects (font (size 1.27 1.27)) (justify left))
     )
@@
   (symbol (lib_id "Device:C") (at 101.6 111.76 0) (mirror y) (unit 1)
     (in_bom yes) (on_board yes) (dnp no)
-    (property "Reference" "C58" (at 97.79 110.49 0)
+    (property "Reference" "C40" (at 97.79 110.49 0)
       (effects (font (size 1.27 1.27)) (justify left))
     )
@@
   (symbol (lib_id "Device:C") (at 82.55 81.28 90) (unit 1)
     (in_bom yes) (on_board yes) (dnp no) (fields_autoplaced)
-    (property "Reference" "C58" (at 82.55 73.66 90)
+    (property "Reference" "C40" (at 82.55 73.66 90)
       (effects (font (size 1.27 1.27)))
     )
@@
   (symbol (lib_id "Device:C") (at 82.55 129.54 90) (unit 1)
     (in_bom yes) (on_board yes) (dnp no) (fields_autoplaced)
-    (property "Reference" "C58" (at 82.55 121.92 90)
+    (property "Reference" "C40" (at 82.55 121.92 90)
       (effects (font (size 1.27 1.27)))
     )
@@
   (symbol (lib_id "Device:C") (at 82.55 105.41 90) (unit 1)
     (in_bom yes) (on_board yes) (dnp no) (fields_autoplaced)
-    (property "Reference" "C58" (at 82.55 97.79 90)
+    (property "Reference" "C40" (at 82.55 97.79 90)
       (effects (font (size 1.27 1.27)))
     )
@@
   (symbol (lib_id "Device:C") (at 148.59 64.77 0) (unit 1)
     (in_bom yes) (on_board yes) (dnp no) (fields_autoplaced)
-    (property "Reference" "C58" (at 152.4 63.5 0)
+    (property "Reference" "C40" (at 152.4 63.5 0)
       (effects (font (size 1.27 1.27)) (justify left))
     )
@@
   (symbol (lib_id "power:+3.3V") (at 143.51 58.42 0) (unit 1)
     (in_bom yes) (on_board yes) (dnp no) (fields_autoplaced)
-    (property "Reference" "#PWR059" (at 143.51 62.23 0)
+    (property "Reference" "#PWR066" (at 143.51 62.23 0)
       (effects (font (size 1.27 1.27)) hide)
     )
@@
   (symbol (lib_id "Device:C") (at 101.6 135.89 0) (mirror y) (unit 1)
     (in_bom yes) (on_board yes) (dnp no)
-    (property "Reference" "C58" (at 97.79 134.62 0)
+    (property "Reference" "C40" (at 97.79 134.62 0)
       (effects (font (size 1.27 1.27)) (justify left))
     )
@@
   (symbol (lib_id "Analog_Switch:SN74CBT3253") (at 143.51 99.06 0) (mirror y) (unit 1)
     (in_bom yes) (on_board yes) (dnp no) (fields_autoplaced)
-    (property "Reference" "U7" (at 141.3159 81.28 0)
+    (property "Reference" "U5" (at 141.3159 81.28 0)
       (effects (font (size 1.27 1.27)) (justify left))
     )
@@
   (symbol (lib_id "Device:C") (at 82.55 57.15 90) (unit 1)
     (in_bom yes) (on_board yes) (dnp no) (fields_autoplaced)
-    (property "Reference" "C58" (at 82.55 49.53 90)
-      (effects (font (size 1.27 1.27)))
-    )
+    (property "Reference" "C40" (at 82.55 49.53 90)
+      (effects (font (size 1.27 1.27)))
+    )

Commit message: QSE: name and title added
Other:
- note added: "Based onfrom Selenite Lite SDR HF Transceiver by Dmitrii Rudnev"
- title: (none) -> Quadrature Sampling Exciter (QSE)
- moved on the sheet: C40, R1, U5

Commit message: Title fixed
Other:
- note added: "Based on Selenite Lite SDR HF Transceiver by Dmitrii Rudnev"
- note removed: "Based onfrom Selenite Lite SDR HF Transceiver by Dmitrii Rudnev"
Changed lines of the file:
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@@
     (effects (font (size 1.27 1.27)) (justify left bottom))
   )
-  (text "Based onfrom Selenite Lite SDR HF Transceiver by Dmitrii Rudnev"
+  (text "Based on Selenite Lite SDR HF Transceiver by Dmitrii Rudnev"
     (at 82.55 25.4 0)
     (effects (font (size 2.5 2.5)) (justify left bottom))

Commit message: comment added
Other:
- note added: "TODO: Необходимость этих резисторов и их номинал под вопросом"
Changed lines of the file:
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@@
+    (effects (font (size 1.27 1.27)) (justify left bottom))
+  )
+  (text "TODO: Необходимость этих резисторов и их номинал под вопросом"
+    (at 95.885 52.07 0)
     (effects (font (size 1.27 1.27)) (justify left bottom))
   )

Commit message: QSD_EN->RX_EN, QSE_EN->TX_EN, FIXME removed
Connections:
- net QSE_EN renamed ENABLE
Changed lines of the file:
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@@
     (effects (font (size 1.27 1.27)) (justify right))
   )
-  (hierarchical_label "QSE_EN" (shape input) (at 165.735 113.03 0) (fields_autoplaced)
+  (hierarchical_label "ENABLE" (shape input) (at 165.735 113.03 0) (fields_autoplaced)
     (effects (font (size 1.27 1.27)) (justify left))
   )
