File: main/voltage_booster.kicad_sch (KiCad schematic)
At the start: 1 part, among them J10 LM2596 DC-DC module

Commit message: Power supply moved to battery
Parts:
- removed J10: LM2596 DC-DC module, symbol Connector:Conn_01x04_Pin
- added J9: LM2596 DC-DC module, symbol Connector:Conn_01x05_Pin
Connections:
- net gnd: now also J9.2 (Pin_2), J9.4 (Pin_4)
- net increased_voltage: now also J9.3 (Pin_3)
- net input+: now also J9.1 (Pin_1)
- new net en: J9.5 (Pin_5)
Changed lines of the file:
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@@
     (effects (font (size 1.27 1.27)) (justify left bottom))
+  )
+  (hierarchical_label "en" (shape input) (at 141.605 86.995 0) (fields_autoplaced)
+    (effects (font (size 1.27 1.27)) (justify left))
   )
   (hierarchical_label "gnd" (shape input) (at 141.605 84.455 0) (fields_autoplaced)
@@
   (hierarchical_label "input+" (shape input) (at 141.605 76.835 0) (fields_autoplaced)
     (effects (font (size 1.27 1.27)) (justify left))
-  )
-  (symbol (lib_id "Connector:Conn_01x04_Pin") (at 136.525 79.375 0) (unit 1)
-    (in_bom yes) (on_board yes) (dnp no) (fields_autoplaced)
-    (property "Reference" "J10" (at 137.16 72.39 0)
-      (effects (font (size 1.27 1.27)))
-    )
-    (property "Value" "LM2596 DC-DC module" (at 137.16 74.93 0)
-      (effects (font (size 1.27 1.27)))
-    )
-    (property "Footprint" "" (at 136.525 79.375 0)
-      (effects (font (size 1.27 1.27)) hide)
-    )
-    (property "Datasheet" "~" (at 136.525 79.375 0)
-      (effects (font (size 1.27 1.27)) hide)
-    )
-    (pin "3")
-    (pin "4")
-    (pin "2")
-    (pin "1")
-    (instances
-      (project "main"
-        (path "/cb08c644-d155-44e5-86e1-31645eace055/6adb75eb-c8b3-4528-8354-bbd7827d10ad"
-          (reference "J10") (unit 1)
-        )
-      )
-    )
   )
   (symbol (lib_id "power:PWR_FLAG") (at 156.21 81.915 0) (unit 1)
@@
     (instances
       (project "main"
-        (path "/cb08c644-d155-44e5-86e1-31645eace055/6adb75eb-c8b3-4528-8354-bbd7827d10ad"
+        (path "/cb08c644-d155-44e5-86e1-31645eace055/c60e9004-e534-4568-b2af-6f7f65cfe3f5/a00e2fe3-8fb5-4127-b32d-290a96cb9615"
           (reference "#FLG04") (unit 1)
         )
       )
+    )
+  )
+  (symbol (lib_id "Connector:Conn_01x05_Pin") (at 136.525 81.915 0) (unit 1)
+    (in_bom yes) (on_board yes) (dnp no) (fields_autoplaced)
+    (property "Reference" "J9" (at 134.62 80.645 0)
+      (effects (font (size 1.27 1.27)) (justify right))
+    )
+    (property "Value" "LM2596 DC-DC module" (at 134.62 83.185 0)
+      (effects (font (size 1.27 1.27)) (justify right))
+    )
+    (property "Footprint" "" (at 136.525 81.915 0)
+      (effects (font (size 1.27 1.27)) hide)
+    )
+    (property "Datasheet" "~" (at 136.525 81.915 0)
+      (effects (font (size 1.27 1.27)) hide)
+    )
+    (pin "1")
+    (pin "5")
+    (pin "4")
+    (pin "3")
+    (pin "2")
+    (instances
+      (project "main"
+        (path "/cb08c644-d155-44e5-86e1-31645eace055/c60e9004-e534-4568-b2af-6f7f65cfe3f5/a00e2fe3-8fb5-4127-b32d-290a96cb9615"
+          (reference "J9") (unit 1)
+        )
+      )
