File: main/power.kicad_sch (KiCad schematic)
At the start: 7 parts, among them J3 USB_B_Micro, J4 Screw_Terminal_01x02

Commit message: PWR flags added
Other:
- moved on the sheet: D1
Changed lines of the file:
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@@
   (junction (at 137.16 121.92) (diameter 0) (color 0 0 0 0)
   )
-  (junction (at 106.68 72.39) (diameter 0) (color 0 0 0 0)
+  (junction (at 101.6 72.39) (diameter 0) (color 0 0 0 0)
+  )
+  (junction (at 109.22 72.39) (diameter 0) (color 0 0 0 0)
   )
   (junction (at 124.46 72.39) (diameter 0) (color 0 0 0 0)
@@
     (stroke (width 0) (type default))
   )
+  (wire (pts (xy 124.46 72.39) (xy 139.7 72.39))
+    (stroke (width 0) (type default))
+  )
   (wire (pts (xy 149.86 111.76) (xy 147.32 111.76))
     (stroke (width 0) (type default))
@@
     (stroke (width 0) (type default))
   )
-  (wire (pts (xy 139.7 72.39) (xy 124.46 72.39))
+  (wire (pts (xy 109.22 72.39) (xy 113.03 72.39))
     (stroke (width 0) (type default))
   )
@@
     (stroke (width 0) (type default))
   )
-  (wire (pts (xy 106.68 72.39) (xy 113.03 72.39))
+  (wire (pts (xy 101.6 72.39) (xy 109.22 72.39))
     (stroke (width 0) (type default))
   )
@@
     (stroke (width 0) (type default))
   )
-  (wire (pts (xy 106.68 68.58) (xy 106.68 72.39))
+  (wire (pts (xy 101.6 68.58) (xy 101.6 72.39))
     (stroke (width 0) (type default))
   )
@@
     (effects (font (size 1.27 1.27)) (justify right))
   )
-  (hierarchical_label "power_5V" (shape output) (at 106.68 68.58 90) (fields_autoplaced)
+  (hierarchical_label "power_5V" (shape output) (at 101.6 68.58 90) (fields_autoplaced)
     (effects (font (size 1.27 1.27)) (justify left))
   )
@@
     (effects (font (size 1.27 1.27)) (justify right))
   )
-  (hierarchical_label "gnd" (shape bidirectional) (at 106.68 80.01 270) (fields_autoplaced)
+  (hierarchical_label "gnd" (shape bidirectional) (at 101.6 80.01 270) (fields_autoplaced)
     (effects (font (size 1.27 1.27)) (justify right))
   )
@@
     )
   )
-  (symbol (lib_id "Device:D") (at 106.68 76.2 270) (unit 1)
-    (in_bom yes) (on_board yes) (dnp no) (fields_autoplaced)
-    (property "Reference" "D1" (at 109.22 74.93 90)
-      (effects (font (size 1.27 1.27)) (justify left))
-    )
-    (property "Value" "D" (at 109.22 77.47 90)
-      (effects (font (size 1.27 1.27)) (justify left))
-    )
-    (property "Footprint" "" (at 106.68 76.2 0)
-      (effects (font (size 1.27 1.27)) hide)
-    )
-    (property "Datasheet" "~" (at 106.68 76.2 0)
-      (effects (font (size 1.27 1.27)) hide)
-    )
-    (property "Sim.Device" "D" (at 106.68 76.2 0)
-      (effects (font (size 1.27 1.27)) hide)
-    )
-    (property "Sim.Pins" "1=K 2=A" (at 106.68 76.2 0)
+  (symbol (lib_id "Device:D") (at 101.6 76.2 270) (unit 1)
+    (in_bom yes) (on_board yes) (dnp no) (fields_autoplaced)
+    (property "Reference" "D1" (at 104.14 74.93 90)
+      (effects (font (size 1.27 1.27)) (justify left))
+    )
+    (property "Value" "D" (at 104.14 77.47 90)
+      (effects (font (size 1.27 1.27)) (justify left))
+    )
+    (property "Footprint" "" (at 101.6 76.2 0)
+      (effects (font (size 1.27 1.27)) hide)
+    )
+    (property "Datasheet" "~" (at 101.6 76.2 0)
+      (effects (font (size 1.27 1.27)) hide)
+    )
+    (property "Sim.Device" "D" (at 101.6 76.2 0)
+      (effects (font (size 1.27 1.27)) hide)
+    )
+    (property "Sim.Pins" "1=K 2=A" (at 101.6 76.2 0)
       (effects (font (size 1.27 1.27)) hide)
     )
@@
         )
         (path "/cb08c644-d155-44e5-86e1-31645eace055/c60e9004-e534-4568-b2af-6f7f65cfe3f5"
-          (reference "D1") (unit 1)
+          (reference "D3") (unit 1)
         )
       )
@@
         )
       )
+    )
+  )
+  (symbol (lib_id "power:PWR_FLAG") (at 109.22 72.39 0) (unit 1)
+    (in_bom yes) (on_board yes) (dnp no) (fields_autoplaced)
+    (property "Reference" "#FLG02" (at 109.22 70.485 0)
+      (effects (font (size 1.27 1.27)) hide)
+    )
+    (property "Value" "PWR_FLAG" (at 109.22 67.31 0)
+      (effects (font (size 1.27 1.27)))
+    )
+    (property "Footprint" "" (at 109.22 72.39 0)
+      (effects (font (size 1.27 1.27)) hide)
+    )
+    (property "Datasheet" "~" (at 109.22 72.39 0)
+      (effects (font (size 1.27 1.27)) hide)
+    )
+    (pin "1")
+    (instances
+      (project "main"
+        (path "/cb08c644-d155-44e5-86e1-31645eace055/c60e9004-e534-4568-b2af-6f7f65cfe3f5"
+          (reference "#FLG02") (unit 1)
+        )
+      )

Commit message: Power supply moved to battery
Parts:
- removed D2: D, symbol Device:D
- removed F2: Fuse, symbol Device:Fuse
- added BT2: LiFePo4 32700 3.2V, symbol Device:Battery_Cell
- added C8: 10uF, symbol Device:C_Polarized
- added U100: AP1117-33, Package_TO_SOT_SMD:SOT-223-3_TabPin2, symbol Regulator_Linear:AP1117-33
- J4: value Screw_Terminal_01x02 -> external_power
Connections:
- net gnd: now also BT2.2 (-), C8.2, U100.1 (GND)
- net at F2.2, J4.1 (Pin_1): now also D1.1 (K), BT2.1 (+)
- net at D1.4 (VCC): now also J3.1 (VBUS)
- net power_5V renamed power_unstable
- net power_unstable: now also U100.3 (VI); no longer D1.1 (K)
- new net power_3V: C8.1, U100.2 (VO)
Other:
- added sheet DC-DC Booster (voltage_booster.kicad_sch)
- moved on the sheet: D1, F2, J3, J4

Commit message: RX and TX labels on main
Changed lines of the file:
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@@
     (stroke (width 0) (type default))
-  )
-  (label "POS" (at 58.42 41.91 0) (fields_autoplaced)
-    (effects (font (size 1.27 1.27)) (justify left bottom))
   )
   (hierarchical_label "usb_dp" (shape bidirectional) (at 128.27 90.17 180) (fields_autoplaced)

Commit message: Battery connection changed
Connections:
- net power_unstable: now also D1.1 (K)
- net at BT2.1 (+), F2.2, J4.1 (Pin_1): no longer D1.1 (K)
Other:
- moved on the sheet: BT2, D1
Changed lines of the file:
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@@
+    (stroke (width 0) (type default))
+  )
+  (wire (pts (xy 47.625 41.91) (xy 47.625 47.625))
     (stroke (width 0) (type default))
   )
@@
     (stroke (width 0) (type default))
   )
-  (wire (pts (xy 57.15 43.815) (xy 57.15 41.91))
+  (wire (pts (xy 57.15 41.91) (xy 57.15 43.815))
     (stroke (width 0) (type default))
   )
@@
     (stroke (width 0) (type default))
   )
+  (wire (pts (xy 47.625 55.245) (xy 47.625 62.865))
+    (stroke (width 0) (type default))
+  )
   (wire (pts (xy 83.82 41.91) (xy 90.17 41.91))
     (stroke (width 0) (type default))
@@
     (stroke (width 0) (type default))
   )
-  (wire (pts (xy 47.625 53.975) (xy 57.15 53.975))
-    (stroke (width 0) (type default))
-  )
   (wire (pts (xy 138.43 87.63) (xy 128.27 87.63))
     (stroke (width 0) (type default))
@@
     (stroke (width 0) (type default))
   )
-  (wire (pts (xy 47.625 53.975) (xy 47.625 55.245))
-    (stroke (width 0) (type default))
-  )
   (wire (pts (xy 138.43 90.17) (xy 132.08 90.17))
     (stroke (width 0) (type default))
@@
     (stroke (width 0) (type default))
   )
+  (wire (pts (xy 47.625 41.91) (xy 57.15 41.91))
+    (stroke (width 0) (type default))
+  )
   (wire (pts (xy 177.8 43.18) (xy 180.975 43.18))
     (stroke (width 0) (type default))
@@
     (effects (font (size 1.27 1.27)) (justify right))
   )
-  (symbol (lib_id "Device:Battery_Cell") (at 47.625 60.325 0) (mirror y) (unit 1)
+  (symbol (lib_id "Device:Battery_Cell") (at 57.15 59.055 0) (mirror y) (unit 1)
     (in_bom yes) (on_board yes) (dnp no)
-    (property "Reference" "BT2" (at 43.815 57.2135 0)
-      (effects (font (size 1.27 1.27)) (justify left))
-    )
-    (property "Value" "LiFePo4 32700 3.2V" (at 43.815 59.7535 0)
-      (effects (font (size 1.27 1.27)) (justify left))
-    )
-    (property "Footprint" "" (at 47.625 58.801 90)
-      (effects (font (size 1.27 1.27)) hide)
-    )
-    (property "Datasheet" "~" (at 47.625 58.801 90)
+    (property "Reference" "BT2" (at 53.34 55.9435 0)
+      (effects (font (size 1.27 1.27)) (justify left))
+    )
+    (property "Value" "LiFePo4 32700 3.2V" (at 53.34 58.4835 0)
+      (effects (font (size 1.27 1.27)) (justify left))
+    )
+    (property "Footprint" "" (at 57.15 57.531 90)
+      (effects (font (size 1.27 1.27)) hide)
+    )
+    (property "Datasheet" "~" (at 57.15 57.531 90)
       (effects (font (size 1.27 1.27)) hide)
     )
@@
     )
   )
-  (symbol (lib_id "Device:D") (at 57.15 57.785 90) (mirror x) (unit 1)
+  (symbol (lib_id "Device:D") (at 47.625 51.435 90) (mirror x) (unit 1)
     (in_bom yes) (on_board yes) (dnp no)
-    (property "Reference" "D1" (at 54.61 56.515 90)
-      (effects (font (size 1.27 1.27)) (justify left))
-    )
-    (property "Value" "D" (at 54.61 59.055 90)
-      (effects (font (size 1.27 1.27)) (justify left))
-    )
-    (property "Footprint" "" (at 57.15 57.785 0)
-      (effects (font (size 1.27 1.27)) hide)
-    )
-    (property "Datasheet" "~" (at 57.15 57.785 0)
-      (effects (font (size 1.27 1.27)) hide)
-    )
-    (property "Sim.Device" "D" (at 57.15 57.785 0)
-      (effects (font (size 1.27 1.27)) hide)
-    )
-    (property "Sim.Pins" "1=K 2=A" (at 57.15 57.785 0)
-      (effects (font (size 1.27 1.27)) hide)
-    )
+    (property "Reference" "D1" (at 45.085 50.165 90)
+      (effects (font (size 1.27 1.27)) (justify left))
+    )
+    (property "Value" "D" (at 45.085 52.705 90)
+      (effects (font (size 1.27 1.27)) (justify left))
+    )
+    (property "Footprint" "" (at 47.625 51.435 0)
+      (effects (font (size 1.27 1.27)) hide)
+    )
+    (property "Datasheet" "~" (at 47.625 51.435 0)
+      (effects (font (size 1.27 1.27)) hide)
+    )
+    (property "Sim.Device" "D" (at 47.625 51.435 0)
+      (effects (font (size 1.27 1.27)) hide)
+    )
+    (property "Sim.Pins" "1=K 2=A" (at 47.625 51.435 0)
+      (effects (font (size 1.27 1.27)) hide)
+    )
